Commit message: ur components spawning - no colours yet

File: src/Universal_Robots_ROS2_Description/urdf/ur10.xacro (robot description, xacro)
@@ -138,14 +138,11 @@
         <origin xyz="0 0 0" rpy="0 0 0"/>
         <geometry>
-          <mesh filename="package://ur_description/meshes/ur10/collision/trolley1.STL"/>
-        </geometry>
-        <material name="">
-          <color rgba="0.89 0.91 0.93 1.0"/>
-        </material>
-      </visual>
-      <collision>
-        <origin xyz="0 0 0" rpy="0 0 0"/>
-        <geometry>
-          <mesh filename="package://ur_description/meshes/ur10/collision/trolley1.STL"/>
+          <xacro:get_mesh name="trolley1" type="visual"/>
+        </geometry>
+      </visual>
+      <collision>
+        <origin xyz="0 0 0" rpy="0 0 0"/>
+        <geometry>
+          <xacro:get_mesh name="trolley1" type="collision"/>
         </geometry>
       </collision>
@@ -162,14 +159,11 @@
         <origin xyz="0 0 0" rpy="0 0 0"/>
         <geometry>
-          <mesh filename="package://ur_description/meshes/ur10_feeder/UR10_feeder.STL"/>
-        </geometry>
-        <material name="">
-          <color rgba="0.59 0.61 0.73 1.0"/>
-        </material>
-      </visual>
-      <collision>
-        <origin xyz="0 0 0" rpy="0 0 0"/>
-        <geometry>
-          <mesh filename="package://ur_description/meshes/ur10_feeder/UR10_feeder.STL"/>
+          <xacro:get_mesh name="ur10_feeder" type="visual"/>
+        </geometry>
+      </visual>
+      <collision>
+        <origin xyz="0 0 0" rpy="0 0 0"/>
+        <geometry>
+          <xacro:get_mesh name="ur10_feeder" type="collision"/>
         </geometry>
       </collision>
@@ -186,14 +180,11 @@
         <origin xyz="0 0 0" rpy="0 0 0"/>
         <geometry>
-          <mesh filename="package://ur_description/meshes/ur10_feeder/heating_plate1.STL"/>
-        </geometry>
-        <material name="">
-          <color rgba="0.85 0.86 0.92 1.0"/>
-        </material>
-      </visual>
-      <collision>
-        <origin xyz="0 0 0" rpy="0 0 0"/>
-        <geometry>
-          <mesh filename="package://ur_description/meshes/ur10_feeder/heating_plate1.STL"/>
+          <xacro:get_mesh name="heating_plate1" type="visual"/>
+        </geometry>
+      </visual>
+      <collision>
+        <origin xyz="0 0 0" rpy="0 0 0"/>
+        <geometry>
+          <xacro:get_mesh name="heating_plate1" type="collision"/>
         </geometry>
       </collision>
@@ -210,14 +201,11 @@
         <origin xyz="0 0 0" rpy="0 0 0"/>
         <geometry>
-          <mesh filename="package://ur_description/meshes/ur10_feeder/heating_plate2.STL"/>
-        </geometry>
-        <material name="">
-          <color rgba="0.85 0.86 0.92 1.0"/>
-        </material>
-      </visual>
-      <collision>
-        <origin xyz="0 0 0" rpy="0 0 0"/>
-        <geometry>
-          <mesh filename="package://ur_description/meshes/ur10_feeder/heating_plate2.STL"/>
+          <xacro:get_mesh name="heating_plate2" type="visual"/>
+        </geometry>
+      </visual>
+      <collision>
+        <origin xyz="0 0 0" rpy="0 0 0"/>
+        <geometry>
+          <xacro:get_mesh name="heating_plate2" type="collision"/>
         </geometry>
       </collision>
@@ -234,14 +222,11 @@
         <origin xyz="0 0 0" rpy="0 0 0"/>
         <geometry>
-          <mesh filename="package://ur_description/meshes/ur10_feeder/heating_plate_cover1.STL"/>
-        </geometry>
-        <material name="">
-          <color rgba="0.2 0.2 0.2 1.0"/>
-        </material>
-      </visual>
-      <collision>
-        <origin xyz="0 0 0" rpy="0 0 0"/>
-        <geometry>
-          <mesh filename="package://ur_description/meshes/ur10_feeder/heating_plate_cover1.STL"/>
+          <xacro:get_mesh name="heating_plate_cover1" type="visual"/>
+        </geometry>
+      </visual>
+      <collision>
+        <origin xyz="0 0 0" rpy="0 0 0"/>
+        <geometry>
+          <xacro:get_mesh name="heating_plate_cover1" type="collision"/>
         </geometry>
       </collision>
@@ -258,14 +243,11 @@
         <origin xyz="0 0 0" rpy="0 0 0"/>
         <geometry>
-          <mesh filename="package://ur_description/meshes/ur10_feeder/heating_plate_cover2.STL"/>
-        </geometry>
-        <material name="">
-          <color rgba="0.2 0.2 0.2 1.0"/>
-        </material>
-      </visual>
-      <collision>
-        <origin xyz="0 0 0" rpy="0 0 0"/>
-        <geometry>
-          <mesh filename="package://ur_description/meshes/ur10_feeder/heating_plate_cover2.STL"/>
+          <xacro:get_mesh name="heating_plate_cover2" type="visual"/>
+        </geometry>
+      </visual>
+      <collision>
+        <origin xyz="0 0 0" rpy="0 0 0"/>
+        <geometry>
+          <xacro:get_mesh name="heating_plate_cover2" type="collision"/>
         </geometry>
       </collision>
@@ -282,14 +264,11 @@
         <origin xyz="0 0 0" rpy="0 0 0"/>
         <geometry>
-          <mesh filename="package://ur_description/meshes/ur10_feeder/heating_plate_cover3-1.STL"/>
-        </geometry>
-        <material name="">
-          <color rgba="0.0 0.0 0.0 1.0"/>
-        </material>
-      </visual>
-      <collision>
-        <origin xyz="0 0 0" rpy="0 0 0"/>
-        <geometry>
-          <mesh filename="package://ur_description/meshes/ur10_feeder/heating_plate_cover3-1.STL"/>
+          <xacro:get_mesh name="heating_plate_cover3_1" type="visual"/>
+        </geometry>
+      </visual>
+      <collision>
+        <origin xyz="0 0 0" rpy="0 0 0"/>
+        <geometry>
+          <xacro:get_mesh name="heating_plate_cover3_1" type="collision"/>
         </geometry>
       </collision>
@@ -306,14 +285,11 @@
         <origin xyz="0 0 0" rpy="0 0 0"/>
         <geometry>
-          <mesh filename="package://ur_description/meshes/ur10_feeder/heating_plate_cover3-2.STL"/>
-        </geometry>
-        <material name="">
-          <color rgba="0.0 0.0 0.0 1.0"/>
-        </material>
-      </visual>
-      <collision>
-        <origin xyz="0 0 0" rpy="0 0 0"/>
-        <geometry>
-          <mesh filename="package://ur_description/meshes/ur10_feeder/heating_plate_cover3-2.STL"/>
+          <xacro:get_mesh name="heating_plate_cover3_2" type="visual"/>
+        </geometry>
+      </visual>
+      <collision>
+        <origin xyz="0 0 0" rpy="0 0 0"/>
+        <geometry>
+          <xacro:get_mesh name="heating_plate_cover3_2" type="collision"/>
         </geometry>
       </collision>
@@ -330,14 +306,11 @@
         <origin xyz="0 0 0" rpy="0 0 0"/>
         <geometry>
-          <mesh filename="package://ur_description/meshes/ur10/collision/UR_plate.STL"/>
-        </geometry>
-        <material name="">
-          <color rgba="0.69 0.71 0.83 1.0"/>
-        </material>
-      </visual>
-      <collision>
-        <origin xyz="0 0 0" rpy="0 0 0"/>
-        <geometry>
-          <mesh filename="package://ur_description/meshes/ur10/collision/UR_plate.STL"/>
+          <xacro:get_mesh name="ur10_plate" type="visual"/>
+        </geometry>
+      </visual>
+      <collision>
+        <origin xyz="0 0 0" rpy="0 0 0"/>
+        <geometry>
+          <xacro:get_mesh name="ur10_plate" type="collision"/>
         </geometry>
       </collision>
