Commit message: deleted quickchanger gripper

File: src/Universal_Robots_ROS2_Description/urdf/gazebo_materials.xacro (robot description, xacro)
@@ -30,23 +30,4 @@
   <gazebo reference="ur10_plate_link">
     <material>Gazebo/Grey</material>
-  </gazebo>
-  <!-- Quickchanger and Gripper Components -->
-  <gazebo reference="quickchanger_link">
-    <material>Gazebo/Grey</material>
-  </gazebo>
-  <gazebo reference="suction_master_link">
-    <material>Gazebo/Grey</material>
-  </gazebo>
-  <gazebo reference="suction_link">
-    <material>Gazebo/DarkGrey</material>
-  </gazebo>
-  <gazebo reference="gripper_link">
-    <material>Gazebo/Black</material>
-  </gazebo>
-  <gazebo reference="tooltip1_link">
-    <material>Gazebo/LightGrey</material>
-  </gazebo>
-  <gazebo reference="tooltip2_link">
-    <material>Gazebo/LightGrey</material>
   </gazebo>
   <!-- Vision Components -->

File: src/Universal_Robots_ROS2_Description/urdf/inc/ur_transmissions.xacro (robot description, xacro)
@@ -61,23 +61,4 @@
       </actuator>
     </transmission>
-    <!-- UR Robot Gripper Tooltips -->
-    <transmission name="tooltip1_trans">
-      <type>transmission_interface/SimpleTransmission</type>
-      <joint name="tooltip1_joint">
-        <hardwareInterface>${hw_interface}</hardwareInterface>
-      </joint>
-      <actuator name="tooltip1_motor">
-        <mechanicalReduction>1</mechanicalReduction>
-      </actuator>
-    </transmission>
-    <transmission name="tooltip2_trans">
-      <type>transmission_interface/SimpleTransmission</type>
-      <joint name="tooltip2_joint">
-        <hardwareInterface>${hw_interface}</hardwareInterface>
-      </joint>
-      <actuator name="tooltip2_motor">
-        <mechanicalReduction>1</mechanicalReduction>
-      </actuator>
-    </transmission>
     <!-- ARF Axis Joints -->
     <transmission name="arf_axis_1_trans">

File: src/Universal_Robots_ROS2_Description/urdf/ur.ros2_control.xacro (robot description, xacro)
@@ -121,25 +121,4 @@
           <!-- initial position for the FakeSystem and simulation -->
           <param name="initial_value">${initial_positions['wrist_3_joint']}</param>
-        </state_interface>
-        <state_interface name="velocity"/>
-        <state_interface name="effort"/>
-      </joint>
-      <!-- UR Robot Gripper Tooltips -->
-      <joint name="${tf_prefix}tooltip1_joint">
-        <command_interface name="position"/>
-        <command_interface name="velocity"/>
-        <state_interface name="position">
-          <!-- initial position for the FakeSystem and simulation -->
-          <param name="initial_value">${initial_positions['tooltip1_joint']}</param>
-        </state_interface>
-        <state_interface name="velocity"/>
-        <state_interface name="effort"/>
-      </joint>
-      <joint name="${tf_prefix}tooltip2_joint">
-        <command_interface name="position"/>
-        <command_interface name="velocity"/>
-        <state_interface name="position">
-          <!-- initial position for the FakeSystem and simulation -->
-          <param name="initial_value">${initial_positions['tooltip2_joint']}</param>
         </state_interface>
         <state_interface name="velocity"/>

File: src/Universal_Robots_ROS2_Description/urdf/ur.urdf.xacro (robot description, xacro)
@@ -5,6 +5,4 @@
    <!-- import main macro -->
    <xacro:include filename="$(find ur_description)/urdf/ur_macro.xacro"/>
-   <!-- import gripper macro -->
-   <xacro:include filename="$(find ur_description)/urdf/quickchanger_gripper_suction.xacro"/>
    <!-- import vision macro -->
    <xacro:include filename="$(find ur_description)/urdf/vision.xacro"/>
@@ -138,6 +136,4 @@
      <origin xyz="0 0 0" rpy="0 0 0" />          <!-- position robot in the world -->
    </xacro:ur_robot>
-    <!-- attach gripper -->
-    <xacro:quickchanger_gripper_suction parent="$(arg tf_prefix)wrist_3_link"/>
    <xacro:if value="$(arg sim_gazebo)">
     <!-- Gazebo plugins -->

Commit message: grippers working now - controllers setup done

File: src/Universal_Robots_ROS2_Description/urdf/gazebo_materials.xacro (robot description, xacro)
@@ -30,4 +30,23 @@
   <gazebo reference="ur10_plate_link">
     <material>Gazebo/Grey</material>
+  </gazebo>
+  <!-- Quickchanger and Gripper Components -->
+  <gazebo reference="quickchanger_link">
+    <material>Gazebo/Grey</material>
+  </gazebo>
+  <gazebo reference="suction_master_link">
+    <material>Gazebo/Grey</material>
+  </gazebo>
+  <gazebo reference="suction_link">
+    <material>Gazebo/DarkGrey</material>
+  </gazebo>
+  <gazebo reference="gripper_link">
+    <material>Gazebo/Black</material>
+  </gazebo>
+  <gazebo reference="tooltip1_link">
+    <material>Gazebo/LightGrey</material>
+  </gazebo>
+  <gazebo reference="tooltip2_link">
+    <material>Gazebo/LightGrey</material>
   </gazebo>
   <!-- Vision Components -->

File: src/Universal_Robots_ROS2_Description/urdf/quickchanger_grippers.xacro (robot description, xacro)
@@ -5,4 +5,91 @@
   <xacro:property name="sec_mesh_files" value="${quickchanger_grippers_visual_params['mesh_files']}" scope="parent"/>
   <xacro:property name="force_abs_paths" value="true" scope="parent"/>
+    <!-- quickchanger_link -->
+    <link name="quickchanger_link">
+      <visual>
+        <origin xyz="0 0 0" rpy="0 0 0"/>
+        <geometry>
+          <xacro:get_mesh name="quickchanger" type="visual"/>
+        </geometry>
+        <material name="${sec_mesh_files['quickchanger']['visual']['material']['name']}">
+          <color rgba="${sec_mesh_files['quickchanger']['visual']['material']['color']}"/>
+        </material>
+      </visual>
+      <collision>
+        <origin xyz="0 0 0" rpy="0 0 0"/>
+        <geometry>
+          <xacro:get_mesh name="quickchanger" type="collision"/>
+        </geometry>
+      </collision>
+      <inertial>
+        <mass value="2.0"/>
+        <origin xyz="0 0 0" rpy="0 0 0"/>
+        <inertia ixx="1e-5" ixy="0" ixz="0" iyy="1e-5" iyz="0" izz="1e-5"/>
+      </inertial>
+    </link>
+    <!-- quickchanger_joint -->
+    <joint name="quickchanger_joint" type="fixed">
+      <parent link="${parent}"/>
+      <child link="quickchanger_link"/>
+      <origin xyz="0 0 0" rpy="0 0 -1.57"/>
+    </joint>
+    <!-- suction_master_link -->
+    <link name="suction_master_link">
+      <visual>
+        <origin xyz="0 0 0" rpy="0 0 0"/>
+        <geometry>
+          <xacro:get_mesh name="suction_master" type="visual"/>
+        </geometry>
+        <material name="${sec_mesh_files['suction_master']['visual']['material']['name']}">
+          <color rgba="${sec_mesh_files['suction_master']['visual']['material']['color']}"/>
+        </material>
+      </visual>
+      <collision>
+        <origin xyz="0 0 0" rpy="0 0 0"/>
+        <geometry>
+          <xacro:get_mesh name="suction_master" type="collision"/>
+        </geometry>
+      </collision>
+      <inertial>
+        <mass value="1.0"/>
+        <origin xyz="0 0 0" rpy="0 0 0"/>
+        <inertia ixx="1e-5" ixy="0" ixz="0" iyy="1e-5" iyz="0" izz="1e-5"/>
+      </inertial>
+    </link>
+    <!-- suction_master_joint -->
+    <joint name="suction_master_joint" type="fixed">
+      <parent link="quickchanger_link"/>
+      <child link="suction_master_link"/>
+      <origin xyz="0 0 0" rpy="0 0 0"/>
+    </joint>
+    <!-- suction_link -->
+    <link name="suction_link">
+      <visual>
+        <origin xyz="0 0 0" rpy="0 0 0"/>
+        <geometry>
+          <xacro:get_mesh name="suction" type="visual"/>
+        </geometry>
+        <material name="${sec_mesh_files['suction']['visual']['material']['name']}">
+          <color rgba="${sec_mesh_files['suction']['visual']['material']['color']}"/>
+        </material>
+      </visual>
+      <collision>
+        <origin xyz="0 0 0" rpy="0 0 0"/>
+        <geometry>
+          <xacro:get_mesh name="suction" type="collision"/>
+        </geometry>
+      </collision>
+      <inertial>
+        <mass value="1.0"/>
+        <origin xyz="0 0 0" rpy="0 0 0"/>
+        <inertia ixx="1e-5" ixy="0" ixz="0" iyy="1e-5" iyz="0" izz="1e-5"/>
+      </inertial>
+    </link>
+    <!-- suction_joint -->
+    <joint name="suction_joint" type="fixed">
+      <parent link="suction_master_link"/>
+      <child link="suction_link"/>
+      <origin xyz="0 0 0" rpy="0 0 0"/>
+    </joint>
     <!-- gripper_link -->
     <link name="gripper_link">
@@ -30,5 +117,5 @@
     <!-- gripper_joint -->
     <joint name="gripper_joint" type="fixed">
-      <parent link="${parent}"/>
+      <parent link="quickchanger_link"/>
       <child link="gripper_link"/>
       <origin xyz="0 0 0" rpy="0 0 0"/>

Commit message: suction link joint to fixed from revolute

File: src/Universal_Robots_ROS2_Description/urdf/gazebo_materials.xacro (robot description, xacro)
@@ -82,4 +82,7 @@
     <preserveFixedJoint>true</preserveFixedJoint>
   </gazebo>
+  <gazebo reference="suction_joint">
+    <preserveFixedJoint>true</preserveFixedJoint>
+  </gazebo>
   <gazebo reference="gripper_joint">
     <preserveFixedJoint>true</preserveFixedJoint>

File: src/Universal_Robots_ROS2_Description/urdf/inc/ur_transmissions.xacro (robot description, xacro)
@@ -80,14 +80,4 @@
   </actuator>
 </transmission>
-<!-- Vacuum Gripper Joint -->
-<transmission name="suction_trans">
-  <type>transmission_interface/SimpleTransmission</type>
-  <joint name="suction_joint">
-    <hardwareInterface>${hw_interface}</hardwareInterface>
-  </joint>
-  <actuator name="suction_motor">
-    <mechanicalReduction>1</mechanicalReduction>
-  </actuator>
-</transmission>
     <!-- ARF Axis Joints -->
     <transmission name="arf_axis_1_trans">

File: src/Universal_Robots_ROS2_Description/urdf/quickchanger_grippers.xacro (robot description, xacro)
@@ -87,11 +87,8 @@
     </link>
     <!-- suction_joint -->
-    <joint name="suction_joint" type="revolute">
+    <joint name="suction_joint" type="fixed">
       <parent link="suction_master_link"/>
       <child link="suction_link"/>
       <origin xyz="0 0 0" rpy="0 0 0"/>
-      <axis xyz="0 0 1"/>
-      <limit effort="50" velocity="50" lower="0" upper="0"/>
-      <dynamics damping="0.0" friction="10"/>
     </joint>
     <!-- gripper_link -->

File: src/Universal_Robots_ROS2_Description/urdf/ur.ros2_control.xacro (robot description, xacro)
@@ -140,14 +140,4 @@
           <!-- initial position for the FakeSystem and simulation -->
           <param name="initial_value">${initial_positions['tooltip2_joint']}</param>
-        </state_interface>
-        <state_interface name="velocity"/>
-        <state_interface name="effort"/>
-      </joint>
-      <!-- Vacuum Gripper Joint -->
-      <joint name="${tf_prefix}suction_joint">
-        <command_interface name="position"/>
-        <state_interface name="position">
-          <!-- initial position for the FakeSystem and simulation -->
-          <param name="initial_value">${initial_positions['suction_joint']}</param>
         </state_interface>
         <state_interface name="velocity"/>

File: src/Universal_Robots_ROS2_Description/urdf/ur.urdf.xacro (robot description, xacro)
@@ -148,15 +148,4 @@
         <parameters>$(arg simulation_controllers)</parameters>
       </plugin>
-    <!-- Vacuum Gripper Plugin -->
-    <plugin name="vacuum_gripper" filename="libgazebo_ros_vacuum_gripper.so">
-      <ros>
-        <namespace>/demo</namespace>
-        <remapping>switch:=switch_demo</remapping>
-        <remapping>grasping:=grasping_demo</remapping>
-      </ros>
-      <link_name>suction_link</link_name>
-      <max_distance>0.5</max_distance>
-      <fixed>ground_plane</fixed>
-    </plugin>
     </gazebo>
   </xacro:if>

Commit message: changed object colour for better visualisation

File: src/Universal_Robots_ROS2_Description/urdf/gazebo_materials.xacro (robot description, xacro)
@@ -8,23 +8,5 @@
   </gazebo>
   <gazebo reference="ur10_feeder_link">
-    <material>Gazebo/Grey</material>
-  </gazebo>
-  <gazebo reference="ur10_heating_plate_1_link">
     <material>Gazebo/LightGrey</material>
-  </gazebo>
-  <gazebo reference="ur10_heating_plate_2_link">
-    <material>Gazebo/LightGrey</material>
-  </gazebo>
-  <gazebo reference="ur10_heating_plate_cover_1_link">
-    <material>Gazebo/DarkGrey</material>
-  </gazebo>
-  <gazebo reference="ur10_heating_plate_cover_2_link">
-    <material>Gazebo/DarkGrey</material>
-  </gazebo>
-  <gazebo reference="ur10_heating_plate_cover_3_1_link">
-    <material>Gazebo/Black</material>
-  </gazebo>
-  <gazebo reference="ur10_heating_plate_cover_3_2_link">
-    <material>Gazebo/Black</material>
   </gazebo>
   <gazebo reference="ur10_plate_link">
@@ -64,5 +46,5 @@
   </gazebo>
   <gazebo reference="suction_link">
-    <material>Gazebo/DarkGrey</material>
+    <material>Gazebo/LightGrey</material>
   </gazebo>
   <gazebo reference="gripper_link">
@@ -93,5 +75,5 @@
   </gazebo>
   <gazebo reference="vision_cam_jig_link">
-    <material>Gazebo/Purple</material>
+    <material>Gazebo/Red</material>
   </gazebo>
   <gazebo reference="vision_feeder_link">
@@ -113,5 +95,5 @@
   </gazebo>
   <gazebo reference="tool_changer_link">
-    <material>Gazebo/Yellow</material>
+    <material>Gazebo/Blue</material>
   </gazebo>
   <!-- Toolchanger Joint Components -->
@@ -133,11 +115,11 @@
   </gazebo>
   <gazebo reference="arf_slider_jig_link">
-    <material>Gazebo/Blue</material>
+    <material>Gazebo/Yellow</material>
   </gazebo>
   <gazebo reference="arf_front_aircyl_link">
-    <material>Gazebo/Blue</material>
+    <material>Gazebo/Yellow</material>
   </gazebo>
   <gazebo reference="arf_back_aircyl_link">
-    <material>Gazebo/Blue</material>
+    <material>Gazebo/Yellow</material>
   </gazebo>
   <!-- ARF Joint Components -->
