Commit message: added sdf files for pick objects (objects under ur10 feeder) + snap link1 and link2

File: src/Universal_Robots_ROS2_Description/urdf/ur_macro.xacro (robot description, xacro)
@@ -191,178 +191,4 @@
       <origin xyz="0.525 0.025 0.82" rpy="0 0 0"/>
     </joint>
-    <!-- heating plate 1 link -->
-    <link name="${tf_prefix}ur10_heating_plate_1_link">
-      <visual>
-        <origin xyz="0 0 0" rpy="0 0 0"/>
-        <geometry>
-          <xacro:get_mesh name="heating_plate1" type="visual"/>
-        </geometry>
-        <material name="${sec_mesh_files['heating_plate1']['visual']['material']['name']}">
-          <color rgba="${sec_mesh_files['heating_plate1']['visual']['material']['color']}"/>
-        </material>
-      </visual>
-      <collision>
-        <origin xyz="0 0 0" rpy="0 0 0"/>
-        <geometry>
-          <xacro:get_mesh name="heating_plate1" type="collision"/>
-        </geometry>
-      </collision>
-      <inertial>
-        <mass value="5.0"/>
-        <origin xyz="0 0 0.01" rpy="0 0 0"/>
-        <inertia ixx="0.01" ixy="0" ixz="0" iyy="0.01" iyz="0" izz="0.02"/>
-      </inertial>
-    </link>
-    <!-- ur feeder to heating plate 1 joint -->
-    <joint name="${tf_prefix}ur10_heating_plate_1_joint" type="fixed">
-      <parent link="${tf_prefix}ur10_feeder_link" />
-      <child link="${tf_prefix}ur10_heating_plate_1_link" />
-      <origin xyz="0.0351 -0.1379 0.01" rpy="0 0 0"/>
-    </joint>
-    <!-- heating plate 2 link -->
-    <link name="${tf_prefix}ur10_heating_plate_2_link">
-      <visual>
-        <origin xyz="0 0 0" rpy="0 0 0"/>
-        <geometry>
-          <xacro:get_mesh name="heating_plate2" type="visual"/>
-        </geometry>
-        <material name="${sec_mesh_files['heating_plate2']['visual']['material']['name']}">
-          <color rgba="${sec_mesh_files['heating_plate2']['visual']['material']['color']}"/>
-        </material>
-      </visual>
-      <collision>
-        <origin xyz="0 0 0" rpy="0 0 0"/>
-        <geometry>
-          <xacro:get_mesh name="heating_plate2" type="collision"/>
-        </geometry>
-      </collision>
-      <inertial>
-        <mass value="5.0"/>
-        <origin xyz="0 0 0.01" rpy="0 0 0"/>
-        <inertia ixx="0.01" ixy="0" ixz="0" iyy="0.01" iyz="0" izz="0.02"/>
-      </inertial>
-    </link>
-    <!-- ur feeder to heating plate 2 joint -->
-    <joint name="${tf_prefix}ur10_heating_plate_2_joint" type="fixed">
-      <parent link="${tf_prefix}ur10_feeder_link" />
-      <child link="${tf_prefix}ur10_heating_plate_2_link" />
-      <origin xyz="0.0351 -0.2521 0.01" rpy="0 0 0"/>
-    </joint>
-    <!-- heating plate cover 1 link -->
-    <link name="${tf_prefix}ur10_heating_plate_cover_1_link">
-      <visual>
-        <origin xyz="0 0 0" rpy="0 0 0"/>
-        <geometry>
-          <xacro:get_mesh name="heating_plate_cover1" type="visual"/>
-        </geometry>
-        <material name="${sec_mesh_files['heating_plate_cover1']['visual']['material']['name']}">
-          <color rgba="${sec_mesh_files['heating_plate_cover1']['visual']['material']['color']}"/>
-        </material>
-      </visual>
-      <collision>
-        <origin xyz="0 0 0" rpy="0 0 0"/>
-        <geometry>
-          <xacro:get_mesh name="heating_plate_cover1" type="collision"/>
-        </geometry>
-      </collision>
-      <inertial>
-        <mass value="2.0"/>
-        <origin xyz="0 0 0.01" rpy="0 0 0"/>
-        <inertia ixx="0.005" ixy="0" ixz="0" iyy="0.005" iyz="0" izz="0.01"/>
-      </inertial>
-    </link>
-    <!-- ur feeder to heating plate cover 1 joint -->
-    <joint name="${tf_prefix}ur10_heating_plate_cover_1_joint" type="fixed">
-      <parent link="${tf_prefix}ur10_feeder_link" />
-      <child link="${tf_prefix}ur10_heating_plate_cover_1_link" />
-      <origin xyz="-0.034 0.125 0.01" rpy="0 0 0"/>
-    </joint>
-    <!-- heating plate cover 2 link -->
-    <link name="${tf_prefix}ur10_heating_plate_cover_2_link">
-      <visual>
-        <origin xyz="0 0 0" rpy="0 0 0"/>
-        <geometry>
-          <xacro:get_mesh name="heating_plate_cover2" type="visual"/>
-        </geometry>
-        <material name="${sec_mesh_files['heating_plate_cover2']['visual']['material']['name']}">
-          <color rgba="${sec_mesh_files['heating_plate_cover2']['visual']['material']['color']}"/>
-        </material>
-      </visual>
-      <collision>
-        <origin xyz="0 0 0" rpy="0 0 0"/>
-        <geometry>
-          <xacro:get_mesh name="heating_plate_cover2" type="collision"/>
-        </geometry>
-      </collision>
-      <inertial>
-        <mass value="2.0"/>
-        <origin xyz="0 0 0.01" rpy="0 0 0"/>
-        <inertia ixx="0.005" ixy="0" ixz="0" iyy="0.005" iyz="0" izz="0.01"/>
-      </inertial>
-    </link>
-    <!-- ur feeder to heating plate cover 2 joint -->
-    <joint name="${tf_prefix}ur10_heating_plate_cover_2_joint" type="fixed">
-      <parent link="${tf_prefix}ur10_feeder_link" />
-      <child link="${tf_prefix}ur10_heating_plate_cover_2_link" />
-      <origin xyz="0.094 0.125 0.01" rpy="0 0 0"/>
-    </joint>
-    <!-- heating plate cover 3-1 link -->
-    <link name="${tf_prefix}ur10_heating_plate_cover_3_1_link">
-      <visual>
-        <origin xyz="0 0 0" rpy="0 0 0"/>
-        <geometry>
-          <xacro:get_mesh name="heating_plate_cover3_1" type="visual"/>
-        </geometry>
-        <material name="${sec_mesh_files['heating_plate_cover3_1']['visual']['material']['name']}">
-          <color rgba="${sec_mesh_files['heating_plate_cover3_1']['visual']['material']['color']}"/>
-        </material>
-      </visual>
-      <collision>
-        <origin xyz="0 0 0" rpy="0 0 0"/>
-        <geometry>
-          <xacro:get_mesh name="heating_plate_cover3_1" type="collision"/>
-        </geometry>
-      </collision>
-      <inertial>
-        <mass value="1.5"/>
-        <origin xyz="0 0 0.01" rpy="0 0 0"/>
-        <inertia ixx="0.003" ixy="0" ixz="0" iyy="0.003" iyz="0" izz="0.006"/>
-      </inertial>
-    </link>
-    <!-- ur feeder to heating plate cover 3-1 joint -->
-    <joint name="${tf_prefix}ur10_heating_plate_cover_3_1_joint" type="fixed">
-      <parent link="${tf_prefix}ur10_feeder_link" />
-      <child link="${tf_prefix}ur10_heating_plate_cover_3_1_link" />
-      <origin xyz="-0.156 -0.0095 0.01" rpy="0 0 0"/>
-    </joint>
-    <!-- heating plate cover 3-2 link -->
-    <link name="${tf_prefix}ur10_heating_plate_cover_3_2_link">
-      <visual>
-        <origin xyz="0 0 0" rpy="0 0 0"/>
-        <geometry>
-          <xacro:get_mesh name="heating_plate_cover3_2" type="visual"/>
-        </geometry>
-        <material name="${sec_mesh_files['heating_plate_cover3_2']['visual']['material']['name']}">
-          <color rgba="${sec_mesh_files['heating_plate_cover3_2']['visual']['material']['color']}"/>
-        </material>
-      </visual>
-      <collision>
-        <origin xyz="0 0 0" rpy="0 0 0"/>
-        <geometry>
-          <xacro:get_mesh name="heating_plate_cover3_2" type="collision"/>
-        </geometry>
-      </collision>
-      <inertial>
-        <mass value="1.5"/>
-        <origin xyz="0 0 0.01" rpy="0 0 0"/>
-        <inertia ixx="0.003" ixy="0" ixz="0" iyy="0.003" iyz="0" izz="0.006"/>
-      </inertial>
-    </link>
-    <!-- ur feeder to heating plate cover 3-2 joint -->
-    <joint name="${tf_prefix}ur10_heating_plate_cover_3_2_joint" type="fixed">
-      <parent link="${tf_prefix}ur10_feeder_link" />
-      <child link="${tf_prefix}ur10_heating_plate_cover_3_2_link" />
-      <origin xyz="-0.156 0.1705 0.01" rpy="0 0 0"/>
-    </joint>
     <!-- UR plate link-->
     <link name="${tf_prefix}ur10_plate_link">

Commit message: edited postion of ur10 heating plate

File: src/Universal_Robots_ROS2_Description/urdf/ur_macro.xacro (robot description, xacro)
@@ -218,5 +218,5 @@
       <parent link="${tf_prefix}ur10_trolley_link" />
       <child link="${tf_prefix}ur10_plate_link" />
-      <origin xyz="0 0.05 0.835" rpy="0 0 0"/>
+      <origin xyz="0 0 0.850" rpy="0 0 0"/>
     </joint>
     <!-- ur robot base link -->

Commit message: ur10 heating plate postiion edited

File: src/Universal_Robots_ROS2_Description/urdf/ur_macro.xacro (robot description, xacro)
@@ -218,5 +218,5 @@
       <parent link="${tf_prefix}ur10_trolley_link" />
       <child link="${tf_prefix}ur10_plate_link" />
-      <origin xyz="0 0 0.850" rpy="0 0 0"/>
+      <origin xyz="0 -0.05 0.835" rpy="0 0 0"/>
     </joint>
     <!-- ur robot base link -->
