Commit message: added joint components for gazebo so theyu show up in model list

File: src/Universal_Robots_ROS2_Description/urdf/denso.xacro (robot description, xacro)
@@ -60,5 +60,5 @@
     </link>
     <!-- trolley to denso slider jig joint -->
-    <joint name="denso slider jig joint" type="fixed">
+    <joint name="denso_slider_jig_joint" type="fixed">
       <parent link="denso_trolley_link" />
       <child link="denso_slider_jig_link" />

File: src/Universal_Robots_ROS2_Description/urdf/gazebo_materials.xacro (robot description, xacro)
@@ -3,5 +3,5 @@
   <!-- Gazebo material definitions for workcell components -->
   <!-- These ensure proper color rendering in Gazebo simulation -->
-  <!-- UR Workcell Components -->
+  <!-- UR Link Components -->
   <gazebo reference="ur10_trolley_link">
     <material>Gazebo/LightGrey</material>
@@ -31,5 +31,30 @@
     <material>Gazebo/Grey</material>
   </gazebo>
-  <!-- Quickchanger and Gripper Components -->
+  <!-- UR Joint Components-->
+  <gazebo reference="ur10_feeder_joint">
+    <preserveFixedJoint>true</preserveFixedJoint>
+  </gazebo>
+  <gazebo reference="ur10_heating_plate_1_joint">
+    <preserveFixedJoint>true</preserveFixedJoint>
+  </gazebo>
+  <gazebo reference="ur10_heating_plate_2_joint">
+    <preserveFixedJoint>true</preserveFixedJoint>
+  </gazebo>
+  <gazebo reference="ur10_heating_plate_cover_1_joint">
+    <preserveFixedJoint>true</preserveFixedJoint>
+  </gazebo>
+  <gazebo reference="ur10_heating_plate_cover_2_joint">
+    <preserveFixedJoint>true</preserveFixedJoint>
+  </gazebo>
+  <gazebo reference="ur10_heating_plate_cover_3_1_joint">
+    <preserveFixedJoint>true</preserveFixedJoint>
+  </gazebo>
+  <gazebo reference="ur10_heating_plate_cover_3_2_joint">
+    <preserveFixedJoint>true</preserveFixedJoint>
+  </gazebo>
+  <gazebo reference="ur10_plate_joint">
+    <preserveFixedJoint>true</preserveFixedJoint>
+  </gazebo>
+  <!-- Quickchanger and Gripper Link Components -->
   <gazebo reference="quickchanger_link">
     <material>Gazebo/Grey</material>
@@ -50,5 +75,15 @@
     <material>Gazebo/LightGrey</material>
   </gazebo>
-  <!-- Vision Components -->
+  <!-- Quickchanger and Gripper Joint Components -->
+  <gazebo reference="quickchanger_joint">
+    <preserveFixedJoint>true</preserveFixedJoint>
+  </gazebo>
+  <gazebo reference="suction_master_joint">
+    <preserveFixedJoint>true</preserveFixedJoint>
+  </gazebo>
+  <gazebo reference="gripper_joint">
+    <preserveFixedJoint>true</preserveFixedJoint>
+  </gazebo>
+  <!-- Vision LinkComponents -->
   <gazebo reference="vision_trolley_link">
     <material>Gazebo/LightGrey</material>
@@ -60,5 +95,15 @@
     <material>Gazebo/Orange</material>
   </gazebo>
-  <!-- Toolchanger Components -->
+  <!-- Vision Joint Components -->
+  <gazebo reference="vision_trolley_joint">
+    <preserveFixedJoint>true</preserveFixedJoint>
+  </gazebo>
+  <gazebo reference="vision_cam_jig_joint">
+    <preserveFixedJoint>true</preserveFixedJoint>
+  </gazebo>
+  <gazebo reference="vision_feeder_joint">
+    <preserveFixedJoint>true</preserveFixedJoint>
+  </gazebo>
+  <!-- Toolchanger Link Components -->
   <gazebo reference="toolchanger_trolley_link">
     <material>Gazebo/LightGrey</material>
@@ -67,5 +112,9 @@
     <material>Gazebo/Yellow</material>
   </gazebo>
-  <!-- ARF Components -->
+  <!-- Toolchanger Joint Components -->
+  <gazebo reference="toolchanger_tool_changer_joint">
+    <preserveFixedJoint>true</preserveFixedJoint>
+  </gazebo>
+  <!-- ARF Link Components -->
   <gazebo reference="arf_trolley_link">
     <material>Gazebo/LightGrey</material>
@@ -89,5 +138,12 @@
     <material>Gazebo/Blue</material>
   </gazebo>
-  <!-- Denso Components -->
+  <!-- ARF Joint Components -->
+  <gazebo reference="arf_base_plate_joint">
+    <preserveFixedJoint>true</preserveFixedJoint>
+  </gazebo>
+  <gazebo reference="arf_slider_base_joint">
+    <preserveFixedJoint>true</preserveFixedJoint>
+  </gazebo>
+  <!-- Denso Link Components -->
   <gazebo reference="denso_trolley_link">
     <material>Gazebo/LightGrey</material>
@@ -96,3 +152,10 @@
     <material>Gazebo/Grey</material>
   </gazebo>
+  <!-- Denso Joint Components -->
+  <gazebo reference="denso_trolley_joint">
+    <preserveFixedJoint>true</preserveFixedJoint>
+  </gazebo>
+  <gazebo reference="denso_slider_jig_joint">
+    <preserveFixedJoint>true</preserveFixedJoint>
+  </gazebo>
 </robot>

File: src/Universal_Robots_ROS2_Description/urdf/ur_macro.xacro (robot description, xacro)
@@ -215,5 +215,5 @@
     </link>
     <!-- ur feeder to heating plate 1 joint -->
-    <joint name="${tf_prefix}ur10_heating_plate1_joint" type="fixed">
+    <joint name="${tf_prefix}ur10_heating_plate_1_joint" type="fixed">
       <parent link="${tf_prefix}ur10_feeder_link" />
       <child link="${tf_prefix}ur10_heating_plate_1_link" />
@@ -244,5 +244,5 @@
     </link>
     <!-- ur feeder to heating plate 2 joint -->
-    <joint name="${tf_prefix}ur10_heating_plate2_joint" type="fixed">
+    <joint name="${tf_prefix}ur10_heating_plate_2_joint" type="fixed">
       <parent link="${tf_prefix}ur10_feeder_link" />
       <child link="${tf_prefix}ur10_heating_plate_2_link" />
@@ -273,5 +273,5 @@
     </link>
     <!-- ur feeder to heating plate cover 1 joint -->
-    <joint name="${tf_prefix}ur10_heating_plate_cover1_joint" type="fixed">
+    <joint name="${tf_prefix}ur10_heating_plate_cover_1_joint" type="fixed">
       <parent link="${tf_prefix}ur10_feeder_link" />
       <child link="${tf_prefix}ur10_heating_plate_cover_1_link" />
@@ -302,5 +302,5 @@
     </link>
     <!-- ur feeder to heating plate cover 2 joint -->
-    <joint name="${tf_prefix}ur10_heating_plate_cover2_joint" type="fixed">
+    <joint name="${tf_prefix}ur10_heating_plate_cover_2_joint" type="fixed">
       <parent link="${tf_prefix}ur10_feeder_link" />
       <child link="${tf_prefix}ur10_heating_plate_cover_2_link" />
@@ -331,5 +331,5 @@
     </link>
     <!-- ur feeder to heating plate cover 3-1 joint -->
-    <joint name="${tf_prefix}ur10_heating_plate_cover3_1_joint" type="fixed">
+    <joint name="${tf_prefix}ur10_heating_plate_cover_3_1_joint" type="fixed">
       <parent link="${tf_prefix}ur10_feeder_link" />
       <child link="${tf_prefix}ur10_heating_plate_cover_3_1_link" />
@@ -360,5 +360,5 @@
     </link>
     <!-- ur feeder to heating plate cover 3-2 joint -->
-    <joint name="${tf_prefix}ur10_heating_plate_cover3_2_joint" type="fixed">
+    <joint name="${tf_prefix}ur10_heating_plate_cover_3_2_joint" type="fixed">
       <parent link="${tf_prefix}ur10_feeder_link" />
       <child link="${tf_prefix}ur10_heating_plate_cover_3_2_link" />

Commit message: denso joint move working - terminal command

File: src/Universal_Robots_ROS2_Description/urdf/denso.xacro (robot description, xacro)
@@ -66,5 +66,9 @@
     </joint>
     <!-- Add Denso robot connected to the slider jig -->
-    <xacro:denso_robot parent="denso_slider_jig_link" />
+    <xacro:denso_robot
+      parent="denso_slider_jig_link"
+      sim="true"
+      namespace="denso_"
+      model="hsr065a1_n32" />
   </xacro:macro>
 </robot>

File: src/denso_robot_drivers_ros2/denso_robot_descriptions/robots/hsr065a1_n32/urdf/denso_robot.ros2_control.xacro (robot description, xacro)
@@ -13,6 +13,4 @@
     ">
     <ros2_control name="${namespace}${name}" type="system">
-	<!-- joint limits include -->
-	<xacro:include filename="$(find denso_robot_descriptions)/robots/${model}/urdf/denso_robot_joint_limits.xacro" />
       <hardware>
         <xacro:if value="${sim}">
@@ -38,5 +36,53 @@
         </xacro:unless>
       </hardware>
-      <xacro:denso_robot_control_limits namespace="${namespace}" />
+      <!-- Joint definitions for simulation -->
+      <xacro:if value="${sim}">
+        <!-- Denso robot arm joints -->
+        <joint name="${namespace}joint_1">
+          <command_interface name="position">
+            <param name="min">-2.268928</param>
+            <param name="max">2.268928</param>
+          </command_interface>
+          <state_interface name="position"/>
+          <state_interface name="velocity"/>
+        </joint>
+        <joint name="${namespace}joint_2">
+          <command_interface name="position">
+            <param name="min">-2.617994</param>
+            <param name="max">2.617994</param>
+          </command_interface>
+          <state_interface name="position"/>
+          <state_interface name="velocity"/>
+        </joint>
+        <joint name="${namespace}joint_3">
+          <command_interface name="position">
+            <param name="min">-0.100000</param>
+            <param name="max">0.220000</param>
+          </command_interface>
+          <state_interface name="position"/>
+          <state_interface name="velocity"/>
+        </joint>
+        <joint name="${namespace}joint_4">
+          <command_interface name="position">
+            <param name="min">-6.283185</param>
+            <param name="max">6.283185</param>
+          </command_interface>
+          <state_interface name="position"/>
+          <state_interface name="velocity"/>
+        </joint>
+        <!-- Denso axis joint -->
+        <joint name="${namespace}axis_joint">
+          <command_interface name="position">
+            <param name="min">0.0</param>
+            <param name="max">0.5</param>
+          </command_interface>
+          <state_interface name="position"/>
+          <state_interface name="velocity"/>
+        </joint>
+      </xacro:if>
+      <!-- Joint limits for real hardware -->
+      <xacro:unless value="${sim}">
+        <xacro:denso_robot_control_limits namespace="${namespace}" />
+      </xacro:unless>
     </ros2_control>
   </xacro:macro>

File: src/denso_robot_drivers_ros2/denso_robot_descriptions/robots/hsr065a1_n32/urdf/denso_robot_macro.xacro (robot description, xacro)
@@ -36,6 +36,6 @@
     <!-- ros2 control instance -->
     <xacro:denso_robot_ros2_control
-      name="GazeboSystem"
-      namespace="${namespace}"
+      name="denso"
+      namespace=""
       sim="${sim}"
       model="${model}"
@@ -58,9 +58,4 @@
     <!-- links -  main serial chain -->
     <xacro:denso_robot_arm_kinematics namespace="${namespace}" model="${model}" parent="${parent}" />
-    <!-- <gazebo>
-	    <plugin filename="libgazebo_ros2_control.so" name="gazebo_ros2_control">
-      		<parameters>$(find denso_robot_moveit_config)/robots/${model}/config/denso_robot_controllers.yaml</parameters>
-    	</plugin>
-  	</gazebo> -->
   </xacro:macro>
 </robot>
