Commit message: remove collision property from suction link

File: src/Universal_Robots_ROS2_Description/urdf/quickchanger_grippers.xacro (robot description, xacro)
@@ -74,10 +74,4 @@
         </material>
       </visual>
-      <collision>
-        <origin xyz="0 0 0" rpy="0 0 0"/>
-        <geometry>
-          <xacro:get_mesh name="suction" type="collision"/>
-        </geometry>
-      </collision>
       <inertial>
         <mass value="1.0"/>

Commit message: edited ur quickchanger joint origin - ur orientation working properly now

File: src/Universal_Robots_ROS2_Description/urdf/quickchanger_grippers.xacro (robot description, xacro)
@@ -8,5 +8,5 @@
     <link name="quickchanger_link">
       <visual>
-        <origin xyz="0 0 0" rpy="0 0 0"/>
+        <origin xyz="0 0 0" rpy="0 0 -1.57"/>
         <geometry>
           <xacro:get_mesh name="quickchanger" type="visual"/>
@@ -17,5 +17,5 @@
       </visual>
       <collision>
-        <origin xyz="0 0 0" rpy="0 0 0"/>
+        <origin xyz="0 0 0" rpy="0 0 -1.57"/>
         <geometry>
           <xacro:get_mesh name="quickchanger" type="collision"/>
@@ -32,10 +32,10 @@
       <parent link="${parent}"/>
       <child link="quickchanger_link"/>
-      <origin xyz="0 0 0" rpy="0 0 -1.57"/>
+      <origin xyz="0 0 0" rpy="0 0 0"/>
     </joint>
     <!-- suction_master_link -->
     <link name="suction_master_link">
       <visual>
-        <origin xyz="0 0 0" rpy="0 0 0"/>
+        <origin xyz="0 0 0" rpy="0 0 -1.57"/>
         <geometry>
           <xacro:get_mesh name="suction_master" type="visual"/>
@@ -46,5 +46,5 @@
       </visual>
       <collision>
-        <origin xyz="0 0 0" rpy="0 0 0"/>
+        <origin xyz="0 0 0" rpy="0 0 -1.57"/>
         <geometry>
           <xacro:get_mesh name="suction_master" type="collision"/>
@@ -66,5 +66,5 @@
     <link name="suction_link">
       <visual>
-        <origin xyz="0 0 0" rpy="0 0 0"/>
+        <origin xyz="0 0 0" rpy="0 0 -1.57"/>
         <geometry>
           <xacro:get_mesh name="suction" type="visual"/>
@@ -89,5 +89,5 @@
     <link name="gripper_link">
       <visual>
-        <origin xyz="0 0 0" rpy="0 0 0"/>
+        <origin xyz="0 0 0" rpy="0 0 -1.57"/>
         <geometry>
           <xacro:get_mesh name="gripper" type="visual"/>
@@ -118,5 +118,5 @@
     <link name="tooltip1_link">
       <visual>
-        <origin xyz="0 0 0" rpy="0 0 0"/>
+        <origin xyz="0 0 0" rpy="0 0 -1.57"/>
         <geometry>
           <xacro:get_mesh name="tooltip1" type="visual"/>
@@ -143,5 +143,5 @@
       <child link="tooltip1_link"/>
       <origin xyz="0 0 0" rpy="0 0 0"/>
-      <axis xyz="1 0 0"/>
+      <axis xyz="0 -1 0"/>
       <limit lower="-1.0" upper="0.041" effort="50" velocity="10"/>
     </joint>
@@ -149,5 +149,5 @@
     <link name="tooltip2_link">
       <visual>
-        <origin xyz="0 0 0" rpy="0 0 0"/>
+        <origin xyz="0 0 0" rpy="0 0 -1.57"/>
         <geometry>
           <xacro:get_mesh name="tooltip2" type="visual"/>
@@ -173,5 +173,5 @@
       <child link="tooltip2_link"/>
       <origin xyz="0 0 0" rpy="0 0 0"/>
-      <axis xyz="1 0 0"/>
+      <axis xyz="0 -1 0"/>
       <limit lower="-1.0" upper="0.041" effort="50" velocity="10"/>
     </joint>

File: src/Universal_Robots_ROS2_Description/urdf/ur.urdf.xacro (robot description, xacro)
@@ -139,5 +139,5 @@
    </xacro:ur_robot>
      <!-- attach gripper -->
-   <xacro:quickchanger_grippers parent="$(arg tf_prefix)wrist_3_link"/>
+   <xacro:quickchanger_grippers parent="$(arg tf_prefix)tool0"/>
    <xacro:if value="$(arg sim_gazebo)">
     <!-- Gazebo plugins -->

File: src/denso_robot_drivers_ros2/denso_robot_descriptions/robots/hsr065a1_n32/urdf/denso_robot_kinematics.xacro (robot description, xacro)
@@ -28,5 +28,5 @@
       <parent link="${parent}"/>
       <child link="${namespace}base_link"/>
-      <origin rpy="0 0 0" xyz="-0.277 0 0.084"/>
+      <origin rpy="0 0 0" xyz="0.01 0 0.084"/>
       <axis xyz="1 0 0"/>
       <limit lower="0.0" upper="0.5" effort="100" velocity="0.5" />
@@ -131,5 +131,5 @@
       <parent link="${namespace}J2"/>
       <child link="${namespace}J3"/>
-      <origin rpy="0.0 0.0 0.0" xyz="0.5 0.0 0.22"/>
+      <origin rpy="0.0 0.0 0.0" xyz="0.5 0.0 0.12"/>
       <axis xyz="0.0 0.0 1.0"/>
       <limit effort="100" lower="-10" upper="10" velocity="1.9"/>
@@ -161,5 +161,5 @@
       <parent link="${namespace}J3"/>
       <child link="${namespace}J4"/>
-      <origin rpy="0.0 0.0 1.57" xyz="0.0 0.0 -0.6047"/>
+      <origin rpy="0.0 0.0 0.0" xyz="0.0 0.0 -0.6047"/>
       <axis xyz="0.0 0.0 1.0"/>
       <limit effort="10" lower="-6.28318530717959" upper="6.28318530717959" velocity="25.2968981715147"/>

Commit message: edited ur10 to be attached to flange - denso not working properly yet

File: src/Universal_Robots_ROS2_Description/urdf/quickchanger_grippers.xacro (robot description, xacro)
@@ -8,5 +8,5 @@
     <link name="quickchanger_link">
       <visual>
-        <origin xyz="0 0 0" rpy="0 0 -1.57"/>
+        <origin xyz="0 0 0" rpy="0 0 0"/>
         <geometry>
           <xacro:get_mesh name="quickchanger" type="visual"/>
@@ -17,5 +17,5 @@
       </visual>
       <collision>
-        <origin xyz="0 0 0" rpy="0 0 -1.57"/>
+        <origin xyz="0 0 0" rpy="0 0 0"/>
         <geometry>
           <xacro:get_mesh name="quickchanger" type="collision"/>
@@ -32,10 +32,11 @@
       <parent link="${parent}"/>
       <child link="quickchanger_link"/>
-      <origin xyz="0 0 0" rpy="0 0 0"/>
+      <!-- adjust quickchanger orientation to match flange orientation -->
+      <origin xyz="0 0 0" rpy="1.57 1.57 1.57"/>
     </joint>
     <!-- suction_master_link -->
     <link name="suction_master_link">
       <visual>
-        <origin xyz="0 0 0" rpy="0 0 -1.57"/>
+        <origin xyz="0 0 0" rpy="0 0 0"/>
         <geometry>
           <xacro:get_mesh name="suction_master" type="visual"/>
@@ -46,5 +47,5 @@
       </visual>
       <collision>
-        <origin xyz="0 0 0" rpy="0 0 -1.57"/>
+        <origin xyz="0 0 0" rpy="0 0 0"/>
         <geometry>
           <xacro:get_mesh name="suction_master" type="collision"/>
@@ -66,5 +67,5 @@
     <link name="suction_link">
       <visual>
-        <origin xyz="0 0 0" rpy="0 0 -1.57"/>
+        <origin xyz="0 0 0" rpy="0 0 0"/>
         <geometry>
           <xacro:get_mesh name="suction" type="visual"/>
@@ -89,5 +90,5 @@
     <link name="gripper_link">
       <visual>
-        <origin xyz="0 0 0" rpy="0 0 -1.57"/>
+        <origin xyz="0 0 0" rpy="0 0 0"/>
         <geometry>
           <xacro:get_mesh name="gripper" type="visual"/>
@@ -118,5 +119,5 @@
     <link name="tooltip1_link">
       <visual>
-        <origin xyz="0 0 0" rpy="0 0 -1.57"/>
+        <origin xyz="0 0 0" rpy="0 0 0"/>
         <geometry>
           <xacro:get_mesh name="tooltip1" type="visual"/>
@@ -143,5 +144,5 @@
       <child link="tooltip1_link"/>
       <origin xyz="0 0 0" rpy="0 0 0"/>
-      <axis xyz="0 -1 0"/>
+      <axis xyz="1 0 0"/>
       <limit lower="-1.0" upper="0.041" effort="50" velocity="10"/>
     </joint>
@@ -149,5 +150,5 @@
     <link name="tooltip2_link">
       <visual>
-        <origin xyz="0 0 0" rpy="0 0 -1.57"/>
+        <origin xyz="0 0 0" rpy="0 0 0"/>
         <geometry>
           <xacro:get_mesh name="tooltip2" type="visual"/>
@@ -173,5 +174,5 @@
       <child link="tooltip2_link"/>
       <origin xyz="0 0 0" rpy="0 0 0"/>
-      <axis xyz="0 -1 0"/>
+      <axis xyz="1 0 0"/>
       <limit lower="-1.0" upper="0.041" effort="50" velocity="10"/>
     </joint>

File: src/Universal_Robots_ROS2_Description/urdf/ur.urdf.xacro (robot description, xacro)
@@ -139,5 +139,5 @@
    </xacro:ur_robot>
      <!-- attach gripper -->
-   <xacro:quickchanger_grippers parent="$(arg tf_prefix)tool0"/>
+   <xacro:quickchanger_grippers parent="$(arg tf_prefix)flange"/>
    <xacro:if value="$(arg sim_gazebo)">
     <!-- Gazebo plugins -->

File: src/denso_robot_drivers_ros2/denso_robot_descriptions/robots/hsr065a1_n32/urdf/denso_robot_kinematics.xacro (robot description, xacro)
@@ -131,5 +131,5 @@
       <parent link="${namespace}J2"/>
       <child link="${namespace}J3"/>
-      <origin rpy="0.0 0.0 0.0" xyz="0.5 0.0 0.12"/>
+      <origin rpy="0.0 0.0 0.0" xyz="0.5 0.0 0.0862"/>
       <axis xyz="0.0 0.0 1.0"/>
       <limit effort="100" lower="-10" upper="10" velocity="1.9"/>
@@ -138,7 +138,7 @@
     <link name="${namespace}J4">
       <visual>
-        <origin rpy="0 0 -3.14" xyz="0 0 0"/>
+        <origin rpy="0 0 0" xyz="0 0 0"/>
         <geometry>
-          <mesh filename="file://$(find denso_robot_descriptions)/robots/${model}/meshes/stl/denso_screwdriver.STL" scale="1 1 1"/>
+          <cylinder radius="0.02" length="0.04"/>
         </geometry>
         <material name="">
@@ -147,13 +147,13 @@
       </visual>
       <collision>
-        <origin rpy="0 0 -3.14" xyz="0 0 0"/>
+        <origin rpy="0 0 0" xyz="0 0 0"/>
         <geometry>
-          <mesh filename="file://$(find denso_robot_descriptions)/robots/${model}/meshes/stl/denso_screwdriver.STL" scale="1 1 1"/>
+          <cylinder radius="0.02" length="0.04"/>
         </geometry>
       </collision>
       <inertial>
-        <mass value="1.5"/>
-        <origin rpy="0.0 0.0 0.0" xyz="0.0 0.0 -0.3"/>
-        <inertia ixx="0.02" ixy="0" ixz="0" iyy="0.02" iyz="0" izz="0.01"/>
+        <mass value="0.1"/>
+        <origin rpy="0.0 0.0 0.0" xyz="0.0 0.0 0.0"/>
+        <inertia ixx="0.001" ixy="0" ixz="0" iyy="0.001" iyz="0" izz="0.001"/>
       </inertial>
     </link>
@@ -161,9 +161,36 @@
       <parent link="${namespace}J3"/>
       <child link="${namespace}J4"/>
-      <origin rpy="0.0 0.0 0.0" xyz="0.0 0.0 -0.6047"/>
+      <origin rpy="0.0 0 0" xyz="0.0 0.0 -0.5207"/>
       <axis xyz="0.0 0.0 1.0"/>
       <limit effort="10" lower="-6.28318530717959" upper="6.28318530717959" velocity="25.2968981715147"/>
       <dynamics damping="0.05" friction="0.005"/>
     </joint>
+    <!-- ROS-Industrial 'flange' frame - attachment point for EEF models -->
+    <link name="${namespace}flange">
+      <inertial>
+        <mass value="0.001"/>
+        <origin xyz="0 0 0" rpy="0 0 0"/>
+        <inertia ixx="0.001" ixy="0" ixz="0" iyy="0.001" iyz="0" izz="0.001"/>
+      </inertial>
+    </link>
+    <joint name="${namespace}J4-flange" type="fixed">
+      <parent link="${namespace}J4" />
+      <child link="${namespace}flange" />
+      <origin xyz="0 0 0" rpy="0 0 0" />
+    </joint>
+    <!-- ROS-Industrial 'tool0' frame - all-zeros tool frame -->
+    <link name="${namespace}tool0">
+      <inertial>
+        <mass value="0.001"/>
+        <origin xyz="0 0 0" rpy="0 0 0"/>
+        <inertia ixx="0.001" ixy="0" ixz="0" iyy="0.001" iyz="0" izz="0.001"/>
+      </inertial>
+    </link>
+    <joint name="${namespace}flange-tool0" type="fixed">
+      <!-- Denso toolframe - X+ front, Y+ right, Z+ up -->
+      <origin xyz="0 0 0" rpy="3.141592 0 0"/>
+      <parent link="${namespace}flange"/>
+      <child link="${namespace}tool0"/>
+    </joint>
   </xacro:macro>
 </robot>

File: src/denso_robot_drivers_ros2/denso_robot_moveit_config/robots/hsr065a1_n32/srdf/denso_robot_macro.srdf.xacro (robot description, xacro)
@@ -12,8 +12,5 @@
     <!--SUBGROUPS - Groups can also be formed by referencing to already defined group names-->
     <group name="${namespace}arm">
-		<joint name="${namespace}joint_1"/>
-		<joint name="${namespace}joint_2"/>
-		<joint name="${namespace}joint_3"/>
-		<joint name="${namespace}joint_4"/>
+		<chain base_link="${namespace}base_link" tip_link="${namespace}tool0" />
 	</group>
     <!--GROUP STATES - Purpose - Define a named state for a particular group, in terms of joint values. This is useful to define states like 'folded arms'-->
@@ -31,4 +28,8 @@
 	<disable_collisions link1="${namespace}J3" link2="${namespace}J4" reason="Adjacent"/>
 	<disable_collisions link1="${namespace}J4" link2="${namespace}base_link" reason="Never"/>
+	<disable_collisions link1="${namespace}J4" link2="${namespace}flange" reason="Adjacent"/>
+	<disable_collisions link1="${namespace}flange" link2="${namespace}tool0" reason="Adjacent"/>
+	<disable_collisions link1="${namespace}J4" link2="${namespace}tool0" reason="Never"/>
+	<disable_collisions link1="${namespace}tool0" link2="${namespace}base_link" reason="Never"/>
   </xacro:macro>
 </robot>
