Commit message: added gazebo materials - colour now showing up in gz

File: src/Universal_Robots_ROS2_Description/urdf/arf.xacro (robot description, xacro)
@@ -12,6 +12,6 @@
           <xacro:get_mesh name="arf_trolley" type="visual"/>
         </geometry>
-        <material name="">
-          <color rgba="0.89 0.91 0.93 1.0"/>
+        <material name="${sec_mesh_files['arf_trolley']['visual']['material']['name']}">
+          <color rgba="${sec_mesh_files['arf_trolley']['visual']['material']['color']}"/>
         </material>
       </visual>
@@ -41,6 +41,6 @@
           <xacro:get_mesh name="arf_base_plate" type="visual"/>
         </geometry>
-        <material name="">
-          <color rgba="0.4 0.42 0.45 1.0"/>
+        <material name="${sec_mesh_files['arf_base_plate']['visual']['material']['name']}">
+          <color rgba="${sec_mesh_files['arf_base_plate']['visual']['material']['color']}"/>
         </material>
       </visual>
@@ -70,6 +70,6 @@
           <xacro:get_mesh name="arf_slider_base" type="visual"/>
         </geometry>
-        <material name="">
-          <color rgba="0.4 0.42 0.45 1.0"/>
+        <material name="${sec_mesh_files['arf_slider_base']['visual']['material']['name']}">
+          <color rgba="${sec_mesh_files['arf_slider_base']['visual']['material']['color']}"/>
         </material>
       </visual>
@@ -99,6 +99,6 @@
           <xacro:get_mesh name="arf_slider" type="visual"/>
         </geometry>
-        <material name="">
-          <color rgba="0.33 0.42 0.18 1.0"/>
+        <material name="${sec_mesh_files['arf_slider']['visual']['material']['name']}">
+          <color rgba="${sec_mesh_files['arf_slider']['visual']['material']['color']}"/>
         </material>
       </visual>
@@ -144,6 +144,6 @@
           <xacro:get_mesh name="arf_slider_jig" type="visual"/>
         </geometry>
-        <material name="">
-          <color rgba="0.33 0.61 0.72 1.0"/>
+        <material name="${sec_mesh_files['arf_slider_jig']['visual']['material']['name']}">
+          <color rgba="${sec_mesh_files['arf_slider_jig']['visual']['material']['color']}"/>
         </material>
       </visual>
@@ -189,6 +189,6 @@
           <xacro:get_mesh name="arf_front_aircyl" type="visual"/>
         </geometry>
-        <material name="">
-          <color rgba="0.23 0.51 0.62 1.0"/>
+        <material name="${sec_mesh_files['arf_front_aircyl']['visual']['material']['name']}">
+          <color rgba="${sec_mesh_files['arf_front_aircyl']['visual']['material']['color']}"/>
         </material>
       </visual>
@@ -220,6 +220,6 @@
           <xacro:get_mesh name="arf_back_aircyl" type="visual"/>
         </geometry>
-        <material name="">
-          <color rgba="0.43 0.71 0.82 1.0"/>
+        <material name="${sec_mesh_files['arf_back_aircyl']['visual']['material']['name']}">
+          <color rgba="${sec_mesh_files['arf_back_aircyl']['visual']['material']['color']}"/>
         </material>
       </visual>

File: src/Universal_Robots_ROS2_Description/urdf/denso.xacro (robot description, xacro)
@@ -14,6 +14,6 @@
           <xacro:get_mesh name="denso_trolley" type="visual"/>
         </geometry>
-        <material name="">
-          <color rgba="0.89 0.91 0.93 1.0"/>
+        <material name="${sec_mesh_files['denso_trolley']['visual']['material']['name']}">
+          <color rgba="${sec_mesh_files['denso_trolley']['visual']['material']['color']}"/>
         </material>
       </visual>
@@ -43,6 +43,6 @@
           <xacro:get_mesh name="denso_slider_jig" type="visual"/>
         </geometry>
-        <material name="">
-          <color rgba="0.4 0.42 0.45 1.0"/>
+        <material name="${sec_mesh_files['denso_slider_jig']['visual']['material']['name']}">
+          <color rgba="${sec_mesh_files['denso_slider_jig']['visual']['material']['color']}"/>
         </material>
       </visual>

File: src/Universal_Robots_ROS2_Description/urdf/toolchanger.xacro (robot description, xacro)
@@ -12,6 +12,6 @@
           <xacro:get_mesh name="toolchanger_trolley" type="visual"/>
         </geometry>
-        <material name="">
-          <color rgba="0.89 0.91 0.93 1.0"/>
+        <material name="${sec_mesh_files['toolchanger_trolley']['visual']['material']['name']}">
+          <color rgba="${sec_mesh_files['toolchanger_trolley']['visual']['material']['color']}"/>
         </material>
       </visual>
@@ -41,6 +41,6 @@
           <xacro:get_mesh name="tool_changer" type="visual"/>
         </geometry>
-        <material name="">
-          <color rgba="0.6 0.5 0.05 1.0"/>
+        <material name="${sec_mesh_files['tool_changer']['visual']['material']['name']}">
+          <color rgba="${sec_mesh_files['tool_changer']['visual']['material']['color']}"/>
         </material>
       </visual>

File: src/Universal_Robots_ROS2_Description/urdf/ur.urdf.xacro (robot description, xacro)
@@ -15,4 +15,6 @@
    <!-- import denso macro -->
    <xacro:include filename="$(find ur_description)/urdf/denso.xacro"/>
+   <!-- import gazebo materials -->
+   <xacro:include filename="$(find ur_description)/urdf/gazebo_materials.xacro"/>
    <!-- possible 'ur_type' values: ur3, ur3e, ur5, ur5e, ur7e, ur10, ur10e, ur12e, ur16e, ur15, ur20, ur30 -->
    <!-- the default value should raise an error in case this was called without defining the type -->
@@ -146,4 +148,5 @@
       </plugin>
     </gazebo>
+    <!-- gazebo material definitions -->
   </xacro:if>
   <xacro:if value="$(arg sim_ignition)">

File: src/Universal_Robots_ROS2_Description/urdf/ur_macro.xacro (robot description, xacro)
@@ -139,6 +139,6 @@
           <xacro:get_mesh name="trolley" type="visual"/>
         </geometry>
-        <material name="">
-          <color rgba="0.89 0.91 0.93 1.0"/>
+        <material name="${sec_mesh_files['trolley']['visual']['material']['name']}">
+          <color rgba="${sec_mesh_files['trolley']['visual']['material']['color']}"/>
         </material>
       </visual>
@@ -149,4 +149,9 @@
         </geometry>
       </collision>
+      <inertial>
+        <mass value="50.0"/>
+        <origin xyz="0 0 0.4" rpy="0 0 0"/>
+        <inertia ixx="8.33" ixy="0" ixz="0" iyy="8.33" iyz="0" izz="2.08"/>
+      </inertial>
     </link>
     <!-- world to trolley 1 joint -->
@@ -163,6 +168,6 @@
           <xacro:get_mesh name="ur10_feeder" type="visual"/>
         </geometry>
-        <material name="">
-          <color rgba="0.59 0.61 0.73 1.0"/>
+        <material name="${sec_mesh_files['ur10_feeder']['visual']['material']['name']}">
+          <color rgba="${sec_mesh_files['ur10_feeder']['visual']['material']['color']}"/>
         </material>
       </visual>
@@ -173,4 +178,9 @@
         </geometry>
       </collision>
+      <inertial>
+        <mass value="25.0"/>
+        <origin xyz="0 0 0.2" rpy="0 0 0"/>
+        <inertia ixx="2.08" ixy="0" ixz="0" iyy="2.08" iyz="0" izz="0.42"/>
+      </inertial>
     </link>
     <!-- UR feeder joint -->
@@ -187,6 +197,6 @@
           <xacro:get_mesh name="heating_plate1" type="visual"/>
         </geometry>
-        <material name="">
-          <color rgba="0.85 0.86 0.92 1.0"/>
+        <material name="${sec_mesh_files['heating_plate1']['visual']['material']['name']}">
+          <color rgba="${sec_mesh_files['heating_plate1']['visual']['material']['color']}"/>
         </material>
       </visual>
@@ -197,4 +207,9 @@
         </geometry>
       </collision>
+      <inertial>
+        <mass value="5.0"/>
+        <origin xyz="0 0 0.01" rpy="0 0 0"/>
+        <inertia ixx="0.01" ixy="0" ixz="0" iyy="0.01" iyz="0" izz="0.02"/>
+      </inertial>
     </link>
     <!-- ur feeder to heating plate 1 joint -->
@@ -211,6 +226,6 @@
           <xacro:get_mesh name="heating_plate2" type="visual"/>
         </geometry>
-        <material name="">
-          <color rgba="0.85 0.86 0.92 1.0"/>
+        <material name="${sec_mesh_files['heating_plate2']['visual']['material']['name']}">
+          <color rgba="${sec_mesh_files['heating_plate2']['visual']['material']['color']}"/>
         </material>
       </visual>
@@ -221,4 +236,9 @@
         </geometry>
       </collision>
+      <inertial>
+        <mass value="5.0"/>
+        <origin xyz="0 0 0.01" rpy="0 0 0"/>
+        <inertia ixx="0.01" ixy="0" ixz="0" iyy="0.01" iyz="0" izz="0.02"/>
+      </inertial>
     </link>
     <!-- ur feeder to heating plate 2 joint -->
@@ -235,6 +255,6 @@
           <xacro:get_mesh name="heating_plate_cover1" type="visual"/>
         </geometry>
-        <material name="">
-          <color rgba="0.2 0.2 0.2 1.0"/>
+        <material name="${sec_mesh_files['heating_plate_cover1']['visual']['material']['name']}">
+          <color rgba="${sec_mesh_files['heating_plate_cover1']['visual']['material']['color']}"/>
         </material>
       </visual>
@@ -245,4 +265,9 @@
         </geometry>
       </collision>
+      <inertial>
+        <mass value="2.0"/>
+        <origin xyz="0 0 0.01" rpy="0 0 0"/>
+        <inertia ixx="0.005" ixy="0" ixz="0" iyy="0.005" iyz="0" izz="0.01"/>
+      </inertial>
     </link>
     <!-- ur feeder to heating plate cover 1 joint -->
@@ -259,6 +284,6 @@
           <xacro:get_mesh name="heating_plate_cover2" type="visual"/>
         </geometry>
-        <material name="">
-          <color rgba="0.2 0.2 0.2 1.0"/>
+        <material name="${sec_mesh_files['heating_plate_cover2']['visual']['material']['name']}">
+          <color rgba="${sec_mesh_files['heating_plate_cover2']['visual']['material']['color']}"/>
         </material>
       </visual>
@@ -269,4 +294,9 @@
         </geometry>
       </collision>
+      <inertial>
+        <mass value="2.0"/>
+        <origin xyz="0 0 0.01" rpy="0 0 0"/>
+        <inertia ixx="0.005" ixy="0" ixz="0" iyy="0.005" iyz="0" izz="0.01"/>
+      </inertial>
     </link>
     <!-- ur feeder to heating plate cover 2 joint -->
@@ -283,6 +313,6 @@
           <xacro:get_mesh name="heating_plate_cover3_1" type="visual"/>
         </geometry>
-        <material name="">
-          <color rgba="0.0 0.0 0.0 1.0"/>
+        <material name="${sec_mesh_files['heating_plate_cover3_1']['visual']['material']['name']}">
+          <color rgba="${sec_mesh_files['heating_plate_cover3_1']['visual']['material']['color']}"/>
         </material>
       </visual>
@@ -293,4 +323,9 @@
         </geometry>
       </collision>
+      <inertial>
+        <mass value="1.5"/>
+        <origin xyz="0 0 0.01" rpy="0 0 0"/>
+        <inertia ixx="0.003" ixy="0" ixz="0" iyy="0.003" iyz="0" izz="0.006"/>
+      </inertial>
     </link>
     <!-- ur feeder to heating plate cover 3-1 joint -->
@@ -307,6 +342,6 @@
           <xacro:get_mesh name="heating_plate_cover3_2" type="visual"/>
         </geometry>
-        <material name="">
-          <color rgba="0.0 0.0 0.0 1.0"/>
+        <material name="${sec_mesh_files['heating_plate_cover3_2']['visual']['material']['name']}">
+          <color rgba="${sec_mesh_files['heating_plate_cover3_2']['visual']['material']['color']}"/>
         </material>
       </visual>
@@ -317,4 +352,9 @@
         </geometry>
       </collision>
+      <inertial>
+        <mass value="1.5"/>
+        <origin xyz="0 0 0.01" rpy="0 0 0"/>
+        <inertia ixx="0.003" ixy="0" ixz="0" iyy="0.003" iyz="0" izz="0.006"/>
+      </inertial>
     </link>
     <!-- ur feeder to heating plate cover 3-2 joint -->
@@ -331,6 +371,6 @@
           <xacro:get_mesh name="plate" type="visual"/>
         </geometry>
-        <material name="">
-          <color rgba="0.69 0.71 0.83 1.0"/>
+        <material name="${sec_mesh_files['plate']['visual']['material']['name']}">
+          <color rgba="${sec_mesh_files['plate']['visual']['material']['color']}"/>
         </material>
       </visual>
@@ -341,4 +381,9 @@
         </geometry>
       </collision>
+      <inertial>
+        <mass value="15.0"/>
+        <origin xyz="0 0 0.05" rpy="0 0 0"/>
+        <inertia ixx="0.125" ixy="0" ixz="0" iyy="0.125" iyz="0" izz="0.25"/>
+      </inertial>
     </link>
     <!-- trolley1 to UR plate joint -->
@@ -349,5 +394,11 @@
     </joint>
     <!-- ur robot base link -->
-    <link name="${tf_prefix}base_link"/>
+    <link name="${tf_prefix}base_link">
+      <inertial>
+        <mass value="0.001"/>
+        <origin xyz="0 0 0" rpy="0 0 0"/>
+        <inertia ixx="0.001" ixy="0" ixz="0" iyy="0.001" iyz="0" izz="0.001"/>
+      </inertial>
+    </link>
     <!-- plate to base joint -->
     <joint name="${tf_prefix}base_joint" type="fixed">
@@ -644,5 +695,11 @@
     </joint>
     <!-- ft_frame link -->
-    <link name="${tf_prefix}ft_frame"/>
+    <link name="${tf_prefix}ft_frame">
+      <inertial>
+        <mass value="0.001"/>
+        <origin xyz="0 0 0" rpy="0 0 0"/>
+        <inertia ixx="0.001" ixy="0" ixz="0" iyy="0.001" iyz="0" izz="0.001"/>
+      </inertial>
+    </link>
     <!-- wrist_3_link to ft_frame joint -->
     <joint name="${tf_prefix}wrist_3_link-ft_frame" type="fixed">
@@ -652,5 +709,11 @@
     </joint>
     <!-- ROS-Industrial 'base' frame - base_link to UR 'Base' Coordinates transform -->
-    <link name="${tf_prefix}base"/>
+    <link name="${tf_prefix}base">
+      <inertial>
+        <mass value="0.001"/>
+        <origin xyz="0 0 0" rpy="0 0 0"/>
+        <inertia ixx="0.001" ixy="0" ixz="0" iyy="0.001" iyz="0" izz="0.001"/>
+      </inertial>
+    </link>
     <joint name="${tf_prefix}base_link-base_fixed_joint" type="fixed">
       <!-- Note the rotation over Z of pi radians - as base_link is REP-103
@@ -664,5 +727,11 @@
     </joint>
     <!-- ROS-Industrial 'flange' frame - attachment point for EEF models -->
-    <link name="${tf_prefix}flange" />
+    <link name="${tf_prefix}flange">
+      <inertial>
+        <mass value="0.001"/>
+        <origin xyz="0 0 0" rpy="0 0 0"/>
+        <inertia ixx="0.001" ixy="0" ixz="0" iyy="0.001" iyz="0" izz="0.001"/>
+      </inertial>
+    </link>
     <joint name="${tf_prefix}wrist_3-flange" type="fixed">
       <parent link="${tf_prefix}wrist_3_link" />
@@ -671,5 +740,11 @@
     </joint>
     <!-- ROS-Industrial 'tool0' frame - all-zeros tool frame -->
-    <link name="${tf_prefix}tool0"/>
+    <link name="${tf_prefix}tool0">
+      <inertial>
+        <mass value="0.001"/>
+        <origin xyz="0 0 0" rpy="0 0 0"/>
+        <inertia ixx="0.001" ixy="0" ixz="0" iyy="0.001" iyz="0" izz="0.001"/>
+      </inertial>
+    </link>
     <joint name="${tf_prefix}flange-tool0" type="fixed">
       <!-- default toolframe - X+ left, Y+ up, Z+ front -->

File: src/Universal_Robots_ROS2_Description/urdf/vision.xacro (robot description, xacro)
@@ -5,5 +5,5 @@
     <xacro:property name="sec_mesh_files" value="${vision_visual_params['mesh_files']}" scope="parent"/>
     <xacro:property name="force_abs_paths" value="true" scope="parent"/>
-<!-- vision trolley link -->
+    <!-- vision trolley link -->
     <link name="vision_trolley_link">
       <visual>
@@ -12,6 +12,6 @@
           <xacro:get_mesh name="vision_trolley" type="visual"/>
         </geometry>
-        <material name="">
-          <color rgba="0.89 0.91 0.93 1.0"/>
+        <material name="${sec_mesh_files['vision_trolley']['visual']['material']['name']}">
+          <color rgba="${sec_mesh_files['vision_trolley']['visual']['material']['color']}"/>
         </material>
       </visual>
@@ -41,6 +41,6 @@
           <xacro:get_mesh name="vision_cam_jig" type="visual"/>
         </geometry>
-        <material name="">
-          <color rgba="0.5 0.4 0.55 1.0"/>
+        <material name="${sec_mesh_files['vision_cam_jig']['visual']['material']['name']}">
+          <color rgba="${sec_mesh_files['vision_cam_jig']['visual']['material']['color']}"/>
         </material>
       </visual>
@@ -68,8 +68,8 @@
         <origin xyz="0 0 0" rpy="0 0 0"/>
         <geometry>
-          <xacro:get_mesh name="vision_feeder" type="collision"/>
+          <xacro:get_mesh name="vision_feeder" type="visual"/>
         </geometry>
-        <material name="">
-          <color rgba="0.7 0.51 0.56 1.0"/>
+        <material name="${sec_mesh_files['vision_feeder']['visual']['material']['name']}">
+          <color rgba="${sec_mesh_files['vision_feeder']['visual']['material']['color']}"/>
         </material>
       </visual>
