Commit message: controllers working except tooltips

File: src/Universal_Robots_ROS2_Description/urdf/arf.xacro (robot description, xacro)
@@ -116,5 +116,5 @@
     </link>
     <!-- ** arf_axis_1_joint ** arf slider base to slider joint -->
-    <joint name="arf_axis_1_joint" type="fixed">
+    <joint name="arf_axis_1_joint" type="prismatic">
       <parent link="arf_slider_base_link" />
       <child link="arf_slider_link" />
@@ -161,5 +161,5 @@
     </link>
     <!-- ** arf_axis_2_joint **arf slider dummy to slider jig joint -->
-    <joint name="arf_axis_2_joint" type="fixed">
+    <joint name="arf_axis_2_joint" type="prismatic">
       <parent link="arf_slider_dummy_link" />
       <child link="arf_slider_jig_link" />
@@ -206,5 +206,5 @@
     </link>
     <!-- arf slider jig to front aircyl joint ****** PRISMATIC ****** -->
-    <joint name="arf_gripper_joint_1" type="fixed">
+    <joint name="arf_gripper_joint_1" type="prismatic">
       <parent link="arf_aircyl_dummy_link" />
       <child link="arf_front_aircyl_link" />
@@ -237,5 +237,5 @@
     </link>
     <!-- arf slider jig to front aircyl joint ****** PRISMATIC ****** -->
-    <joint name="arf_gripper_joint_2" type="fixed">
+    <joint name="arf_gripper_joint_2" type="prismatic">
       <parent link="arf_aircyl_dummy_link" />
       <child link="arf_back_aircyl_link" />

File: src/Universal_Robots_ROS2_Description/urdf/inc/ur_transmissions.xacro (robot description, xacro)
@@ -61,4 +61,71 @@
       </actuator>
     </transmission>
+    <!-- UR Robot Gripper Tooltips -->
+    <transmission name="tooltip1_trans">
+      <type>transmission_interface/SimpleTransmission</type>
+      <joint name="tooltip1_joint">
+        <hardwareInterface>${hw_interface}</hardwareInterface>
+      </joint>
+      <actuator name="tooltip1_motor">
+        <mechanicalReduction>1</mechanicalReduction>
+      </actuator>
+    </transmission>
+    <transmission name="tooltip2_trans">
+      <type>transmission_interface/SimpleTransmission</type>
+      <joint name="tooltip2_joint">
+        <hardwareInterface>${hw_interface}</hardwareInterface>
+      </joint>
+      <actuator name="tooltip2_motor">
+        <mechanicalReduction>1</mechanicalReduction>
+      </actuator>
+    </transmission>
+    <!-- ARF Axis Joints -->
+    <transmission name="arf_axis_1_trans">
+      <type>transmission_interface/SimpleTransmission</type>
+      <joint name="arf_axis_1_joint">
+        <hardwareInterface>${hw_interface}</hardwareInterface>
+      </joint>
+      <actuator name="arf_axis_1_motor">
+        <mechanicalReduction>1</mechanicalReduction>
+      </actuator>
+    </transmission>
+    <transmission name="arf_axis_2_trans">
+      <type>transmission_interface/SimpleTransmission</type>
+      <joint name="arf_axis_2_joint">
+        <hardwareInterface>${hw_interface}</hardwareInterface>
+      </joint>
+      <actuator name="arf_axis_2_motor">
+        <mechanicalReduction>1</mechanicalReduction>
+      </actuator>
+    </transmission>
+    <!-- ARF Gripper Joints -->
+    <transmission name="arf_gripper1_trans">
+      <type>transmission_interface/SimpleTransmission</type>
+      <joint name="arf_gripper_joint_1">
+        <hardwareInterface>${hw_interface}</hardwareInterface>
+      </joint>
+      <actuator name="arf_gripper_motor_1">
+        <mechanicalReduction>1</mechanicalReduction>
+      </actuator>
+    </transmission>
+    <transmission name="arf_gripper2_trans">
+      <type>transmission_interface/SimpleTransmission</type>
+      <joint name="arf_gripper_joint_2">
+        <hardwareInterface>${hw_interface}</hardwareInterface>
+      </joint>
+      <actuator name="arf_gripper_motor_2">
+        <mechanicalReduction>1</mechanicalReduction>
+      </actuator>
+    </transmission>
+    <!-- Denso Axis Joint -->
+    <transmission name="denso_axis_trans">
+      <type>transmission_interface/SimpleTransmission</type>
+      <joint name="denso_axis_joint">
+        <hardwareInterface>${hw_interface}</hardwareInterface>
+      </joint>
+      <actuator name="denso_axis_motor">
+        <mechanicalReduction>1</mechanicalReduction>
+      </actuator>
+    </transmission>
   </xacro:macro>
 </robot>

File: src/Universal_Robots_ROS2_Description/urdf/quickchanger_gripper_suction.xacro (robot description, xacro)
@@ -15,6 +15,6 @@
           <xacro:get_mesh name="quickchanger" type="visual"/>
         </geometry>
-        <material name="Grey">
-          <color rgba="0.6 0.6 0.6 1.0"/>
+        <material name="${sec_mesh_files['quickchanger']['visual']['material']['name']}">
+          <color rgba="${sec_mesh_files['quickchanger']['visual']['material']['color']}"/>
         </material>
       </visual>
@@ -41,6 +41,6 @@
           <xacro:get_mesh name="suction_master" type="visual"/>
         </geometry>
-        <material name="DarkGrey">
-          <color rgba="0.3 0.3 0.3 1.0"/>
+        <material name="${sec_mesh_files['suction_master']['visual']['material']['name']}">
+          <color rgba="${sec_mesh_files['suction_master']['visual']['material']['color']}"/>
         </material>
       </visual>
@@ -67,6 +67,6 @@
           <xacro:get_mesh name="suction" type="visual"/>
         </geometry>
-        <material name="DarkGray">
-          <color rgba="0.3 0.3 0.3 1.0"/>
+        <material name="${sec_mesh_files['suction']['visual']['material']['name']}">
+          <color rgba="${sec_mesh_files['suction']['visual']['material']['color']}"/>
         </material>
       </visual>
@@ -93,6 +93,6 @@
           <xacro:get_mesh name="gripper" type="visual"/>
         </geometry>
-        <material name="Black">
-          <color rgba="0.1 0.1 0.1 1.0"/>
+        <material name="${sec_mesh_files['gripper']['visual']['material']['name']}">
+          <color rgba="${sec_mesh_files['gripper']['visual']['material']['color']}"/>
         </material>
       </visual>
@@ -122,6 +122,6 @@
           <xacro:get_mesh name="tooltip1" type="visual"/>
         </geometry>
-        <material name="Silver">
-          <color rgba="0.8 0.8 0.8 1.0"/>
+        <material name="${sec_mesh_files['tooltip1']['visual']['material']['name']}">
+          <color rgba="${sec_mesh_files['tooltip1']['visual']['material']['color']}"/>
         </material>
       </visual>
@@ -134,5 +134,5 @@
     </link>
     <!-- tooltip1_joint -->
-    <joint name="tooltip1_joint" type="fixed">
+    <joint name="tooltip1_joint" type="prismatic">
       <parent link="gripper_link"/>
       <child link="tooltip1_link"/>
@@ -140,4 +140,5 @@
       <axis xyz="1 0 0"/>
       <limit lower="-1.0" upper="0.041" effort="50" velocity="10"/>
+      <dynamics damping="0.1" friction="0.1"/>
     </joint>
     <!-- tooltip2 -->
@@ -153,6 +154,6 @@
           <xacro:get_mesh name="tooltip2" type="visual"/>
         </geometry>
-        <material name="Silver">
-          <color rgba="0.8 0.8 0.8 1.0"/>
+        <material name="${sec_mesh_files['tooltip2']['visual']['material']['name']}">
+          <color rgba="${sec_mesh_files['tooltip2']['visual']['material']['color']}"/>
         </material>
       </visual>
@@ -164,5 +165,5 @@
       </collision>
     </link>
-    <joint name="tooltip2_joint" type="fixed">
+    <joint name="tooltip2_joint" type="prismatic">
       <parent link="gripper_link"/>
       <child link="tooltip2_link"/>
@@ -170,4 +171,5 @@
       <axis xyz="1 0 0"/>
       <limit lower="-1.0" upper="0.041" effort="50" velocity="10"/>
+      <dynamics damping="0.1" friction="0.1"/>
     </joint>
   </xacro:macro>

File: src/Universal_Robots_ROS2_Description/urdf/ur.ros2_control.xacro (robot description, xacro)
@@ -121,4 +121,119 @@
           <!-- initial position for the FakeSystem and simulation -->
           <param name="initial_value">${initial_positions['wrist_3_joint']}</param>
+        </state_interface>
+        <state_interface name="velocity"/>
+        <state_interface name="effort"/>
+      </joint>
+      <!-- UR Robot Gripper Tooltips -->
+      <joint name="${tf_prefix}tooltip1_joint">
+        <command_interface name="position"/>
+        <command_interface name="velocity"/>
+        <state_interface name="position">
+          <!-- initial position for the FakeSystem and simulation -->
+          <param name="initial_value">${initial_positions['tooltip1_joint']}</param>
+        </state_interface>
+        <state_interface name="velocity"/>
+        <state_interface name="effort"/>
+      </joint>
+      <joint name="${tf_prefix}tooltip2_joint">
+        <command_interface name="position"/>
+        <command_interface name="velocity"/>
+        <state_interface name="position">
+          <!-- initial position for the FakeSystem and simulation -->
+          <param name="initial_value">${initial_positions['tooltip2_joint']}</param>
+        </state_interface>
+        <state_interface name="velocity"/>
+        <state_interface name="effort"/>
+      </joint>
+      <!-- ARF Axis Joints -->
+      <joint name="${tf_prefix}arf_axis_1_joint">
+        <command_interface name="position"/>
+        <command_interface name="velocity"/>
+        <state_interface name="position">
+          <!-- initial position for the FakeSystem and simulation -->
+          <param name="initial_value">${initial_positions['arf_axis_1_joint']}</param>
+        </state_interface>
+        <state_interface name="velocity"/>
+        <state_interface name="effort"/>
+      </joint>
+      <joint name="${tf_prefix}arf_axis_2_joint">
+        <command_interface name="position"/>
+        <command_interface name="velocity"/>
+        <state_interface name="position">
+          <!-- initial position for the FakeSystem and simulation -->
+          <param name="initial_value">${initial_positions['arf_axis_2_joint']}</param>
+        </state_interface>
+        <state_interface name="velocity"/>
+        <state_interface name="effort"/>
+      </joint>
+      <!-- ARF Gripper Joints -->
+      <joint name="arf_gripper_joint_1">
+        <command_interface name="position"/>
+        <command_interface name="velocity"/>
+        <state_interface name="position">
+          <!-- initial position for the FakeSystem and simulation -->
+          <param name="initial_value">${initial_positions['arf_gripper_joint_1']}</param>
+        </state_interface>
+        <state_interface name="velocity"/>
+        <state_interface name="effort"/>
+      </joint>
+      <joint name="arf_gripper_joint_2">
+        <command_interface name="position"/>
+        <command_interface name="velocity"/>
+        <state_interface name="position">
+          <!-- initial position for the FakeSystem and simulation -->
+          <param name="initial_value">${initial_positions['arf_gripper_joint_2']}</param>
+        </state_interface>
+        <state_interface name="velocity"/>
+        <state_interface name="effort"/>
+      </joint>
+      <!-- Denso Robot Joints -->
+      <joint name="denso_joint_1">
+        <command_interface name="position"/>
+        <command_interface name="velocity"/>
+        <state_interface name="position">
+          <!-- initial position for the FakeSystem and simulation -->
+          <param name="initial_value">${initial_positions['denso_joint_1']}</param>
+        </state_interface>
+        <state_interface name="velocity"/>
+        <state_interface name="effort"/>
+      </joint>
+      <joint name="denso_joint_2">
+        <command_interface name="position"/>
+        <command_interface name="velocity"/>
+        <state_interface name="position">
+          <!-- initial position for the FakeSystem and simulation -->
+          <param name="initial_value">${initial_positions['denso_joint_2']}</param>
+        </state_interface>
+        <state_interface name="velocity"/>
+        <state_interface name="effort"/>
+      </joint>
+      <joint name="denso_joint_3">
+        <command_interface name="position"/>
+        <command_interface name="velocity"/>
+        <state_interface name="position">
+          <!-- initial position for the FakeSystem and simulation -->
+          <param name="initial_value">${initial_positions['denso_joint_3']}</param>
+        </state_interface>
+        <state_interface name="velocity"/>
+        <state_interface name="effort"/>
+      </joint>
+      <joint name="denso_joint_4">
+        <command_interface name="position"/>
+        <command_interface name="velocity"/>
+        <state_interface name="position">
+          <!-- initial position for the FakeSystem and simulation -->
+          <param name="initial_value">${initial_positions['denso_joint_4']}</param>
+        </state_interface>
+        <state_interface name="velocity"/>
+        <state_interface name="effort"/>
+      </joint>
+      <!-- Denso Axis Joint -->
+      <joint name="denso_axis_joint">
+        <command_interface name="position"/>
+        <command_interface name="velocity"/>
+        <state_interface name="position">
+          <!-- initial position for the FakeSystem and simulation -->
+          <param name="initial_value">${initial_positions['denso_axis_joint']}</param>
         </state_interface>
         <state_interface name="velocity"/>

File: src/Universal_Robots_ROS2_Description/urdf/ur.urdf.xacro (robot description, xacro)
@@ -102,4 +102,5 @@
      tf_prefix="$(arg tf_prefix)"
      parent="world"
+     prefix=""
      joint_limits_parameters_file="$(arg joint_limit_params)"
      kinematics_parameters_file="$(arg kinematics_params)"
@@ -148,5 +149,4 @@
       </plugin>
     </gazebo>
-    <!-- gazebo material definitions -->
   </xacro:if>
   <xacro:if value="$(arg sim_ignition)">

File: src/Universal_Robots_ROS2_Description/urdf/ur_macro.xacro (robot description, xacro)
@@ -47,4 +47,5 @@
     name
     tf_prefix
+    prefix
     parent
     *origin
@@ -129,5 +130,5 @@
     </xacro:if>
     <!-- Add URDF transmission elements (for ros_control) -->
-    <!--<xacro:ur_arm_transmission prefix="${prefix}" hw_interface="${transmission_hw_interface}" />-->
+    <xacro:ur_arm_transmission prefix="${prefix}" hw_interface="${transmission_hw_interface}" />
     <!-- Placeholder for ros2_control transmission which don't yet exist -->
     <!-- links and joints - main serial chain -->

File: src/denso_robot_drivers_ros2/denso_robot_descriptions/robots/hsr065a1_n32/urdf/denso_robot_kinematics.xacro (robot description, xacro)
@@ -25,5 +25,5 @@
       </inertial>
     </link>
-    <joint name="${namespace}axis_joint" type="fixed">
+    <joint name="${namespace}axis_joint" type="prismatic">
       <parent link="${parent}"/>
       <child link="${namespace}base_link"/>

Commit message: edited arf spawn position by 1mm for 151mm positioning, light pink colour for heating_plate_covoer_1 for visualisation purpose

File: src/Universal_Robots_ROS2_Description/urdf/arf.xacro (robot description, xacro)
@@ -119,5 +119,5 @@
       <parent link="arf_slider_base_link" />
       <child link="arf_slider_link" />
-      <origin xyz="-0.1068 0 0.04" rpy="0 0 0"/>
+      <origin xyz="-0.1078 0 0.04" rpy="0 0 0"/>
       <axis xyz="1 0 0"/>
       <limit lower="-0.35" upper="0" effort="100" velocity="10" />

Commit message: edited arf spawn position

File: src/Universal_Robots_ROS2_Description/urdf/arf.xacro (robot description, xacro)
@@ -119,5 +119,5 @@
       <parent link="arf_slider_base_link" />
       <child link="arf_slider_link" />
-      <origin xyz="-0.1078 0 0.04" rpy="0 0 0"/>
+      <origin xyz="-0.2588 0 0.04" rpy="0 0 0"/>
       <axis xyz="1 0 0"/>
       <limit lower="-0.35" upper="0" effort="100" velocity="10" />

Commit message: spawn arf at 000 + cleaned up world

File: src/Universal_Robots_ROS2_Description/urdf/arf.xacro (robot description, xacro)
@@ -119,5 +119,5 @@
       <parent link="arf_slider_base_link" />
       <child link="arf_slider_link" />
-      <origin xyz="-0.2588 0 0.04" rpy="0 0 0"/>
+      <origin xyz="-0.1068 0 0.04" rpy="0 0 0"/>
       <axis xyz="1 0 0"/>
       <limit lower="-0.35" upper="0" effort="100" velocity="10" />

File: src/Universal_Robots_ROS2_Description/urdf/ur_macro.xacro (robot description, xacro)
@@ -218,5 +218,5 @@
       <parent link="${tf_prefix}ur10_trolley_link" />
       <child link="${tf_prefix}ur10_plate_link" />
-      <origin xyz="0 0 0.850" rpy="0 0 0"/>
+      <origin xyz="0 0 0.835" rpy="0 0 0"/>
     </joint>
     <!-- ur robot base link -->

Commit message: spawning arf at 150 0

File: src/Universal_Robots_ROS2_Description/urdf/arf.xacro (robot description, xacro)
@@ -119,5 +119,5 @@
       <parent link="arf_slider_base_link" />
       <child link="arf_slider_link" />
-      <origin xyz="-0.1068 0 0.04" rpy="0 0 0"/>
+      <origin xyz="-0.2578 0 0.04" rpy="0 0 0"/>
       <axis xyz="1 0 0"/>
       <limit lower="-0.35" upper="0" effort="100" velocity="10" />

File: src/Universal_Robots_ROS2_Description/urdf/ur_macro.xacro (robot description, xacro)
@@ -218,5 +218,5 @@
       <parent link="${tf_prefix}ur10_trolley_link" />
       <child link="${tf_prefix}ur10_plate_link" />
-      <origin xyz="0 -0.05 0.835" rpy="0 0 0"/>
+      <origin xyz="0 0 0.835" rpy="0 0 0"/>
     </joint>
     <!-- ur robot base link -->

Commit message: fixed arf axis direction and limit - working version

File: src/Universal_Robots_ROS2_Description/urdf/arf.xacro (robot description, xacro)
@@ -119,7 +119,7 @@
       <parent link="arf_slider_base_link" />
       <child link="arf_slider_link" />
-      <origin xyz="-0.2578 0 0.04" rpy="0 0 0"/>
-      <axis xyz="1 0 0"/>
-      <limit lower="-0.35" upper="0" effort="100" velocity="10" />
+      <origin xyz="-0.1068 0 0.04" rpy="0 0 0"/>
+      <axis xyz="-1 0 0"/>
+      <limit lower="0.0" upper="0.35" effort="100" velocity="10" />
     </joint>
   <!-- dummy link for slider and jig joints -->

Commit message: adjusted arf axis 1 spawn position so that cover plates can be placed in the middle

File: src/Universal_Robots_ROS2_Description/urdf/arf.xacro (robot description, xacro)
@@ -119,5 +119,5 @@
       <parent link="arf_slider_base_link" />
       <child link="arf_slider_link" />
-      <origin xyz="-0.1068 0 0.04" rpy="0 0 0"/>
+      <origin xyz="-0.12 0 0.04" rpy="0 0 0"/>
       <axis xyz="-1 0 0"/>
       <limit lower="0.0" upper="0.35" effort="100" velocity="10" />
