Commit message: added files - fortress version

File: src/Universal_Robots_ROS2_Description/urdf/inc/ur_transmissions.xacro (robot description, xacro)
@@ -61,4 +61,71 @@
       </actuator>
     </transmission>
+<!-- UR Robot Gripper Tooltips -->
+<transmission name="tooltip1_trans">
+  <type>transmission_interface/SimpleTransmission</type>
+  <joint name="tooltip1_joint">
+    <hardwareInterface>${hw_interface}</hardwareInterface>
+  </joint>
+  <actuator name="tooltip1_motor">
+    <mechanicalReduction>1</mechanicalReduction>
+  </actuator>
+</transmission>
+<transmission name="tooltip2_trans">
+  <type>transmission_interface/SimpleTransmission</type>
+  <joint name="tooltip2_joint">
+    <hardwareInterface>${hw_interface}</hardwareInterface>
+  </joint>
+  <actuator name="tooltip2_motor">
+    <mechanicalReduction>1</mechanicalReduction>
+  </actuator>
+</transmission>
+<!-- ARF Axis Joints -->
+<transmission name="arf_axis_1_trans">
+  <type>transmission_interface/SimpleTransmission</type>
+  <joint name="arf_axis_1_joint">
+    <hardwareInterface>${hw_interface}</hardwareInterface>
+  </joint>
+  <actuator name="arf_axis_1_motor">
+    <mechanicalReduction>1</mechanicalReduction>
+  </actuator>
+</transmission>
+<transmission name="arf_axis_2_trans">
+  <type>transmission_interface/SimpleTransmission</type>
+  <joint name="arf_axis_2_joint">
+    <hardwareInterface>${hw_interface}</hardwareInterface>
+  </joint>
+  <actuator name="arf_axis_2_motor">
+    <mechanicalReduction>1</mechanicalReduction>
+  </actuator>
+</transmission>
+<!-- ARF Gripper Joints -->
+<transmission name="arf_gripper1_trans">
+  <type>transmission_interface/SimpleTransmission</type>
+  <joint name="arf_gripper_joint_1">
+    <hardwareInterface>${hw_interface}</hardwareInterface>
+  </joint>
+  <actuator name="arf_gripper_motor_1">
+    <mechanicalReduction>1</mechanicalReduction>
+  </actuator>
+</transmission>
+<transmission name="arf_gripper2_trans">
+  <type>transmission_interface/SimpleTransmission</type>
+  <joint name="arf_gripper_joint_2">
+    <hardwareInterface>${hw_interface}</hardwareInterface>
+  </joint>
+  <actuator name="arf_gripper_motor_2">
+    <mechanicalReduction>1</mechanicalReduction>
+  </actuator>
+</transmission>
+<!-- Denso Axis Joint -->
+<transmission name="denso_axis_trans">
+  <type>transmission_interface/SimpleTransmission</type>
+  <joint name="denso_axis_joint">
+    <hardwareInterface>${hw_interface}</hardwareInterface>
+  </joint>
+  <actuator name="denso_axis_motor">
+    <mechanicalReduction>1</mechanicalReduction>
+  </actuator>
+</transmission>
   </xacro:macro>
 </robot>

File: src/Universal_Robots_ROS2_Description/urdf/ur.ros2_control.xacro (robot description, xacro)
@@ -7,5 +7,5 @@
     sim_ignition:=false
     headless_mode:=false
-    initial_positions:=${dict(shoulder_pan_joint=0.0,shoulder_lift_joint=-1.57,elbow_joint=0.0,wrist_1_joint=-1.57,wrist_2_joint=0.0,wrist_3_joint=0.0)}
+    initial_positions:=${dict(shoulder_pan_joint=0.0,shoulder_lift_joint=-1.57,elbow_joint=0.0,wrist_1_joint=-1.57,wrist_2_joint=0.0,wrist_3_joint=0.0,tooltip1_joint=0.0,tooltip2_joint=0.0,arf_axis_1_joint=0.0,arf_axis_2_joint=0.0)}
     use_tool_communication:=false
     script_filename output_recipe_filename
@@ -65,4 +65,5 @@
         </xacro:unless>
       </hardware>
+      <!-- UR Robot Joints -->
       <joint name="${tf_prefix}shoulder_pan_joint">
         <command_interface name="position"/>
@@ -121,4 +122,117 @@
           <!-- initial position for the FakeSystem and simulation -->
           <param name="initial_value">${initial_positions['wrist_3_joint']}</param>
+        </state_interface>
+        <state_interface name="velocity"/>
+        <state_interface name="effort"/>
+      </joint>
+      <!-- UR Robot Gripper Tooltips -->
+      <joint name="${tf_prefix}tooltip1_joint">
+        <command_interface name="position"/>
+        <state_interface name="position">
+          <!-- initial position for the FakeSystem and simulation -->
+          <param name="initial_value">${initial_positions['tooltip1_joint']}</param>
+        </state_interface>
+        <state_interface name="velocity"/>
+        <state_interface name="effort"/>
+      </joint>
+      <joint name="${tf_prefix}tooltip2_joint">
+        <command_interface name="position"/>
+        <state_interface name="position">
+          <!-- initial position for the FakeSystem and simulation -->
+          <param name="initial_value">${initial_positions['tooltip2_joint']}</param>
+        </state_interface>
+        <state_interface name="velocity"/>
+        <state_interface name="effort"/>
+      </joint>
+      <!-- ARF Axis Joints -->
+      <joint name="${tf_prefix}arf_axis_1_joint">
+        <command_interface name="position"/>
+        <command_interface name="velocity"/>
+        <state_interface name="position">
+          <!-- initial position for the FakeSystem and simulation -->
+          <param name="initial_value">${initial_positions['arf_axis_1_joint']}</param>
+        </state_interface>
+        <state_interface name="velocity"/>
+        <state_interface name="effort"/>
+      </joint>
+      <joint name="${tf_prefix}arf_axis_2_joint">
+        <command_interface name="position"/>
+        <command_interface name="velocity"/>
+        <state_interface name="position">
+          <!-- initial position for the FakeSystem and simulation -->
+          <param name="initial_value">${initial_positions['arf_axis_2_joint']}</param>
+        </state_interface>
+        <state_interface name="velocity"/>
+        <state_interface name="effort"/>
+      </joint>
+      <!-- ARF Gripper Joints -->
+      <joint name="arf_gripper_joint_1">
+        <command_interface name="position"/>
+        <command_interface name="velocity"/>
+        <state_interface name="position">
+          <!-- initial position for the FakeSystem and simulation -->
+          <param name="initial_value">${initial_positions['arf_gripper_joint_1']}</param>
+        </state_interface>
+        <state_interface name="velocity"/>
+        <state_interface name="effort"/>
+      </joint>
+      <joint name="arf_gripper_joint_2">
+        <command_interface name="position"/>
+        <command_interface name="velocity"/>
+        <state_interface name="position">
+          <!-- initial position for the FakeSystem and simulation -->
+          <param name="initial_value">${initial_positions['arf_gripper_joint_2']}</param>
+        </state_interface>
+        <state_interface name="velocity"/>
+        <state_interface name="effort"/>
+      </joint>
+      <!-- Denso Robot Joints -->
+      <joint name="denso_joint_1">
+        <command_interface name="position"/>
+        <command_interface name="velocity"/>
+        <state_interface name="position">
+          <!-- initial position for the FakeSystem and simulation -->
+          <param name="initial_value">${initial_positions['denso_joint_1']}</param>
+        </state_interface>
+        <state_interface name="velocity"/>
+        <state_interface name="effort"/>
+      </joint>
+      <joint name="denso_joint_2">
+        <command_interface name="position"/>
+        <command_interface name="velocity"/>
+        <state_interface name="position">
+          <!-- initial position for the FakeSystem and simulation -->
+          <param name="initial_value">${initial_positions['denso_joint_2']}</param>
+        </state_interface>
+        <state_interface name="velocity"/>
+        <state_interface name="effort"/>
+      </joint>
+      <joint name="denso_joint_3">
+        <command_interface name="position"/>
+        <command_interface name="velocity"/>
+        <state_interface name="position">
+          <!-- initial position for the FakeSystem and simulation -->
+          <param name="initial_value">${initial_positions['denso_joint_3']}</param>
+        </state_interface>
+        <state_interface name="velocity"/>
+        <state_interface name="effort"/>
+      </joint>
+      <joint name="denso_joint_4">
+        <command_interface name="position"/>
+        <command_interface name="velocity"/>
+        <state_interface name="position">
+          <!-- initial position for the FakeSystem and simulation -->
+          <param name="initial_value">${initial_positions['denso_joint_4']}</param>
+        </state_interface>
+        <state_interface name="velocity"/>
+        <state_interface name="effort"/>
+      </joint>
+      <!-- Denso Axis Joint -->
+      <joint name="denso_axis_joint">
+        <command_interface name="position"/>
+        <command_interface name="velocity"/>
+        <state_interface name="position">
+          <!-- initial position for the FakeSystem and simulation -->
+          <param name="initial_value">${initial_positions['denso_axis_joint']}</param>
         </state_interface>
         <state_interface name="velocity"/>

File: src/Universal_Robots_ROS2_Description/urdf/ur.urdf.xacro (robot description, xacro)
@@ -3,6 +3,16 @@
    <!-- robot name parameter -->
    <xacro:arg name="name" default="ur"/>
-   <!-- import main macro -->
-   <xacro:include filename="$(find ur_description)/urdf/ur_macro.xacro"/>
+   <!-- import main ur10 + trolley macro -->
+   <xacro:include filename="$(find ur_description)/urdf/ur10.xacro"/>
+   <!-- import quickchanger + gripper + suction macro -->
+   <xacro:include filename="$(find ur_description)/urdf/quickchanger_gripper_suction.xacro"/>
+   <!-- import arf + trolley macro -->
+   <xacro:include filename="$(find ur_description)/urdf/arf.xacro"/>
+   <!-- import vision + trolley macro -->
+   <xacro:include filename="$(find ur_description)/urdf/vision.xacro"/>
+   <!-- import toolchanger + trolley macro -->
+   <xacro:include filename="$(find ur_description)/urdf/toolchanger.xacro"/>
+   <!-- import denso + trolley macro -->
+   <xacro:include filename="$(find ur_description)/urdf/denso.xacro"/>
    <!-- possible 'ur_type' values: ur3, ur3e, ur5, ur5e, ur7e, ur10, ur10e, ur12e, ur16e, ur15, ur20, ur30 -->
    <!-- the default value should raise an error in case this was called without defining the type -->
@@ -77,4 +87,12 @@
      </joint>
    </xacro:if>
+      <!-- vision components -->
+   <xacro:vision parent="world"/>
+   <!-- ARF components -->
+   <xacro:arf parent="world"/>
+   <!-- toolchanger components -->
+   <xacro:toolchanger parent="world"/>
+   <!-- denso components -->
+   <xacro:denso parent="world"/>
    <!-- arm -->
    <xacro:ur_robot
@@ -82,4 +100,5 @@
      tf_prefix="$(arg tf_prefix)"
      parent="world"
+     prefix=""
      joint_limits_parameters_file="$(arg joint_limit_params)"
      kinematics_parameters_file="$(arg kinematics_params)"
@@ -117,4 +136,6 @@
      <origin xyz="0 0 0" rpy="0 0 0" />          <!-- position robot in the world -->
    </xacro:ur_robot>
+  <!-- attach gripper -->
+   <xacro:quickchanger_gripper_suction parent="$(arg tf_prefix)wrist_3_link"/>
    <xacro:if value="$(arg sim_gazebo)">
     <!-- Gazebo plugins -->

File: src/Universal_Robots_ROS2_Driver/ur_moveit_config/srdf/ur_macro.srdf.xacro (robot description, xacro)
@@ -11,15 +11,39 @@
     <!--CHAINS - When a chain is specified, all the links along the chain (including endpoints) are included in the group. Additionally, all the joints that are parents to included links are also included. This means that joints along the chain and the parent joint of the base link are included in the group-->
     <!--SUBGROUPS - Groups can also be formed by referencing to already defined group names-->
+   <!-- Manipulator group -->
     <group name="${prefix}${name}_manipulator">
       <chain base_link="${prefix}base_link" tip_link="${prefix}tool0" />
     </group>
+        <!-- Gripper group for controlling tooltip joints -->
+    <group name="${prefix}${name}_gripper">
+      <joint name="${prefix}tooltip1_joint"/>
+      <joint name="${prefix}tooltip2_joint"/>
+    </group>
+    <!-- Robot model group - includes all robot links for visualization and collision detection -->
+    <group name="${prefix}${name}_robot">
+      <link name="${prefix}base_link"/>
+      <link name="${prefix}shoulder_link"/>
+      <link name="${prefix}upper_arm_link"/>
+      <link name="${prefix}forearm_link"/>
+      <link name="${prefix}wrist_1_link"/>
+      <link name="${prefix}wrist_2_link"/>
+      <link name="${prefix}wrist_3_link"/>
+      <link name="${prefix}flange"/>
+      <link name="${prefix}tool0"/>
+      <link name="${prefix}quickchanger_link"/>
+      <link name="${prefix}suction_master_link"/>
+      <link name="${prefix}suction_link"/>
+      <link name="${prefix}gripper_link"/>
+      <link name="${prefix}tooltip1_link"/>
+      <link name="${prefix}tooltip2_link"/>
+    </group>
     <!--GROUP STATES - Purpose - Define a named state for a particular group, in terms of joint values. This is useful to define states like 'folded arms'-->
     <group_state name="${prefix}home" group="${prefix}${name}_manipulator">
-      <joint name="${prefix}elbow_joint" value="0" />
-      <joint name="${prefix}shoulder_lift_joint" value="-1.5707" />
-      <joint name="${prefix}shoulder_pan_joint" value="0" />
-      <joint name="${prefix}wrist_1_joint" value="0" />
-      <joint name="${prefix}wrist_2_joint" value="0" />
-      <joint name="${prefix}wrist_3_joint" value="0" />
+      <joint name="${prefix}elbow_joint" value="-1.623660393" />
+      <joint name="${prefix}shoulder_lift_joint" value="-1.155004847" />
+      <joint name="${prefix}shoulder_pan_joint" value="-3.72" />
+      <joint name="${prefix}wrist_1_joint" value="-1.559093451" />
+      <joint name="${prefix}wrist_2_joint" value="1.740479197" />
+      <joint name="${prefix}wrist_3_joint" value="-0.009424778" />
     </group_state>
     <group_state name="${prefix}up" group="${prefix}${name}_manipulator">
@@ -39,5 +63,19 @@
       <joint name="${prefix}wrist_3_joint" value="-0.11" />
     </group_state>
+    <!-- Gripper states -->
+    <group_state name="${prefix}gripper_open" group="${prefix}${name}_gripper">
+      <joint name="${prefix}tooltip1_joint" value="0.02" />
+      <joint name="${prefix}tooltip2_joint" value="-0.02" />
+    </group_state>
+    <group_state name="${prefix}gripper_closed" group="${prefix}${name}_gripper">
+      <joint name="${prefix}tooltip1_joint" value="0.03" />
+      <joint name="${prefix}tooltip2_joint" value="-0.03" />
+    </group_state>
+    <group_state name="${prefix}gripper_half_open" group="${prefix}${name}_gripper">
+      <joint name="${prefix}tooltip1_joint" value="0.01" />
+      <joint name="${prefix}tooltip2_joint" value="-0.01" />
+    </group_state>
     <!--END EFFECTOR - Purpose - Represent information about an end effector.-->
+    <end_effector name="${prefix}${name}_gripper" parent_link="${prefix}gripper_link" group="${prefix}${name}_gripper" />
     <!--VIRTUAL JOINT - Purpose - this element defines a virtual joint between a robot link and an external frame of reference (considered fixed with respect to the robot)-->
     <!--DISABLE COLLISIONS - By default it is assumed that any link of the robot could potentially come into collision with any other link in the robot. This tag disables collision checking between a specified pair of links. -->
@@ -53,4 +91,15 @@
     <disable_collisions link1="${prefix}wrist_1_link" link2="${prefix}wrist_3_link" reason="Never" />
     <disable_collisions link1="${prefix}wrist_2_link" link2="${prefix}wrist_3_link" reason="Adjacent" />
+    <!-- Quickchanger-gripper-suction collision exclusions -->
+    <disable_collisions link1="${prefix}wrist_3_link" link2="${prefix}quickchanger_link" reason="Adjacent" />
+    <disable_collisions link1="${prefix}quickchanger_link" link2="${prefix}suction_master_link" reason="Adjacent" />
+    <disable_collisions link1="${prefix}quickchanger_link" link2="${prefix}suction_link" reason="Adjacent" />
+    <disable_collisions link1="${prefix}quickchanger_link" link2="${prefix}gripper_link" reason="Adjacent" />
+    <disable_collisions link1="${prefix}gripper_link" link2="${prefix}tooltip1_link" reason="Adjacent" />
+    <disable_collisions link1="${prefix}gripper_link" link2="${prefix}tooltip2_link" reason="Adjacent" />
+    <disable_collisions link1="${prefix}suction_master_link" link2="${prefix}suction_link" reason="Adjacent" />
+    <!-- Additional collision exclusions for better collision detection -->
+    <disable_collisions link1="${prefix}flange" link2="${prefix}quickchanger_link" reason="Adjacent" />
+    <disable_collisions link1="${prefix}tool0" link2="${prefix}quickchanger_link" reason="Adjacent" />
   </xacro:macro>
 </robot>
