Commit message: ADDED CLEAN GAZEBO AGAIN

File: src/Universal_Robots_ROS2_Description/urdf/inc/ur_transmissions.xacro (robot description, xacro)
@@ -61,71 +61,4 @@
       </actuator>
     </transmission>
-<!-- UR Robot Gripper Tooltips -->
-<transmission name="tooltip1_trans">
-  <type>transmission_interface/SimpleTransmission</type>
-  <joint name="tooltip1_joint">
-    <hardwareInterface>${hw_interface}</hardwareInterface>
-  </joint>
-  <actuator name="tooltip1_motor">
-    <mechanicalReduction>1</mechanicalReduction>
-  </actuator>
-</transmission>
-<transmission name="tooltip2_trans">
-  <type>transmission_interface/SimpleTransmission</type>
-  <joint name="tooltip2_joint">
-    <hardwareInterface>${hw_interface}</hardwareInterface>
-  </joint>
-  <actuator name="tooltip2_motor">
-    <mechanicalReduction>1</mechanicalReduction>
-  </actuator>
-</transmission>
-<!-- ARF Axis Joints -->
-<transmission name="arf_axis_1_trans">
-  <type>transmission_interface/SimpleTransmission</type>
-  <joint name="arf_axis_1_joint">
-    <hardwareInterface>${hw_interface}</hardwareInterface>
-  </joint>
-  <actuator name="arf_axis_1_motor">
-    <mechanicalReduction>1</mechanicalReduction>
-  </actuator>
-</transmission>
-<transmission name="arf_axis_2_trans">
-  <type>transmission_interface/SimpleTransmission</type>
-  <joint name="arf_axis_2_joint">
-    <hardwareInterface>${hw_interface}</hardwareInterface>
-  </joint>
-  <actuator name="arf_axis_2_motor">
-    <mechanicalReduction>1</mechanicalReduction>
-  </actuator>
-</transmission>
-<!-- ARF Gripper Joints -->
-<transmission name="arf_gripper1_trans">
-  <type>transmission_interface/SimpleTransmission</type>
-  <joint name="arf_gripper_joint_1">
-    <hardwareInterface>${hw_interface}</hardwareInterface>
-  </joint>
-  <actuator name="arf_gripper_motor_1">
-    <mechanicalReduction>1</mechanicalReduction>
-  </actuator>
-</transmission>
-<transmission name="arf_gripper2_trans">
-  <type>transmission_interface/SimpleTransmission</type>
-  <joint name="arf_gripper_joint_2">
-    <hardwareInterface>${hw_interface}</hardwareInterface>
-  </joint>
-  <actuator name="arf_gripper_motor_2">
-    <mechanicalReduction>1</mechanicalReduction>
-  </actuator>
-</transmission>
-<!-- Denso Axis Joint -->
-<transmission name="denso_axis_trans">
-  <type>transmission_interface/SimpleTransmission</type>
-  <joint name="denso_axis_joint">
-    <hardwareInterface>${hw_interface}</hardwareInterface>
-  </joint>
-  <actuator name="denso_axis_motor">
-    <mechanicalReduction>1</mechanicalReduction>
-  </actuator>
-</transmission>
   </xacro:macro>
 </robot>

File: src/Universal_Robots_ROS2_Description/urdf/ur.ros2_control.xacro (robot description, xacro)
@@ -7,5 +7,5 @@
     sim_ignition:=false
     headless_mode:=false
-    initial_positions:=${dict(shoulder_pan_joint=0.0,shoulder_lift_joint=-1.57,elbow_joint=0.0,wrist_1_joint=-1.57,wrist_2_joint=0.0,wrist_3_joint=0.0,tooltip1_joint=0.0,tooltip2_joint=0.0,arf_axis_1_joint=0.0,arf_axis_2_joint=0.0)}
+    initial_positions:=${dict(shoulder_pan_joint=0.0,shoulder_lift_joint=-1.57,elbow_joint=0.0,wrist_1_joint=-1.57,wrist_2_joint=0.0,wrist_3_joint=0.0)}
     use_tool_communication:=false
     script_filename output_recipe_filename
@@ -65,5 +65,4 @@
         </xacro:unless>
       </hardware>
-      <!-- UR Robot Joints -->
       <joint name="${tf_prefix}shoulder_pan_joint">
         <command_interface name="position"/>
@@ -122,117 +121,4 @@
           <!-- initial position for the FakeSystem and simulation -->
           <param name="initial_value">${initial_positions['wrist_3_joint']}</param>
-        </state_interface>
-        <state_interface name="velocity"/>
-        <state_interface name="effort"/>
-      </joint>
-      <!-- UR Robot Gripper Tooltips -->
-      <joint name="${tf_prefix}tooltip1_joint">
-        <command_interface name="position"/>
-        <state_interface name="position">
-          <!-- initial position for the FakeSystem and simulation -->
-          <param name="initial_value">${initial_positions['tooltip1_joint']}</param>
-        </state_interface>
-        <state_interface name="velocity"/>
-        <state_interface name="effort"/>
-      </joint>
-      <joint name="${tf_prefix}tooltip2_joint">
-        <command_interface name="position"/>
-        <state_interface name="position">
-          <!-- initial position for the FakeSystem and simulation -->
-          <param name="initial_value">${initial_positions['tooltip2_joint']}</param>
-        </state_interface>
-        <state_interface name="velocity"/>
-        <state_interface name="effort"/>
-      </joint>
-      <!-- ARF Axis Joints -->
-      <joint name="${tf_prefix}arf_axis_1_joint">
-        <command_interface name="position"/>
-        <command_interface name="velocity"/>
-        <state_interface name="position">
-          <!-- initial position for the FakeSystem and simulation -->
-          <param name="initial_value">${initial_positions['arf_axis_1_joint']}</param>
-        </state_interface>
-        <state_interface name="velocity"/>
-        <state_interface name="effort"/>
-      </joint>
-      <joint name="${tf_prefix}arf_axis_2_joint">
-        <command_interface name="position"/>
-        <command_interface name="velocity"/>
-        <state_interface name="position">
-          <!-- initial position for the FakeSystem and simulation -->
-          <param name="initial_value">${initial_positions['arf_axis_2_joint']}</param>
-        </state_interface>
-        <state_interface name="velocity"/>
-        <state_interface name="effort"/>
-      </joint>
-      <!-- ARF Gripper Joints -->
-      <joint name="arf_gripper_joint_1">
-        <command_interface name="position"/>
-        <command_interface name="velocity"/>
-        <state_interface name="position">
-          <!-- initial position for the FakeSystem and simulation -->
-          <param name="initial_value">${initial_positions['arf_gripper_joint_1']}</param>
-        </state_interface>
-        <state_interface name="velocity"/>
-        <state_interface name="effort"/>
-      </joint>
-      <joint name="arf_gripper_joint_2">
-        <command_interface name="position"/>
-        <command_interface name="velocity"/>
-        <state_interface name="position">
-          <!-- initial position for the FakeSystem and simulation -->
-          <param name="initial_value">${initial_positions['arf_gripper_joint_2']}</param>
-        </state_interface>
-        <state_interface name="velocity"/>
-        <state_interface name="effort"/>
-      </joint>
-      <!-- Denso Robot Joints -->
-      <joint name="denso_joint_1">
-        <command_interface name="position"/>
-        <command_interface name="velocity"/>
-        <state_interface name="position">
-          <!-- initial position for the FakeSystem and simulation -->
-          <param name="initial_value">${initial_positions['denso_joint_1']}</param>
-        </state_interface>
-        <state_interface name="velocity"/>
-        <state_interface name="effort"/>
-      </joint>
-      <joint name="denso_joint_2">
-        <command_interface name="position"/>
-        <command_interface name="velocity"/>
-        <state_interface name="position">
-          <!-- initial position for the FakeSystem and simulation -->
-          <param name="initial_value">${initial_positions['denso_joint_2']}</param>
-        </state_interface>
-        <state_interface name="velocity"/>
-        <state_interface name="effort"/>
-      </joint>
-      <joint name="denso_joint_3">
-        <command_interface name="position"/>
-        <command_interface name="velocity"/>
-        <state_interface name="position">
-          <!-- initial position for the FakeSystem and simulation -->
-          <param name="initial_value">${initial_positions['denso_joint_3']}</param>
-        </state_interface>
-        <state_interface name="velocity"/>
-        <state_interface name="effort"/>
-      </joint>
-      <joint name="denso_joint_4">
-        <command_interface name="position"/>
-        <command_interface name="velocity"/>
-        <state_interface name="position">
-          <!-- initial position for the FakeSystem and simulation -->
-          <param name="initial_value">${initial_positions['denso_joint_4']}</param>
-        </state_interface>
-        <state_interface name="velocity"/>
-        <state_interface name="effort"/>
-      </joint>
-      <!-- Denso Axis Joint -->
-      <joint name="denso_axis_joint">
-        <command_interface name="position"/>
-        <command_interface name="velocity"/>
-        <state_interface name="position">
-          <!-- initial position for the FakeSystem and simulation -->
-          <param name="initial_value">${initial_positions['denso_axis_joint']}</param>
         </state_interface>
         <state_interface name="velocity"/>

File: src/Universal_Robots_ROS2_Description/urdf/ur.urdf.xacro (robot description, xacro)
@@ -3,16 +3,6 @@
    <!-- robot name parameter -->
    <xacro:arg name="name" default="ur"/>
-   <!-- import main ur10 + trolley macro -->
-   <xacro:include filename="$(find ur_description)/urdf/ur10.xacro"/>
-   <!-- import quickchanger + gripper + suction macro -->
-   <xacro:include filename="$(find ur_description)/urdf/quickchanger_gripper_suction.xacro"/>
-   <!-- import arf + trolley macro -->
-   <xacro:include filename="$(find ur_description)/urdf/arf.xacro"/>
-   <!-- import vision + trolley macro -->
-   <xacro:include filename="$(find ur_description)/urdf/vision.xacro"/>
-   <!-- import toolchanger + trolley macro -->
-   <xacro:include filename="$(find ur_description)/urdf/toolchanger.xacro"/>
-   <!-- import denso + trolley macro -->
-   <xacro:include filename="$(find ur_description)/urdf/denso.xacro"/>
+   <!-- import main macro -->
+   <xacro:include filename="$(find ur_description)/urdf/ur_macro.xacro"/>
    <!-- possible 'ur_type' values: ur3, ur3e, ur5, ur5e, ur7e, ur10, ur10e, ur12e, ur16e, ur15, ur20, ur30 -->
    <!-- the default value should raise an error in case this was called without defining the type -->
@@ -87,12 +77,4 @@
      </joint>
    </xacro:if>
-      <!-- vision components -->
-   <xacro:vision parent="world"/>
-   <!-- ARF components -->
-   <xacro:arf parent="world"/>
-   <!-- toolchanger components -->
-   <xacro:toolchanger parent="world"/>
-   <!-- denso components -->
-   <xacro:denso parent="world"/>
    <!-- arm -->
    <xacro:ur_robot
@@ -100,5 +82,4 @@
      tf_prefix="$(arg tf_prefix)"
      parent="world"
-     prefix=""
      joint_limits_parameters_file="$(arg joint_limit_params)"
      kinematics_parameters_file="$(arg kinematics_params)"
@@ -136,6 +117,4 @@
      <origin xyz="0 0 0" rpy="0 0 0" />          <!-- position robot in the world -->
    </xacro:ur_robot>
-  <!-- attach gripper -->
-   <xacro:quickchanger_gripper_suction parent="$(arg tf_prefix)wrist_3_link"/>
    <xacro:if value="$(arg sim_gazebo)">
     <!-- Gazebo plugins -->

File: src/Universal_Robots_ROS2_Driver/ur_moveit_config/srdf/ur_macro.srdf.xacro (robot description, xacro)
@@ -11,39 +11,15 @@
     <!--CHAINS - When a chain is specified, all the links along the chain (including endpoints) are included in the group. Additionally, all the joints that are parents to included links are also included. This means that joints along the chain and the parent joint of the base link are included in the group-->
     <!--SUBGROUPS - Groups can also be formed by referencing to already defined group names-->
-   <!-- Manipulator group -->
     <group name="${prefix}${name}_manipulator">
       <chain base_link="${prefix}base_link" tip_link="${prefix}tool0" />
     </group>
-        <!-- Gripper group for controlling tooltip joints -->
-    <group name="${prefix}${name}_gripper">
-      <joint name="${prefix}tooltip1_joint"/>
-      <joint name="${prefix}tooltip2_joint"/>
-    </group>
-    <!-- Robot model group - includes all robot links for visualization and collision detection -->
-    <group name="${prefix}${name}_robot">
-      <link name="${prefix}base_link"/>
-      <link name="${prefix}shoulder_link"/>
-      <link name="${prefix}upper_arm_link"/>
-      <link name="${prefix}forearm_link"/>
-      <link name="${prefix}wrist_1_link"/>
-      <link name="${prefix}wrist_2_link"/>
-      <link name="${prefix}wrist_3_link"/>
-      <link name="${prefix}flange"/>
-      <link name="${prefix}tool0"/>
-      <link name="${prefix}quickchanger_link"/>
-      <link name="${prefix}suction_master_link"/>
-      <link name="${prefix}suction_link"/>
-      <link name="${prefix}gripper_link"/>
-      <link name="${prefix}tooltip1_link"/>
-      <link name="${prefix}tooltip2_link"/>
-    </group>
     <!--GROUP STATES - Purpose - Define a named state for a particular group, in terms of joint values. This is useful to define states like 'folded arms'-->
     <group_state name="${prefix}home" group="${prefix}${name}_manipulator">
-      <joint name="${prefix}elbow_joint" value="-1.623660393" />
-      <joint name="${prefix}shoulder_lift_joint" value="-1.155004847" />
-      <joint name="${prefix}shoulder_pan_joint" value="-3.72" />
-      <joint name="${prefix}wrist_1_joint" value="-1.559093451" />
-      <joint name="${prefix}wrist_2_joint" value="1.740479197" />
-      <joint name="${prefix}wrist_3_joint" value="-0.009424778" />
+      <joint name="${prefix}elbow_joint" value="0" />
+      <joint name="${prefix}shoulder_lift_joint" value="-1.5707" />
+      <joint name="${prefix}shoulder_pan_joint" value="0" />
+      <joint name="${prefix}wrist_1_joint" value="0" />
+      <joint name="${prefix}wrist_2_joint" value="0" />
+      <joint name="${prefix}wrist_3_joint" value="0" />
     </group_state>
     <group_state name="${prefix}up" group="${prefix}${name}_manipulator">
@@ -63,19 +39,5 @@
       <joint name="${prefix}wrist_3_joint" value="-0.11" />
     </group_state>
-    <!-- Gripper states -->
-    <group_state name="${prefix}gripper_open" group="${prefix}${name}_gripper">
-      <joint name="${prefix}tooltip1_joint" value="0.02" />
-      <joint name="${prefix}tooltip2_joint" value="-0.02" />
-    </group_state>
-    <group_state name="${prefix}gripper_closed" group="${prefix}${name}_gripper">
-      <joint name="${prefix}tooltip1_joint" value="0.03" />
-      <joint name="${prefix}tooltip2_joint" value="-0.03" />
-    </group_state>
-    <group_state name="${prefix}gripper_half_open" group="${prefix}${name}_gripper">
-      <joint name="${prefix}tooltip1_joint" value="0.01" />
-      <joint name="${prefix}tooltip2_joint" value="-0.01" />
-    </group_state>
     <!--END EFFECTOR - Purpose - Represent information about an end effector.-->
-    <end_effector name="${prefix}${name}_gripper" parent_link="${prefix}gripper_link" group="${prefix}${name}_gripper" />
     <!--VIRTUAL JOINT - Purpose - this element defines a virtual joint between a robot link and an external frame of reference (considered fixed with respect to the robot)-->
     <!--DISABLE COLLISIONS - By default it is assumed that any link of the robot could potentially come into collision with any other link in the robot. This tag disables collision checking between a specified pair of links. -->
@@ -91,15 +53,4 @@
     <disable_collisions link1="${prefix}wrist_1_link" link2="${prefix}wrist_3_link" reason="Never" />
     <disable_collisions link1="${prefix}wrist_2_link" link2="${prefix}wrist_3_link" reason="Adjacent" />
-    <!-- Quickchanger-gripper-suction collision exclusions -->
-    <disable_collisions link1="${prefix}wrist_3_link" link2="${prefix}quickchanger_link" reason="Adjacent" />
-    <disable_collisions link1="${prefix}quickchanger_link" link2="${prefix}suction_master_link" reason="Adjacent" />
-    <disable_collisions link1="${prefix}quickchanger_link" link2="${prefix}suction_link" reason="Adjacent" />
-    <disable_collisions link1="${prefix}quickchanger_link" link2="${prefix}gripper_link" reason="Adjacent" />
-    <disable_collisions link1="${prefix}gripper_link" link2="${prefix}tooltip1_link" reason="Adjacent" />
-    <disable_collisions link1="${prefix}gripper_link" link2="${prefix}tooltip2_link" reason="Adjacent" />
-    <disable_collisions link1="${prefix}suction_master_link" link2="${prefix}suction_link" reason="Adjacent" />
-    <!-- Additional collision exclusions for better collision detection -->
-    <disable_collisions link1="${prefix}flange" link2="${prefix}quickchanger_link" reason="Adjacent" />
-    <disable_collisions link1="${prefix}tool0" link2="${prefix}quickchanger_link" reason="Adjacent" />
   </xacro:macro>
 </robot>

Commit message: gripper tooltips working (need to add quickchanger + suction)

File: src/Universal_Robots_ROS2_Description/urdf/inc/ur_transmissions.xacro (robot description, xacro)
@@ -61,4 +61,23 @@
       </actuator>
     </transmission>
+    <!-- UR Robot Gripper Tooltips -->
+<transmission name="tooltip1_trans">
+  <type>transmission_interface/SimpleTransmission</type>
+  <joint name="tooltip1_joint">
+    <hardwareInterface>${hw_interface}</hardwareInterface>
+  </joint>
+  <actuator name="tooltip1_motor">
+    <mechanicalReduction>1</mechanicalReduction>
+  </actuator>
+</transmission>
+<transmission name="tooltip2_trans">
+  <type>transmission_interface/SimpleTransmission</type>
+  <joint name="tooltip2_joint">
+    <hardwareInterface>${hw_interface}</hardwareInterface>
+  </joint>
+  <actuator name="tooltip2_motor">
+    <mechanicalReduction>1</mechanicalReduction>
+  </actuator>
+</transmission>
     <!-- ARF Axis Joints -->
     <transmission name="arf_axis_1_trans">

File: src/Universal_Robots_ROS2_Description/urdf/ur.ros2_control.xacro (robot description, xacro)
@@ -121,4 +121,23 @@
           <!-- initial position for the FakeSystem and simulation -->
           <param name="initial_value">${initial_positions['wrist_3_joint']}</param>
+        </state_interface>
+        <state_interface name="velocity"/>
+        <state_interface name="effort"/>
+      </joint>
+      <!-- UR Robot Gripper Tooltips -->
+      <joint name="${tf_prefix}tooltip1_joint">
+        <command_interface name="position"/>
+        <state_interface name="position">
+          <!-- initial position for the FakeSystem and simulation -->
+          <param name="initial_value">${initial_positions['tooltip1_joint']}</param>
+        </state_interface>
+        <state_interface name="velocity"/>
+        <state_interface name="effort"/>
+      </joint>
+      <joint name="${tf_prefix}tooltip2_joint">
+        <command_interface name="position"/>
+        <state_interface name="position">
+          <!-- initial position for the FakeSystem and simulation -->
+          <param name="initial_value">${initial_positions['tooltip2_joint']}</param>
         </state_interface>
         <state_interface name="velocity"/>

File: src/Universal_Robots_ROS2_Description/urdf/ur.urdf.xacro (robot description, xacro)
@@ -9,4 +9,6 @@
    <!-- import toolchanger macro -->
    <xacro:include filename="$(find ur_description)/urdf/toolchanger.xacro"/>
+   <!-- import quickchanger_grippers macro -->
+   <xacro:include filename="$(find ur_description)/urdf/quickchanger_grippers.xacro"/>
    <!-- import arf macro -->
    <xacro:include filename="$(find ur_description)/urdf/arf.xacro"/>
@@ -136,4 +138,6 @@
      <origin xyz="0 0 0" rpy="0 0 0" />          <!-- position robot in the world -->
    </xacro:ur_robot>
+     <!-- attach gripper -->
+   <xacro:quickchanger_grippers parent="$(arg tf_prefix)wrist_3_link"/>
    <xacro:if value="$(arg sim_gazebo)">
     <!-- Gazebo plugins -->

Commit message: setup suction gripper on/off using vacuum gripper plugin

File: src/Universal_Robots_ROS2_Description/urdf/inc/ur_transmissions.xacro (robot description, xacro)
@@ -80,4 +80,14 @@
   </actuator>
 </transmission>
+<!-- Vacuum Gripper Joint -->
+<transmission name="suction_trans">
+  <type>transmission_interface/SimpleTransmission</type>
+  <joint name="suction_joint">
+    <hardwareInterface>${hw_interface}</hardwareInterface>
+  </joint>
+  <actuator name="suction_motor">
+    <mechanicalReduction>1</mechanicalReduction>
+  </actuator>
+</transmission>
     <!-- ARF Axis Joints -->
     <transmission name="arf_axis_1_trans">

File: src/Universal_Robots_ROS2_Description/urdf/quickchanger_grippers.xacro (robot description, xacro)
@@ -87,8 +87,11 @@
     </link>
     <!-- suction_joint -->
-    <joint name="suction_joint" type="fixed">
+    <joint name="suction_joint" type="revolute">
       <parent link="suction_master_link"/>
       <child link="suction_link"/>
       <origin xyz="0 0 0" rpy="0 0 0"/>
+      <axis xyz="0 0 1"/>
+      <limit effort="50" velocity="50" lower="0" upper="0"/>
+      <dynamics damping="0.0" friction="10"/>
     </joint>
     <!-- gripper_link -->

File: src/Universal_Robots_ROS2_Description/urdf/ur.ros2_control.xacro (robot description, xacro)
@@ -140,4 +140,14 @@
           <!-- initial position for the FakeSystem and simulation -->
           <param name="initial_value">${initial_positions['tooltip2_joint']}</param>
+        </state_interface>
+        <state_interface name="velocity"/>
+        <state_interface name="effort"/>
+      </joint>
+      <!-- Vacuum Gripper Joint -->
+      <joint name="${tf_prefix}suction_joint">
+        <command_interface name="position"/>
+        <state_interface name="position">
+          <!-- initial position for the FakeSystem and simulation -->
+          <param name="initial_value">${initial_positions['suction_joint']}</param>
         </state_interface>
         <state_interface name="velocity"/>

File: src/Universal_Robots_ROS2_Description/urdf/ur.urdf.xacro (robot description, xacro)
@@ -148,4 +148,15 @@
         <parameters>$(arg simulation_controllers)</parameters>
       </plugin>
+    <!-- Vacuum Gripper Plugin -->
+    <plugin name="vacuum_gripper" filename="libgazebo_ros_vacuum_gripper.so">
+      <ros>
+        <namespace>/demo</namespace>
+        <remapping>switch:=switch_demo</remapping>
+        <remapping>grasping:=grasping_demo</remapping>
+      </ros>
+      <link_name>suction_link</link_name>
+      <max_distance>0.5</max_distance>
+      <fixed>ground_plane</fixed>
+    </plugin>
     </gazebo>
   </xacro:if>
