Commit message: edited denso j3 position and kinematics solver config (movel not working when connected to client gui yet)

File: src/denso_robot_drivers_ros2/denso_robot_descriptions/robots/hsr065a1_n32/urdf/denso_robot_kinematics.xacro (robot description, xacro)
@@ -131,7 +131,7 @@
       <parent link="${namespace}J2"/>
       <child link="${namespace}J3"/>
-      <origin rpy="0.0 0.0 0.0" xyz="0.5 0.0 0.5067"/>
+      <origin rpy="0.0 0.0 0.0" xyz="0.5 0.0 0.22"/>
       <axis xyz="0.0 0.0 1.0"/>
-      <limit effort="100" lower="-0.1" upper="0.22" velocity="1.9"/>
+      <limit effort="100" lower="-10" upper="10" velocity="1.9"/>
       <dynamics damping="0.2" friction="0.01"/>
     </joint>
@@ -161,5 +161,5 @@
       <parent link="${namespace}J3"/>
       <child link="${namespace}J4"/>
-      <origin rpy="0.0 0.0 0.0" xyz="0.0 0.0 -0.6047"/>
+      <origin rpy="0.0 0.0 1.57" xyz="0.0 0.0 -0.6047"/>
       <axis xyz="0.0 0.0 1.0"/>
       <limit effort="10" lower="-6.28318530717959" upper="6.28318530717959" velocity="25.2968981715147"/>

Commit message: edited denso to be j4-flange-tool-screwdriver / working fine

File: src/denso_robot_drivers_ros2/denso_robot_descriptions/robots/hsr065a1_n32/urdf/denso_robot_kinematics.xacro (robot description, xacro)
@@ -174,5 +174,5 @@
       </inertial>
     </link>
-    <joint name="${namespace}J4-flange" type="fixed">
+    <joint name="${namespace}joint_flange" type="fixed">
       <parent link="${namespace}J4" />
       <child link="${namespace}flange" />
@@ -187,5 +187,5 @@
       </inertial>
     </link>
-    <joint name="${namespace}flange-tool0" type="fixed">
+    <joint name="${namespace}joint_tool0" type="fixed">
       <!-- Denso toolframe - X+ front, Y+ right, Z+ up -->
       <origin xyz="0 0 0" rpy="3.141592 0 0"/>
@@ -193,4 +193,33 @@
       <child link="${namespace}tool0"/>
     </joint>
+         <!-- Screwdriver link attached after J4 -->
+    <link name="${namespace}screwdriver">
+      <visual>
+        <origin rpy="0 0 -1.57" xyz="0 0 0"/>
+        <geometry>
+          <mesh filename="file://$(find denso_robot_descriptions)/robots/${model}/meshes/stl/denso_screwdriver.STL" scale="1 1 1"/>
+        </geometry>
+        <material name="">
+          <color rgba="0.7 0.7 0.7 1.0"/>
+        </material>
+      </visual>
+      <collision>
+        <origin rpy="0 0 -1.57" xyz="0 0 0"/>
+        <geometry>
+          <mesh filename="file://$(find denso_robot_descriptions)/robots/${model}/meshes/stl/denso_screwdriver.STL" scale="1 1 1"/>
+        </geometry>
+      </collision>
+      <inertial>
+        <mass value="1.5"/>
+        <origin rpy="0.0 0.0 0.0" xyz="0.0 0.0 -0.3"/>
+        <inertia ixx="0.02" ixy="0" ixz="0" iyy="0.02" iyz="0" izz="0.01"/>
+      </inertial>
+    </link>
+    <!-- Joint connecting J4 to screwdriver -->
+    <joint name="${namespace}screwdriver_joint" type="fixed">
+      <parent link="${namespace}flange"/>
+      <child link="${namespace}screwdriver"/>
+      <origin rpy="0.0 0 0" xyz="0.0 0.0 0.0"/>
+    </joint>
   </xacro:macro>
 </robot>
