Commit message: edited denso folder structure + spawn arf gripper closed

File: src/UR10/ur_description/urdf/denso.xacro (robot description, xacro)
@@ -3,5 +3,5 @@
   <!-- Include Denso robot descriptions -->
   <xacro:macro name="denso" params="parent">
-  <xacro:include filename="$(find denso_robot_descriptions)/robots/hsr065a1_n32/urdf/denso_robot_macro.xacro" />
+  <xacro:include filename="$(find denso_description)/robot/urdf/denso_robot_macro.xacro" />
   <xacro:property name="denso_visual_params" value="${xacro.load_yaml('$(find ur_description)/config/denso_visual_parameters.yaml')}"/>
   <xacro:property name="sec_mesh_files" value="${denso_visual_params['mesh_files']}" scope="parent"/>
@@ -70,5 +70,5 @@
       sim="true"
       namespace="denso_"
-      model="hsr065a1_n32" />
+      />
   </xacro:macro>
 </robot>

File: src/UR10/ur_moveit/srdf/ur_denso.srdf.xacro (robot description, xacro)
@@ -11,5 +11,5 @@
   <xacro:include filename="$(find ur_moveit)/srdf/ur_macro.srdf.xacro"/>
   <!-- Include Denso SRDF macro -->
-  <xacro:include filename="$(find denso_robot_moveit_config)/robots/$(arg denso_model)/srdf/denso_robot_macro.srdf.xacro"/>
+  <xacro:include filename="$(find denso_moveit)/robot/srdf/denso_robot_macro.srdf.xacro"/>
   <!-- Create UR planning group -->
   <xacro:ur_srdf name="$(arg name)" prefix="$(arg prefix)"/>

File: src/denso/denso_description/robot/urdf/denso_robot.ros2_control.xacro (robot description, xacro)
@@ -5,5 +5,4 @@
     sim:=false fake_sensor_commands:=false
     ip_address
-    model
     robot_joints joint_1 joint_2 joint_3 joint_4
     arm_group
@@ -23,5 +22,5 @@
           <param name="robot_name">${robot_name}</param>
           <param name="node_name">denso_robot_control</param>
-          <param name="node_namespace">${namespace}${model}</param>
+          <param name="node_namespace">${namespace}</param>
           <param name="robot_joints">${robot_joints}</param>
           <param name="joint_1">${joint_1}</param>

File: src/denso/denso_description/robot/urdf/denso_robot_kinematics.xacro (robot description, xacro)
@@ -1,5 +1,5 @@
 <?xml version='1.0' encoding='UTF-8'?>
 <robot xmlns:xacro="http://www.ros.org/wiki/xacro">
-  <xacro:macro name="denso_robot_arm_kinematics" params="namespace model parent">
+  <xacro:macro name="denso_robot_arm_kinematics" params="namespace parent">
     <!-- denso base link -->
     <link name="${namespace}base_link">
@@ -7,14 +7,14 @@
         <origin rpy="0 0 0" xyz="0 0 0"/>
         <geometry>
-          <mesh filename="file://$(find denso_robot_descriptions)/robots/${model}/meshes/stl/denso_base_link.STL" scale="1 1 1"/>
-        </geometry>
-        <material name="">
-          <color rgba="0.7 0.7 0.7 1.0"/>
-        </material>
-      </visual>
-      <collision>
-        <origin rpy="0 0 0" xyz="0 0 0"/>
-        <geometry>
-          <mesh filename="file://$(find denso_robot_descriptions)/robots/${model}/meshes/stl/denso_base_link.STL" scale="1 1 1"/>
+          <mesh filename="file://$(find denso_description)/robot/meshes/stl/denso_base_link.STL" scale="1 1 1"/>
+        </geometry>
+        <material name="">
+          <color rgba="0.7 0.7 0.7 1.0"/>
+        </material>
+      </visual>
+      <collision>
+        <origin rpy="0 0 0" xyz="0 0 0"/>
+        <geometry>
+          <mesh filename="file://$(find denso_description)/robot/meshes/stl/denso_base_link.STL" scale="1 1 1"/>
         </geometry>
       </collision>
@@ -50,14 +50,14 @@
         <origin rpy="0 0 0" xyz="0 0 0"/>
         <geometry>
-          <mesh filename="file://$(find denso_robot_descriptions)/robots/${model}/meshes/stl/denso_link1.STL" scale="1 1 1"/>
-        </geometry>
-        <material name="">
-          <color rgba="0.7 0.7 0.7 1.0"/>
-        </material>
-      </visual>
-      <collision>
-        <origin rpy="0 0 0" xyz="0 0 0"/>
-        <geometry>
-          <mesh filename="file://$(find denso_robot_descriptions)/robots/${model}/meshes/stl/denso_link1.STL" scale="1 1 1"/>
+          <mesh filename="file://$(find denso_description)/robot/meshes/stl/denso_link1.STL" scale="1 1 1"/>
+        </geometry>
+        <material name="">
+          <color rgba="0.7 0.7 0.7 1.0"/>
+        </material>
+      </visual>
+      <collision>
+        <origin rpy="0 0 0" xyz="0 0 0"/>
+        <geometry>
+          <mesh filename="file://$(find denso_description)/robot/meshes/stl/denso_link1.STL" scale="1 1 1"/>
         </geometry>
       </collision>
@@ -80,14 +80,14 @@
         <origin rpy="0 0 0" xyz="0 0 0"/>
         <geometry>
-          <mesh filename="file://$(find denso_robot_descriptions)/robots/${model}/meshes/stl/denso_link2.STL" scale="1 1 1"/>
-        </geometry>
-        <material name="">
-          <color rgba="0.7 0.7 0.7 1.0"/>
-        </material>
-      </visual>
-      <collision>
-        <origin rpy="0 0 0" xyz="0 0 0"/>
-        <geometry>
-          <mesh filename="file://$(find denso_robot_descriptions)/robots/${model}/meshes/stl/denso_link2.STL" scale="1 1 1"/>
+          <mesh filename="file://$(find denso_description)/robot/meshes/stl/denso_link2.STL" scale="1 1 1"/>
+        </geometry>
+        <material name="">
+          <color rgba="0.7 0.7 0.7 1.0"/>
+        </material>
+      </visual>
+      <collision>
+        <origin rpy="0 0 0" xyz="0 0 0"/>
+        <geometry>
+          <mesh filename="file://$(find denso_description)/robot/meshes/stl/denso_link2.STL" scale="1 1 1"/>
         </geometry>
       </collision>
@@ -110,14 +110,14 @@
         <origin rpy="0 0 0" xyz="0 0 0"/>
         <geometry>
-          <mesh filename="file://$(find denso_robot_descriptions)/robots/${model}/meshes/stl/denso_link3.STL" scale="1 1 1"/>
-        </geometry>
-        <material name="">
-          <color rgba="0.7 0.7 0.7 1.0"/>
-        </material>
-      </visual>
-      <collision>
-        <origin rpy="0 0 0" xyz="0 0 0"/>
-        <geometry>
-          <mesh filename="file://$(find denso_robot_descriptions)/robots/${model}/meshes/stl/denso_link3.STL" scale="1 1 1"/>
+          <mesh filename="file://$(find denso_description)/robot/meshes/stl/denso_link3.STL" scale="1 1 1"/>
+        </geometry>
+        <material name="">
+          <color rgba="0.7 0.7 0.7 1.0"/>
+        </material>
+      </visual>
+      <collision>
+        <origin rpy="0 0 0" xyz="0 0 0"/>
+        <geometry>
+          <mesh filename="file://$(find denso_description)/robot/meshes/stl/denso_link3.STL" scale="1 1 1"/>
         </geometry>
       </collision>
@@ -198,5 +198,5 @@
         <origin rpy="0 0 -1.57" xyz="0 0 0"/>
         <geometry>
-          <mesh filename="file://$(find denso_robot_descriptions)/robots/${model}/meshes/stl/denso_screwdriver.STL" scale="1 1 1"/>
+          <mesh filename="file://$(find denso_description)/robot/meshes/stl/denso_screwdriver.STL" scale="1 1 1"/>
         </geometry>
         <material name="">
@@ -207,5 +207,5 @@
         <origin rpy="0 0 -1.57" xyz="0 0 0"/>
         <geometry>
-          <mesh filename="file://$(find denso_robot_descriptions)/robots/${model}/meshes/stl/denso_screwdriver.STL" scale="1 1 1"/>
+          <mesh filename="file://$(find denso_description)/robot/meshes/stl/denso_screwdriver.STL" scale="1 1 1"/>
         </geometry>
       </collision>

File: src/denso/denso_description/robot/urdf/denso_robot_macro.xacro (robot description, xacro)
@@ -10,5 +10,4 @@
   -->
   <xacro:macro name="denso_robot" params="
-    model:=hsr065a1_n32
     namespace:=denso_
     transmission_hw_interface:=hardware_interface/PositionJointInterface
@@ -29,9 +28,9 @@
   >
     <!-- Robot data required by the denso driver -->
-    <xacro:include filename="$(find denso_robot_descriptions)/robots/${model}/urdf/denso_robot_transmissions.xacro" />
+    <xacro:include filename="$(find denso_description)/robot/urdf/denso_robot_transmissions.xacro" />
     <!-- robot kinematics include -->
-    <xacro:include filename="$(find denso_robot_descriptions)/robots/${model}/urdf/denso_robot_kinematics.xacro" />
+    <xacro:include filename="$(find denso_description)/robot/urdf/denso_robot_kinematics.xacro" />
     <!-- ros2 control include -->
-    <xacro:include filename="$(find denso_robot_descriptions)/robots/${model}/urdf/denso_robot.ros2_control.xacro" />
+    <xacro:include filename="$(find denso_description)/robot/urdf/denso_robot.ros2_control.xacro" />
     <!-- ros2 control instance -->
     <xacro:denso_robot_ros2_control
@@ -39,5 +38,4 @@
       namespace=""
       sim="${sim}"
-      model="${model}"
       ip_address="${ip_address}"
       robot_name="${robot_name}"
@@ -57,5 +55,5 @@
     <!-- Placeholder for ros2_control transmission which don't yet exist -->
     <!-- links -  main serial chain -->
-    <xacro:denso_robot_arm_kinematics namespace="${namespace}" model="${model}" parent="${parent}" />
+    <xacro:denso_robot_arm_kinematics namespace="${namespace}" parent="${parent}" />
   </xacro:macro>
 </robot>

File: src/denso/denso_description/urdf/denso_robot.urdf.xacro (robot description, xacro)
@@ -1,8 +1,6 @@
 <?xml version="1.0"?>
-<robot xmlns:xacro="http://wiki.ros.org/xacro" name="$(arg model)">
-   <!-- robot name parameter -->
-   <xacro:arg name="model" default="denso_robot"/>
+<robot xmlns:xacro="http://wiki.ros.org/xacro" name="denso_robot">
    <!-- import main macro -->
-   <xacro:include filename="$(find denso_robot_descriptions)/robots/$(arg model)/urdf/denso_robot_macro.xacro"/>
+   <xacro:include filename="$(find denso_description)/robot/urdf/denso_robot_macro.xacro"/>
    <!-- parameters -->
    <xacro:arg name="namespace" default="" />
@@ -16,5 +14,4 @@
    <!-- arm -->
    <xacro:denso_robot
-     model="$(arg model)"
      namespace="$(arg namespace)"
      transmission_hw_interface="$(arg transmission_hw_interface)"

File: src/denso/denso_moveit/srdf/denso_robot.srdf.xacro (robot description, xacro)
@@ -5,5 +5,5 @@
   <!-- parameters -->
   <xacro:arg name="namespace" default="" />
-  <xacro:include filename="$(find denso_robot_moveit_config)/robots/$(arg model)/srdf/denso_robot_macro.srdf.xacro"/>
+  <xacro:include filename="$(find denso_moveit)/robot/srdf/denso_robot_macro.srdf.xacro"/>
   <xacro:denso_robot_srdf name="$(arg namespace)$(arg model)" namespace="$(arg namespace)"/>
 </robot>

Commit message: edited denso folder (delete unused, moveit file location changed)

File: src/UR10/ur_description/urdf/denso.xacro (robot description, xacro)
@@ -3,5 +3,5 @@
   <!-- Include Denso robot descriptions -->
   <xacro:macro name="denso" params="parent">
-  <xacro:include filename="$(find denso_description)/robot/urdf/denso_robot_macro.xacro" />
+  <xacro:include filename="$(find denso_description)/urdf/denso_robot_macro.xacro" />
   <xacro:property name="denso_visual_params" value="${xacro.load_yaml('$(find ur_description)/config/denso_visual_parameters.yaml')}"/>
   <xacro:property name="sec_mesh_files" value="${denso_visual_params['mesh_files']}" scope="parent"/>

File: src/UR10/ur_moveit/srdf/ur_denso.srdf.xacro (robot description, xacro)
@@ -11,5 +11,5 @@
   <xacro:include filename="$(find ur_moveit)/srdf/ur_macro.srdf.xacro"/>
   <!-- Include Denso SRDF macro -->
-  <xacro:include filename="$(find denso_moveit)/robot/srdf/denso_robot_macro.srdf.xacro"/>
+  <xacro:include filename="$(find ur_moveit)/srdf/denso_robot_macro.srdf.xacro"/>
   <!-- Create UR planning group -->
   <xacro:ur_srdf name="$(arg name)" prefix="$(arg prefix)"/>

File: src/denso/denso_description/urdf/denso_robot_kinematics.xacro (robot description, xacro)
@@ -7,14 +7,14 @@
         <origin rpy="0 0 0" xyz="0 0 0"/>
         <geometry>
-          <mesh filename="file://$(find denso_description)/robot/meshes/stl/denso_base_link.STL" scale="1 1 1"/>
-        </geometry>
-        <material name="">
-          <color rgba="0.7 0.7 0.7 1.0"/>
-        </material>
-      </visual>
-      <collision>
-        <origin rpy="0 0 0" xyz="0 0 0"/>
-        <geometry>
-          <mesh filename="file://$(find denso_description)/robot/meshes/stl/denso_base_link.STL" scale="1 1 1"/>
+          <mesh filename="file://$(find denso_description)/meshes/denso_base_link.STL" scale="1 1 1"/>
+        </geometry>
+        <material name="">
+          <color rgba="0.7 0.7 0.7 1.0"/>
+        </material>
+      </visual>
+      <collision>
+        <origin rpy="0 0 0" xyz="0 0 0"/>
+        <geometry>
+          <mesh filename="file://$(find denso_description)/meshes/denso_base_link.STL" scale="1 1 1"/>
         </geometry>
       </collision>
@@ -50,14 +50,14 @@
         <origin rpy="0 0 0" xyz="0 0 0"/>
         <geometry>
-          <mesh filename="file://$(find denso_description)/robot/meshes/stl/denso_link1.STL" scale="1 1 1"/>
-        </geometry>
-        <material name="">
-          <color rgba="0.7 0.7 0.7 1.0"/>
-        </material>
-      </visual>
-      <collision>
-        <origin rpy="0 0 0" xyz="0 0 0"/>
-        <geometry>
-          <mesh filename="file://$(find denso_description)/robot/meshes/stl/denso_link1.STL" scale="1 1 1"/>
+          <mesh filename="file://$(find denso_description)/meshes/denso_link1.STL" scale="1 1 1"/>
+        </geometry>
+        <material name="">
+          <color rgba="0.7 0.7 0.7 1.0"/>
+        </material>
+      </visual>
+      <collision>
+        <origin rpy="0 0 0" xyz="0 0 0"/>
+        <geometry>
+          <mesh filename="file://$(find denso_description)/meshes/denso_link1.STL" scale="1 1 1"/>
         </geometry>
       </collision>
@@ -80,14 +80,14 @@
         <origin rpy="0 0 0" xyz="0 0 0"/>
         <geometry>
-          <mesh filename="file://$(find denso_description)/robot/meshes/stl/denso_link2.STL" scale="1 1 1"/>
-        </geometry>
-        <material name="">
-          <color rgba="0.7 0.7 0.7 1.0"/>
-        </material>
-      </visual>
-      <collision>
-        <origin rpy="0 0 0" xyz="0 0 0"/>
-        <geometry>
-          <mesh filename="file://$(find denso_description)/robot/meshes/stl/denso_link2.STL" scale="1 1 1"/>
+          <mesh filename="file://$(find denso_description)/meshes/denso_link2.STL" scale="1 1 1"/>
+        </geometry>
+        <material name="">
+          <color rgba="0.7 0.7 0.7 1.0"/>
+        </material>
+      </visual>
+      <collision>
+        <origin rpy="0 0 0" xyz="0 0 0"/>
+        <geometry>
+          <mesh filename="file://$(find denso_description)/meshes/denso_link2.STL" scale="1 1 1"/>
         </geometry>
       </collision>
@@ -110,14 +110,14 @@
         <origin rpy="0 0 0" xyz="0 0 0"/>
         <geometry>
-          <mesh filename="file://$(find denso_description)/robot/meshes/stl/denso_link3.STL" scale="1 1 1"/>
-        </geometry>
-        <material name="">
-          <color rgba="0.7 0.7 0.7 1.0"/>
-        </material>
-      </visual>
-      <collision>
-        <origin rpy="0 0 0" xyz="0 0 0"/>
-        <geometry>
-          <mesh filename="file://$(find denso_description)/robot/meshes/stl/denso_link3.STL" scale="1 1 1"/>
+          <mesh filename="file://$(find denso_description)/meshes/denso_link3.STL" scale="1 1 1"/>
+        </geometry>
+        <material name="">
+          <color rgba="0.7 0.7 0.7 1.0"/>
+        </material>
+      </visual>
+      <collision>
+        <origin rpy="0 0 0" xyz="0 0 0"/>
+        <geometry>
+          <mesh filename="file://$(find denso_description)/meshes/denso_link3.STL" scale="1 1 1"/>
         </geometry>
       </collision>
@@ -198,5 +198,5 @@
         <origin rpy="0 0 -1.57" xyz="0 0 0"/>
         <geometry>
-          <mesh filename="file://$(find denso_description)/robot/meshes/stl/denso_screwdriver.STL" scale="1 1 1"/>
+          <mesh filename="file://$(find denso_description)/meshes/denso_screwdriver.STL" scale="1 1 1"/>
         </geometry>
         <material name="">
@@ -207,5 +207,5 @@
         <origin rpy="0 0 -1.57" xyz="0 0 0"/>
         <geometry>
-          <mesh filename="file://$(find denso_description)/robot/meshes/stl/denso_screwdriver.STL" scale="1 1 1"/>
+          <mesh filename="file://$(find denso_description)/meshes/denso_screwdriver.STL" scale="1 1 1"/>
         </geometry>
       </collision>

File: src/denso/denso_description/urdf/denso_robot_macro.xacro (robot description, xacro)
@@ -28,9 +28,9 @@
   >
     <!-- Robot data required by the denso driver -->
-    <xacro:include filename="$(find denso_description)/robot/urdf/denso_robot_transmissions.xacro" />
+    <xacro:include filename="$(find denso_description)/urdf/denso_robot_transmissions.xacro" />
     <!-- robot kinematics include -->
-    <xacro:include filename="$(find denso_description)/robot/urdf/denso_robot_kinematics.xacro" />
+    <xacro:include filename="$(find denso_description)/urdf/denso_robot_kinematics.xacro" />
     <!-- ros2 control include -->
-    <xacro:include filename="$(find denso_description)/robot/urdf/denso_robot.ros2_control.xacro" />
+    <xacro:include filename="$(find denso_description)/urdf/denso_robot.ros2_control.xacro" />
     <!-- ros2 control instance -->
     <xacro:denso_robot_ros2_control
