Commit message: added controllers for supply x,y (direction needs to be fixed) , edited objects spawn position +40mm

File: src/descriptions/ur_description/urdf/inc/ur_transmissions.xacro (robot description, xacro)
@@ -128,4 +128,17 @@
       </actuator>
     </transmission>
+    <!-- Supply Joints -->
+    <transmission name="supply_y_axis_plate_trans">
+      <type>transmission_interface/SimpleTransmission</type>
+      <joint name="supply_y_axis_plate_joint">
+        <hardwareInterface>${hw_interface}</hardwareInterface>
+      </joint>
+    </transmission>
+    <transmission name="supply_x_axis_mobile_base_trans">
+      <type>transmission_interface/SimpleTransmission</type>
+      <joint name="supply_x_axis_mobile_base_joint">
+        <hardwareInterface>${hw_interface}</hardwareInterface>
+      </joint>
+    </transmission>
   </xacro:macro>
 </robot>

File: src/descriptions/ur_description/urdf/supply.xacro (robot description, xacro)
@@ -61,8 +61,10 @@
     </link>
     <!-- supply x axis mobile base to supply y axis plate joint (needs to be prismatic) **********-->
-    <joint name="supply_x_axis_mobile_base_supply_y_axis_plate_joint" type="fixed">
+    <joint name="supply_y_axis_plate_joint" type="prismatic">
       <parent link="supply_base_link" />
       <child link="supply_y_axis_plate_link" />
       <origin xyz="0.0 -0.98 0.0" rpy="0 0 0"/>
+      <axis xyz="-1 0 0"/>
+      <limit lower="-0.98" upper="0.98" effort="100" velocity="10" />
     </joint>
 <!-- supply x axis mobile base link -->
@@ -90,8 +92,10 @@
     </link>
       <!-- supply base to supply x axis mobile base joint (needs to be prismatic) **********-->
-  <joint name="supply_base_x_axis_mobile_base_joint" type="fixed">
+  <joint name="supply_x_axis_mobile_base_joint" type="prismatic">
       <parent link="supply_base_link" />
       <child link="supply_x_axis_mobile_base_link" />
       <origin xyz="0.0 0.0 0.01" rpy="0 0 0"/>
+      <axis xyz="0 0 1"/>
+      <limit lower="-0.98" upper="0.98" effort="100" velocity="10" />
     </joint>
 <!-- supply arm base link -->
@@ -116,5 +120,5 @@
     </link>
     <!-- supply y axis plate to supply arm base joint (needs to be prismatic??) **********-->
-    <joint name="supply_y_axis_plate_supply_arm_base_joint" type="fixed">
+    <joint name="supply_arm_base_joint" type="fixed">
       <parent link="supply_x_axis_mobile_base_link" />
       <child link="supply_arm_base_link" />
@@ -142,5 +146,5 @@
     </link>
     <!-- supply arm base to supply arm slider joint (needs to be prismatic??) **********-->
-    <joint name="supply_arm_base_supply_arm_slider_joint" type="fixed">
+    <joint name="supply_arm_slider_joint" type="fixed">
       <parent link="supply_arm_base_link" />
       <child link="supply_arm_slider_link" />
@@ -168,5 +172,5 @@
     </link>
     <!-- supply arm slider to supply arm plate joint (needs to be prismatic?? & need z offset) **********-->
-    <joint name="supply_arm_slider_supply_arm_plate_joint" type="fixed">
+    <joint name="supply_arm_plate_joint" type="fixed">
       <parent link="supply_arm_slider_link" />
       <child link="supply_arm_plate_link" />

File: src/descriptions/ur_description/urdf/ur.ros2_control.xacro (robot description, xacro)
@@ -234,4 +234,25 @@
           <!-- initial position for the FakeSystem and simulation -->
           <param name="initial_value">${initial_positions['denso_axis_joint']}</param>
+        </state_interface>
+        <state_interface name="velocity"/>
+        <state_interface name="effort"/>
+      </joint>
+      <!-- Supply Joints -->
+      <joint name="supply_y_axis_plate_joint">
+        <command_interface name="position"/>
+        <command_interface name="velocity"/>
+        <state_interface name="position">
+          <!-- initial position for the FakeSystem and simulation -->
+          <param name="initial_value">${initial_positions['supply_y_axis_plate_joint']}</param>
+        </state_interface>
+        <state_interface name="velocity"/>
+        <state_interface name="effort"/>
+      </joint>
+      <joint name="supply_x_axis_mobile_base_joint">
+        <command_interface name="position"/>
+        <command_interface name="velocity"/>
+        <state_interface name="position">
+          <!-- initial position for the FakeSystem and simulation -->
+          <param name="initial_value">${initial_positions['supply_x_axis_mobile_base_joint']}</param>
         </state_interface>
         <state_interface name="velocity"/>

Commit message: added controllers for supply arms

File: src/descriptions/ur_description/urdf/inc/ur_transmissions.xacro (robot description, xacro)
@@ -141,4 +141,22 @@
       </joint>
     </transmission>
+    <transmission name="supply_arm_base_trans">
+      <type>transmission_interface/SimpleTransmission</type>
+      <joint name="supply_arm_base_joint">
+        <hardwareInterface>${hw_interface}</hardwareInterface>
+      </joint>
+    </transmission>
+    <transmission name="supply_arm_slider_trans">
+      <type>transmission_interface/SimpleTransmission</type>
+      <joint name="supply_arm_slider_joint">
+        <hardwareInterface>${hw_interface}</hardwareInterface>
+      </joint>
+    </transmission>
+    <transmission name="supply_arm_plate_trans">
+      <type>transmission_interface/SimpleTransmission</type>
+      <joint name="supply_arm_plate_joint">
+        <hardwareInterface>${hw_interface}</hardwareInterface>
+      </joint>
+    </transmission>
   </xacro:macro>
 </robot>

File: src/descriptions/ur_description/urdf/supply.xacro (robot description, xacro)
@@ -60,10 +60,10 @@
       </inertial>
     </link>
-    <!-- supply x axis mobile base to supply y axis plate joint (needs to be prismatic) **********-->
+    <!-- supply base to supply y axis plate joint (needs to be prismatic) **********-->
     <joint name="supply_y_axis_plate_joint" type="prismatic">
       <parent link="supply_base_link" />
       <child link="supply_y_axis_plate_link" />
       <origin xyz="0.0 -0.98 0.0" rpy="0 0 0"/>
-      <axis xyz="-1 0 0"/>
+      <axis xyz="0 0 1"/>
       <limit lower="-0.98" upper="0.98" effort="100" velocity="10" />
     </joint>
@@ -96,5 +96,5 @@
       <child link="supply_x_axis_mobile_base_link" />
       <origin xyz="0.0 0.0 0.01" rpy="0 0 0"/>
-      <axis xyz="0 0 1"/>
+      <axis xyz="0 1 0"/>
       <limit lower="-0.98" upper="0.98" effort="100" velocity="10" />
     </joint>
@@ -120,8 +120,10 @@
     </link>
     <!-- supply y axis plate to supply arm base joint (needs to be prismatic??) **********-->
-    <joint name="supply_arm_base_joint" type="fixed">
+    <joint name="supply_arm_base_joint" type="prismatic">
       <parent link="supply_x_axis_mobile_base_link" />
       <child link="supply_arm_base_link" />
       <origin xyz="0.0 0.0 0.2566" rpy="0 0 0"/>
+      <axis xyz="0 0 1"/>
+      <limit lower="-0.98" upper="0.98" effort="100" velocity="10" />
     </joint>
 <!-- supply arm slider link -->
@@ -146,8 +148,10 @@
     </link>
     <!-- supply arm base to supply arm slider joint (needs to be prismatic??) **********-->
-    <joint name="supply_arm_slider_joint" type="fixed">
+    <joint name="supply_arm_slider_joint" type="prismatic">
       <parent link="supply_arm_base_link" />
       <child link="supply_arm_slider_link" />
       <origin xyz="0.0 0.0 0.0215" rpy="0 0 0"/>
+      <axis xyz="1 0 0"/>
+      <limit lower="-0.98" upper="0.98" effort="100" velocity="10" />
     </joint>
 <!-- supply arm plate link -->
@@ -172,8 +176,10 @@
     </link>
     <!-- supply arm slider to supply arm plate joint (needs to be prismatic?? & need z offset) **********-->
-    <joint name="supply_arm_plate_joint" type="fixed">
+    <joint name="supply_arm_plate_joint" type="prismatic">
       <parent link="supply_arm_slider_link" />
       <child link="supply_arm_plate_link" />
       <origin xyz="0.0 0.0 0.01" rpy="0 0 0"/>
+      <axis xyz="1 0 0"/>
+      <limit lower="-0.98" upper="0.98" effort="100" velocity="10" />
     </joint>
   </xacro:macro>

File: src/descriptions/ur_description/urdf/ur.ros2_control.xacro (robot description, xacro)
@@ -239,4 +239,5 @@
       </joint>
       <!-- Supply Joints -->
+      <!-- Supply Y Axis Plate Joint -->
       <joint name="supply_y_axis_plate_joint">
         <command_interface name="position"/>
@@ -249,4 +250,5 @@
         <state_interface name="effort"/>
       </joint>
+      <!-- Supply X Axis Mobile Base Joint -->
       <joint name="supply_x_axis_mobile_base_joint">
         <command_interface name="position"/>
@@ -255,4 +257,37 @@
           <!-- initial position for the FakeSystem and simulation -->
           <param name="initial_value">${initial_positions['supply_x_axis_mobile_base_joint']}</param>
+        </state_interface>
+        <state_interface name="velocity"/>
+        <state_interface name="effort"/>
+      </joint>
+      <!-- Supply Arm Base Joint -->
+      <joint name="supply_arm_base_joint">
+        <command_interface name="position"/>
+        <command_interface name="velocity"/>
+        <state_interface name="position">
+          <!-- initial position for the FakeSystem and simulation -->
+          <param name="initial_value">${initial_positions['supply_arm_base_joint']}</param>
+        </state_interface>
+        <state_interface name="velocity"/>
+        <state_interface name="effort"/>
+      </joint>
+      <!-- Supply Arm Slider Joint -->
+      <joint name="supply_arm_slider_joint">
+        <command_interface name="position"/>
+        <command_interface name="velocity"/>
+        <state_interface name="position">
+          <!-- initial position for the FakeSystem and simulation -->
+          <param name="initial_value">${initial_positions['supply_arm_slider_joint']}</param>
+        </state_interface>
+        <state_interface name="velocity"/>
+        <state_interface name="effort"/>
+      </joint>
+      <!-- Supply Arm Plate Joint -->
+      <joint name="supply_arm_plate_joint">
+        <command_interface name="position"/>
+        <command_interface name="velocity"/>
+        <state_interface name="position">
+          <!-- initial position for the FakeSystem and simulation -->
+          <param name="initial_value">${initial_positions['supply_arm_plate_joint']}</param>
         </state_interface>
         <state_interface name="velocity"/>

Commit message: gripper tips spawned - axis not properly configured yet

File: src/descriptions/ur_description/urdf/inc/ur_transmissions.xacro (robot description, xacro)
@@ -62,19 +62,19 @@
     </transmission>
     <!-- UR Robot Gripper Tooltips -->
-<transmission name="tooltip1_trans">
+<transmission name="tooltip_adapter1_trans">
   <type>transmission_interface/SimpleTransmission</type>
-  <joint name="tooltip1_joint">
+  <joint name="tooltip_adapter1_joint">
     <hardwareInterface>${hw_interface}</hardwareInterface>
   </joint>
-  <actuator name="tooltip1_motor">
+  <actuator name="tooltip_adapter1_motor">
     <mechanicalReduction>1</mechanicalReduction>
   </actuator>
 </transmission>
-<transmission name="tooltip2_trans">
+<transmission name="tooltip_adapter2_trans">
   <type>transmission_interface/SimpleTransmission</type>
-  <joint name="tooltip2_joint">
+  <joint name="tooltip_adapter2_joint">
     <hardwareInterface>${hw_interface}</hardwareInterface>
   </joint>
-  <actuator name="tooltip2_motor">
+  <actuator name="tooltip_adapter2_motor">
     <mechanicalReduction>1</mechanicalReduction>
   </actuator>

File: src/descriptions/ur_description/urdf/quickchanger_grippers.xacro (robot description, xacro)
@@ -52,31 +52,58 @@
       <origin xyz="0.1208 0.0019 0.1088" rpy="0 0.785 0"/>
     </joint>
-    <!-- tooltip_adapter_link -->
-    <link name="tooltip_adapter_link">
+    <!-- tooltip_adapter_1_link -->
+    <link name="tooltip_adapter_1_link">
+      <visual>
+        <origin xyz="0 0 0" rpy="0 0 3.14159"/>
+        <geometry>
+          <xacro:get_mesh name="tooltip_adapter_1" type="visual"/>
+        </geometry>
+        <material name="${sec_mesh_files['tooltip_adapter_1']['visual']['material']['name']}">
+          <color rgba="${sec_mesh_files['tooltip_adapter_1']['visual']['material']['color']}"/>
+        </material>
+      </visual>
+      <inertial>
+        <mass value="0.5"/>
+        <origin xyz="0 0 0" rpy="0 0 3.14159"/>
+        <inertia ixx="0.001" ixy="0" ixz="0" iyy="0.001" iyz="0" izz="0.001"/>
+      </inertial>
+    </link>
+    <!-- tooltip_adapter1_joint -->
+    <joint name="tooltip_adapter1_joint" type="prismatic">
+      <parent link="quickchanger_link"/>
+      <child link="tooltip_adapter_1_link"/>
+      <origin xyz="-0.1341 0.053 0.1221" rpy="0.785398 0 -1.5708"/>
+      <axis xyz="1 0 0"/>
+      <limit lower="-0.041" upper="0.041" effort="50" velocity="10"/>
+    </joint>
+    <!-- tooltip_adapter_2_link -->
+    <link name="tooltip_adapter_2_link">
       <visual>
         <origin xyz="0 0 0" rpy="0 0 0"/>
         <geometry>
-          <xacro:get_mesh name="tooltip_adapter" type="visual"/>
+          <xacro:get_mesh name="tooltip_adapter_2" type="visual"/>
         </geometry>
-        <material name="${sec_mesh_files['tooltip_adapter']['visual']['material']['name']}">
-          <color rgba="${sec_mesh_files['tooltip_adapter']['visual']['material']['color']}"/>
+        <material name="${sec_mesh_files['tooltip_adapter_2']['visual']['material']['name']}">
+          <color rgba="${sec_mesh_files['tooltip_adapter_2']['visual']['material']['color']}"/>
         </material>
       </visual>
       <inertial>
-        <mass value="1.0"/>
+        <mass value="0.5"/>
         <origin xyz="0 0 0" rpy="0 0 0"/>
-        <inertia ixx="1e-5" ixy="0" ixz="0" iyy="1e-5" iyz="0" izz="1e-5"/>
+        <inertia ixx="0.001" ixy="0" ixz="0" iyy="0.001" iyz="0" izz="0.001"/>
       </inertial>
     </link>
-    <!-- tooltip_adapter_joint -->
-    <joint name="tooltip_adapter_joint" type="fixed">
+    <!-- tooltip_adapter_2_joint -->
+    <joint name="tooltip_adapter2_joint" type="prismatic">
       <parent link="quickchanger_link"/>
-      <child link="tooltip_adapter_link"/>
-      <origin xyz="-0.1341 0.053 0.1221" rpy="-0.785 0 1.57"/>
+      <child link="tooltip_adapter_2_link"/>
+      <origin xyz="-0.1341 -0.053 0.1221" rpy="0.785398 0 -1.5708"/>
+      <axis xyz="0 1 0"/>
+      <limit lower="-0.041" upper="0.041" effort="50" velocity="10"/>
     </joint>
     <!-- tooltip1_link -->
     <link name="tooltip1_link">
       <visual>
-        <origin xyz="0 0 0" rpy="0 0 0"/>
+        <origin xyz="0 0 0" rpy="0 0 1.5708"/>
         <geometry>
           <xacro:get_mesh name="tooltip1" type="visual"/>
@@ -88,20 +115,18 @@
       <inertial>
         <mass value="0.5"/>
-        <origin xyz="0 0 0" rpy="0 0 0"/>
+        <origin xyz="0 0 0" rpy="0 0 1.5708"/>
         <inertia ixx="0.001" ixy="0" ixz="0" iyy="0.001" iyz="0" izz="0.001"/>
       </inertial>
     </link>
     <!-- tooltip1_joint -->
-    <joint name="tooltip1_joint" type="prismatic">
-      <parent link="tooltip_adapter_link"/>
+    <joint name="tooltip1_joint" type="fixed">
+      <parent link="tooltip_adapter_1_link"/>
       <child link="tooltip1_link"/>
       <origin xyz="-0.002 0 0.04" rpy="0 0 0"/>
-      <axis xyz="1 0 0"/>
-      <limit lower="-1.0" upper="0.041" effort="50" velocity="10"/>
     </joint>
-    <!-- tooltip2 -->
+    <!-- tooltip2_link -->
     <link name="tooltip2_link">
       <visual>
-        <origin xyz="0 0 0" rpy="0 0 0"/>
+        <origin xyz="0 0 0" rpy="0 0 1.5708"/>
         <geometry>
           <xacro:get_mesh name="tooltip2" type="visual"/>
@@ -113,14 +138,13 @@
       <inertial>
         <mass value="0.5"/>
-        <origin xyz="0 0 0" rpy="0 0 0"/>
+        <origin xyz="0 0 0" rpy="0 0 1.5708"/>
         <inertia ixx="0.001" ixy="0" ixz="0" iyy="0.001" iyz="0" izz="0.001"/>
       </inertial>
     </link>
-    <joint name="tooltip2_joint" type="prismatic">
-      <parent link="tooltip_adapter_link"/>
+    <!-- tooltip2_joint -->
+    <joint name="tooltip2_joint" type="fixed">
+      <parent link="tooltip_adapter_2_link"/>
       <child link="tooltip2_link"/>
       <origin xyz="0.002 0 0.04" rpy="0 0 3.14"/>
-      <axis xyz="1 0 0"/>
-      <limit lower="-1.0" upper="0.041" effort="50" velocity="10"/>
     </joint>
   </xacro:macro>

File: src/descriptions/ur_description/urdf/ur.ros2_control.xacro (robot description, xacro)
@@ -126,18 +126,18 @@
       </joint>
       <!-- UR Robot Gripper Tooltips -->
-      <joint name="${tf_prefix}tooltip1_joint">
-        <command_interface name="position"/>
-        <state_interface name="position">
-          <!-- initial position for the FakeSystem and simulation -->
-          <param name="initial_value">${initial_positions['tooltip1_joint']}</param>
-        </state_interface>
-        <state_interface name="velocity"/>
-        <state_interface name="effort"/>
-      </joint>
-      <joint name="${tf_prefix}tooltip2_joint">
-        <command_interface name="position"/>
-        <state_interface name="position">
-          <!-- initial position for the FakeSystem and simulation -->
-          <param name="initial_value">${initial_positions['tooltip2_joint']}</param>
+      <joint name="${tf_prefix}tooltip_adapter1_joint">
+        <command_interface name="position"/>
+        <state_interface name="position">
+          <!-- initial position for the FakeSystem and simulation -->
+          <param name="initial_value">${initial_positions['tooltip_adapter1_joint']}</param>
+        </state_interface>
+        <state_interface name="velocity"/>
+        <state_interface name="effort"/>
+      </joint>
+      <joint name="${tf_prefix}tooltip_adapter2_joint">
+        <command_interface name="position"/>
+        <state_interface name="position">
+          <!-- initial position for the FakeSystem and simulation -->
+          <param name="initial_value">${initial_positions['tooltip_adapter2_joint']}</param>
         </state_interface>
         <state_interface name="velocity"/>
