Commit message: replaced toolchanger stl

File: src/descriptions/ur_description/urdf/toolchanger.xacro (robot description, xacro)
@@ -64,5 +64,5 @@
       <parent link="toolchanger_trolley_link" />
       <child link="tool_changer_link" />
-      <origin xyz="0.2 0.15 0.0" rpy="0 0 0"/>
+      <origin xyz="0.3 0.0 0.0" rpy="0 0 0"/>
     </joint>
   </xacro:macro>
