Commit message: spawn supply base + mobile + yaxis plate+ arm - controllers not set yet

File: src/descriptions/ur_description/urdf/gazebo_materials.xacro (robot description, xacro)
@@ -141,3 +141,23 @@
     <preserveFixedJoint>true</preserveFixedJoint>
   </gazebo>
+  <!-- Supply Link Components -->
+  <gazebo reference="supply_base_link">
+    <material>Gazebo/LightGrey</material>
+  </gazebo>
+  <gazebo reference="supply_x_axis_mobile_base_link">
+    <material>Gazebo/Grey</material>
+  </gazebo>
+  <gazebo reference="supply_y_axis_plate_link">
+    <material>Gazebo/Grey</material>
+  </gazebo>
+  <!-- Supply Joint Components -->
+  <gazebo reference="supply_base_joint">
+    <preserveFixedJoint>true</preserveFixedJoint>
+  </gazebo>
+  <gazebo reference="supply_x_axis_mobile_base_joint">
+    <preserveFixedJoint>true</preserveFixedJoint>
+  </gazebo>
+  <gazebo reference="supply_y_axis_plate_joint">
+    <preserveFixedJoint>true</preserveFixedJoint>
+  </gazebo>
 </robot>

File: src/descriptions/ur_description/urdf/quickchanger_grippers.xacro (robot description, xacro)
@@ -2,5 +2,5 @@
 <robot xmlns:xacro="http://wiki.ros.org/xacro">
   <xacro:macro name="quickchanger_grippers" params="parent">
-  <xacro:property name="quickchanger_grippers_visual_params" value="${xacro.load_yaml('$(find ur_description)/config/quickchanger_grippers.yaml')}"/>
+  <xacro:property name="quickchanger_grippers_visual_params" value="${xacro.load_yaml('$(find ur_description)/config/quickchanger_grippers_visual_parameters.yaml')}"/>
   <xacro:property name="sec_mesh_files" value="${quickchanger_grippers_visual_params['mesh_files']}" scope="parent"/>
   <xacro:property name="force_abs_paths" value="true" scope="parent"/>

File: src/descriptions/ur_description/urdf/ur.urdf.xacro (robot description, xacro)
@@ -15,4 +15,6 @@
    <!-- import denso macro -->
    <xacro:include filename="$(find ur_description)/urdf/denso.xacro"/>
+   <!-- import supply macro -->
+   <xacro:include filename="$(find ur_description)/urdf/supply.xacro"/>
    <!-- import gazebo materials -->
    <xacro:include filename="$(find ur_description)/urdf/gazebo_materials.xacro"/>
@@ -97,4 +99,6 @@
   <!-- denso components -->
   <xacro:denso parent="world"/>
+  <!-- supply components -->
+  <xacro:supply parent="world"/>
    <!-- Load trolley positions configuration -->
    <xacro:property name="trolley_positions" value="${xacro.load_yaml('$(find ur_description)/config/trolley_positions.yaml')}"/>

Commit message: add gazebo materials xacro for supply components

File: src/descriptions/ur_description/urdf/gazebo_materials.xacro (robot description, xacro)
@@ -151,4 +151,13 @@
     <material>Gazebo/Grey</material>
   </gazebo>
+  <gazebo reference="supply_arm_base_link">
+    <material>Gazebo/LightGrey</material>
+  </gazebo>
+  <gazebo reference="supply_arm_slider_link">
+    <material>Gazebo/Yellow</material>
+  </gazebo>
+  <gazebo reference="supply_arm_plate_link">
+    <material>Gazebo/Green</material>
+  </gazebo>
   <!-- Supply Joint Components -->
   <gazebo reference="supply_base_joint">
@@ -161,3 +170,15 @@
     <preserveFixedJoint>true</preserveFixedJoint>
   </gazebo>
+  <gazebo reference="supply_y_axis_plate_supply_arm_base_joint">
+    <preserveFixedJoint>true</preserveFixedJoint>
+  </gazebo>
+  <gazebo reference="supply_arm_base_supply_arm_slider_joint">
+    <preserveFixedJoint>true</preserveFixedJoint>
+  </gazebo>
+  <gazebo reference="supply_arm_slider_supply_arm_plate_joint">
+    <preserveFixedJoint>true</preserveFixedJoint>
+  </gazebo>
+  <gazebo reference="supply_arm_plate_supply_arm_joint">
+    <preserveFixedJoint>true</preserveFixedJoint>
+  </gazebo>
 </robot>

File: src/descriptions/ur_description/urdf/supply.xacro (robot description, xacro)
@@ -167,9 +167,9 @@
       </inertial>
     </link>
-    <!-- supply arm slider to supply arm plate joint (needs to be prismatic??) **********-->
+    <!-- supply arm slider to supply arm plate joint (needs to be prismatic?? & need z offset) **********-->
     <joint name="supply_arm_slider_supply_arm_plate_joint" type="fixed">
       <parent link="supply_arm_slider_link" />
       <child link="supply_arm_plate_link" />
-      <origin xyz="0.0 0.0 0.0" rpy="0 0 0"/>
+      <origin xyz="0.0 0.0 0.01" rpy="0 0 0"/>
     </joint>
   </xacro:macro>

Commit message: added elec arf (fixed joints yet) + matched rviz and gazebo colours

File: src/descriptions/ur_description/urdf/gazebo_materials.xacro (robot description, xacro)
@@ -95,5 +95,5 @@
   </gazebo>
   <gazebo reference="tool_changer_link">
-    <material>Gazebo/Blue</material>
+    <material>Gazebo/Yellow</material>
   </gazebo>
   <!-- Toolchanger Joint Components -->
@@ -115,8 +115,8 @@
   </gazebo>
   <gazebo reference="arf_front_aircyl_link">
-    <material>Gazebo/Yellow</material>
+    <material>Gazebo/Green</material>
   </gazebo>
   <gazebo reference="arf_back_aircyl_link">
-    <material>Gazebo/Yellow</material>
+    <material>Gazebo/Green</material>
   </gazebo>
   <!-- ARF Joint Components -->
@@ -127,4 +127,45 @@
     <preserveFixedJoint>true</preserveFixedJoint>
   </gazebo>
+  <!-- ARF Elec Link Components -->
+  <gazebo reference="arf_elec_trolley_link">
+    <material>Gazebo/LightGrey</material>
+  </gazebo>
+  <gazebo reference="arf_elec_x_axis_link">
+    <material>Gazebo/Blue</material>
+  </gazebo>
+  <gazebo reference="arf_elec_y_axis_link">
+    <material>Gazebo/Blue</material>
+  </gazebo>
+  <gazebo reference="arf_elec_jig_link">
+    <material>Gazebo/Blue</material>
+  </gazebo>
+  <gazebo reference="arf_elec_aircyl_1_link">
+    <material>Gazebo/Blue</material>
+  </gazebo>
+  <gazebo reference="arf_elec_aircyl_1_2_link">
+    <material>Gazebo/Blue</material>
+  </gazebo>
+  <gazebo reference="arf_elec_aircyl_2_link">
+    <material>Gazebo/Blue</material>
+  </gazebo>
+  <!-- ARF Elec Joint Components -->
+  <gazebo reference="arf_elec_x_axis_joint">
+    <preserveFixedJoint>true</preserveFixedJoint>
+  </gazebo>
+  <gazebo reference="arf_elec_y_axis_joint">
+    <preserveFixedJoint>true</preserveFixedJoint>
+  </gazebo>
+  <gazebo reference="arf_elec_jig_joint">
+    <preserveFixedJoint>true</preserveFixedJoint>
+  </gazebo>
+  <gazebo reference="arf_elec_aircyl_1_joint">
+    <preserveFixedJoint>true</preserveFixedJoint>
+  </gazebo>
+  <gazebo reference="arf_elec_aircyl_1_2_joint">
+    <preserveFixedJoint>true</preserveFixedJoint>
+  </gazebo>
+  <gazebo reference="arf_elec_aircyl_2_joint">
+    <preserveFixedJoint>true</preserveFixedJoint>
+  </gazebo>
   <!-- Denso Link Components -->
   <gazebo reference="denso_trolley_link">
@@ -152,11 +193,11 @@
   </gazebo>
   <gazebo reference="feeder_arm_base_link">
-    <material>Gazebo/LightGrey</material>
+    <material>Gazebo/Grey</material>
   </gazebo>
   <gazebo reference="feeder_arm_slider_link">
-    <material>Gazebo/Yellow</material>
+    <material>Gazebo/Grey</material>
   </gazebo>
   <gazebo reference="feeder_arm_plate_link">
-    <material>Gazebo/Green</material>
+    <material>Gazebo/Grey</material>
   </gazebo>
   <!-- Supply Joint Components -->

File: src/descriptions/ur_description/urdf/ur.urdf.xacro (robot description, xacro)
@@ -13,4 +13,6 @@
    <!-- import arf macro -->
    <xacro:include filename="$(find ur_description)/urdf/arf.xacro"/>
+   <!-- import arf_elec macro -->
+   <xacro:include filename="$(find ur_description)/urdf/arf_elec.xacro"/>
    <!-- import denso macro -->
    <xacro:include filename="$(find ur_description)/urdf/denso.xacro"/>
@@ -97,4 +99,6 @@
   <!-- arf components -->
   <xacro:arf parent="world"/>
+  <!-- arf_elec components -->
+  <xacro:arf_elec parent="world"/>
   <!-- denso components -->
   <xacro:denso parent="world"/>
