Commit message: removed collision from arf slide (+edited kinematics for ur to have more time for ik)

File: src/descriptions/ur_description/urdf/arf.xacro (robot description, xacro)
@@ -103,10 +103,4 @@
         </material>
       </visual>
-      <collision>
-        <origin xyz="0 0 0" rpy="0 0 0"/>
-        <geometry>
-          <xacro:get_mesh name="arf_slider" type="collision"/>
-        </geometry>
-      </collision>
       <inertial>
         <mass value="1.0"/>

Commit message: added trolley_positions.yaml for separate trolley position spawning later on

File: src/descriptions/ur_description/urdf/arf.xacro (robot description, xacro)
@@ -5,4 +5,7 @@
   <xacro:property name="sec_mesh_files" value="${arf_visual_params['mesh_files']}" scope="parent"/>
   <xacro:property name="force_abs_paths" value="true" scope="parent"/>
+  <!-- Load trolley positions configuration -->
+  <xacro:property name="trolley_positions" value="${xacro.load_yaml('$(find ur_description)/config/trolley_positions.yaml')}"/>
+  <xacro:property name="arf_pos" value="${trolley_positions['trolley_positions']['arf']}"/>
 <!-- arf trolley link -->
     <link name="arf_trolley_link">
@@ -32,5 +35,5 @@
       <parent link="${parent}" />
       <child link="arf_trolley_link" />
-      <origin xyz="0 0.805 0" rpy="0 0 0"/>
+      <origin xyz="${arf_pos['x']} ${arf_pos['y']} ${arf_pos['z']}" rpy="${arf_pos['roll']} ${arf_pos['pitch']} ${arf_pos['yaw']}"/>
     </joint>
 <!-- arf base plate link -->

File: src/descriptions/ur_description/urdf/denso.xacro (robot description, xacro)
@@ -7,4 +7,7 @@
   <xacro:property name="sec_mesh_files" value="${denso_visual_params['mesh_files']}" scope="parent"/>
   <xacro:property name="force_abs_paths" value="true" scope="parent"/>
+  <!-- Load trolley positions configuration -->
+  <xacro:property name="trolley_positions" value="${xacro.load_yaml('$(find ur_description)/config/trolley_positions.yaml')}"/>
+  <xacro:property name="denso_pos" value="${trolley_positions['trolley_positions']['denso']}"/>
 <!-- denso trolley link -->
     <link name="denso_trolley_link">
@@ -34,5 +37,5 @@
       <parent link="${parent}" />
       <child link="denso_trolley_link" />
-      <origin xyz="-0.8049 0.805 0" rpy="0 0 0"/>
+      <origin xyz="${denso_pos['x']} ${denso_pos['y']} ${denso_pos['z']}" rpy="${denso_pos['roll']} ${denso_pos['pitch']} ${denso_pos['yaw']}"/>
     </joint>
 <!-- denso slider jig link -->

File: src/descriptions/ur_description/urdf/toolchanger.xacro (robot description, xacro)
@@ -5,4 +5,7 @@
   <xacro:property name="sec_mesh_files" value="${toolchanger_visual_params['mesh_files']}" scope="parent"/>
   <xacro:property name="force_abs_paths" value="true" scope="parent"/>
+  <!-- Load trolley positions configuration -->
+  <xacro:property name="trolley_positions" value="${xacro.load_yaml('$(find ur_description)/config/trolley_positions.yaml')}"/>
+  <xacro:property name="toolchanger_pos" value="${trolley_positions['trolley_positions']['toolchanger']}"/>
 <!-- toolchanger trolley link -->
     <link name="toolchanger_trolley_link">
@@ -32,5 +35,5 @@
       <parent link="${parent}" />
       <child link="toolchanger_trolley_link" />
-      <origin xyz="-0.8049 0 0" rpy="0 0 0"/>
+      <origin xyz="${toolchanger_pos['x']} ${toolchanger_pos['y']} ${toolchanger_pos['z']}" rpy="${toolchanger_pos['roll']} ${toolchanger_pos['pitch']} ${toolchanger_pos['yaw']}"/>
     </joint>
 <!-- toolchanger tool stand link -->

File: src/descriptions/ur_description/urdf/ur.urdf.xacro (robot description, xacro)
@@ -93,8 +93,11 @@
   <!-- toolchanger components -->
   <xacro:toolchanger parent="world"/>
-   <!-- arf components -->
-   <xacro:arf parent="world"/>
-   <!-- denso components -->
-   <xacro:denso parent="world"/>
+  <!-- arf components -->
+  <xacro:arf parent="world"/>
+  <!-- denso components -->
+  <xacro:denso parent="world"/>
+   <!-- Load trolley positions configuration -->
+   <xacro:property name="trolley_positions" value="${xacro.load_yaml('$(find ur_description)/config/trolley_positions.yaml')}"/>
+   <xacro:property name="ur_pos" value="${trolley_positions['trolley_positions']['ur']}"/>
    <!-- arm -->
    <xacro:ur_robot
@@ -136,5 +139,5 @@
      trajectory_port="$(arg trajectory_port)"
      >
-     <origin xyz="0 0 0" rpy="0 0 0" />          <!-- position robot in the world -->
+     <origin xyz="${ur_pos['x']} ${ur_pos['y']} ${ur_pos['z']}" rpy="${ur_pos['roll']} ${ur_pos['pitch']} ${ur_pos['yaw']}" />
    </xacro:ur_robot>
      <!-- attach gripper -->

File: src/descriptions/ur_description/urdf/vision.xacro (robot description, xacro)
@@ -5,4 +5,7 @@
     <xacro:property name="sec_mesh_files" value="${vision_visual_params['mesh_files']}" scope="parent"/>
     <xacro:property name="force_abs_paths" value="true" scope="parent"/>
+    <!-- Load trolley positions configuration -->
+    <xacro:property name="trolley_positions" value="${xacro.load_yaml('$(find ur_description)/config/trolley_positions.yaml')}"/>
+    <xacro:property name="vision_pos" value="${trolley_positions['trolley_positions']['vision']}"/>
     <!-- vision trolley link -->
     <link name="vision_trolley_link">
@@ -32,5 +35,5 @@
       <parent link="${parent}" />
       <child link="vision_trolley_link" />
-      <origin xyz="0 1.605 0" rpy="0 0 0"/>
+      <origin xyz="${vision_pos['x']} ${vision_pos['y']} ${vision_pos['z']}" rpy="${vision_pos['roll']} ${vision_pos['pitch']} ${vision_pos['yaw']}"/>
     </joint>
     <!-- vision cam jig link -->

Commit message: Replaced Trolleys and ARF components - LFS used for large files

File: src/descriptions/ur_description/urdf/arf.xacro (robot description, xacro)
@@ -20,7 +20,7 @@
       </visual>
       <collision>
-        <origin xyz="0 0 0" rpy="0 0 0"/>
-        <geometry>
-          <xacro:get_mesh name="arf_trolley" type="collision"/>
+        <origin xyz="${sec_mesh_files['arf_trolley']['collision']['box']['origin']}" rpy="0 0 0"/>
+        <geometry>
+          <box size="${sec_mesh_files['arf_trolley']['collision']['box']['size']}"/>
         </geometry>
       </collision>
@@ -37,19 +37,19 @@
       <origin xyz="${arf_pos['x']} ${arf_pos['y']} ${arf_pos['z']}" rpy="${arf_pos['roll']} ${arf_pos['pitch']} ${arf_pos['yaw']}"/>
     </joint>
-<!-- arf base plate link -->
-    <link name="arf_base_plate_link">
-      <visual>
-        <origin xyz="0 0 0" rpy="0 0 0"/>
-        <geometry>
-          <xacro:get_mesh name="arf_base_plate" type="visual"/>
-        </geometry>
-        <material name="${sec_mesh_files['arf_base_plate']['visual']['material']['name']}">
-          <color rgba="${sec_mesh_files['arf_base_plate']['visual']['material']['color']}"/>
-        </material>
-      </visual>
-      <collision>
-        <origin xyz="0 0 0" rpy="0 0 0"/>
-        <geometry>
-          <xacro:get_mesh name="arf_base_plate" type="collision"/>
+<!-- arf x axis link -->
+    <link name="arf_x_axis_link">
+      <visual>
+        <origin xyz="0 0 0" rpy="0 0 0"/>
+        <geometry>
+          <xacro:get_mesh name="arf_x_axis" type="visual"/>
+        </geometry>
+        <material name="${sec_mesh_files['arf_x_axis']['visual']['material']['name']}">
+          <color rgba="${sec_mesh_files['arf_x_axis']['visual']['material']['color']}"/>
+        </material>
+      </visual>
+      <collision>
+        <origin xyz="0 0 0" rpy="0 0 0"/>
+        <geometry>
+          <xacro:get_mesh name="arf_x_axis" type="collision"/>
         </geometry>
       </collision>
@@ -60,25 +60,25 @@
       </inertial>
     </link>
-    <!-- trolley to arf base jig joint -->
-    <joint name="arf_base_plate_joint" type="fixed">
+    <!-- trolley to arf x axis joint -->
+    <joint name="arf_x_axis_joint" type="fixed">
       <parent link="arf_trolley_link" />
-      <child link="arf_base_plate_link" />
-      <origin xyz="0.37 -0.385 0.820" rpy="0 0 0"/>
-    </joint>
-<!-- arf slider base link -->
-    <link name="arf_slider_base_link">
-      <visual>
-        <origin xyz="0 0 0" rpy="0 0 0"/>
-        <geometry>
-          <xacro:get_mesh name="arf_slider_base" type="visual"/>
-        </geometry>
-        <material name="${sec_mesh_files['arf_slider_base']['visual']['material']['name']}">
-          <color rgba="${sec_mesh_files['arf_slider_base']['visual']['material']['color']}"/>
-        </material>
-      </visual>
-      <collision>
-        <origin xyz="0 0 0" rpy="0 0 0"/>
-        <geometry>
-          <xacro:get_mesh name="arf_slider_base" type="collision"/>
+      <child link="arf_x_axis_link" />
+      <origin xyz="0.37 -0.2975 0.0" rpy="0 0 0"/>
+    </joint>
+    <!-- arf y axis link (slider) -->
+    <link name="arf_y_axis_link">
+      <visual>
+        <origin xyz="0 0 0" rpy="0 0 0"/>
+        <geometry>
+          <xacro:get_mesh name="arf_y_axis" type="visual"/>
+        </geometry>
+        <material name="${sec_mesh_files['arf_y_axis']['visual']['material']['name']}">
+          <color rgba="${sec_mesh_files['arf_y_axis']['visual']['material']['color']}"/>
+        </material>
+      </visual>
+      <collision>
+        <origin xyz="0 0 0" rpy="0 0 0"/>
+        <geometry>
+          <xacro:get_mesh name="arf_y_axis" type="collision"/>
         </geometry>
       </collision>
@@ -89,37 +89,14 @@
       </inertial>
     </link>
-    <!-- arf base plate to arf slider base joint -->
-    <joint name="arf_slider_base_joint" type="fixed">
-      <parent link="arf_base_plate_link" />
-      <child link="arf_slider_base_link" />
-      <origin xyz="-0.03426 0.0375 0.014" rpy="0 0 0"/>
-    </joint>
-    <!-- arf slider link -->
-    <link name="arf_slider_link">
-      <visual>
-        <origin xyz="0 0 0" rpy="0 0 0"/>
-        <geometry>
-          <xacro:get_mesh name="arf_slider" type="visual"/>
-        </geometry>
-        <material name="${sec_mesh_files['arf_slider']['visual']['material']['name']}">
-          <color rgba="${sec_mesh_files['arf_slider']['visual']['material']['color']}"/>
-        </material>
-      </visual>
-      <inertial>
-        <mass value="1.0"/>
-        <origin xyz="0 0 0" rpy="0 0 0"/>
-        <inertia ixx="0.001" ixy="0" ixz="0" iyy="0.001" iyz="0" izz="0.001"/>
-      </inertial>
-    </link>
-    <!-- ** arf_axis_1_joint ** arf slider base to slider joint -->
+    <!-- arf_x_axis to arf_y_axis joint (prismatic) -->
     <joint name="arf_axis_1_joint" type="prismatic">
-      <parent link="arf_slider_base_link" />
-      <child link="arf_slider_link" />
-      <origin xyz="-0.12 0 0.04" rpy="0 0 0"/>
+      <parent link="arf_x_axis_link" />
+      <child link="arf_y_axis_link" />
+      <origin xyz="-0.360 0.0 0.054" rpy="0 0 0"/>
       <axis xyz="-1 0 0"/>
       <limit lower="0.0" upper="0.35" effort="100" velocity="10" />
     </joint>
-  <!-- dummy link for slider and jig joints -->
-    <link name = "arf_slider_dummy_link">
+  <!-- dummy link for jig joint -->
+    <link name = "arf_jig_dummy_link">
       <inertial>
         <mass value="0.001"/>
@@ -128,25 +105,25 @@
       </inertial>
     </link>
-      <!-- slider to dummy link joint -->
-    <joint name="arf_slider_dummy_joint" type="fixed">
-      <parent link="arf_slider_link" />
-      <child link="arf_slider_dummy_link" />
+      <!-- y axis to dummy link joint -->
+    <joint name="arf_jig_dummy_joint" type="fixed">
+      <parent link="arf_y_axis_link" />
+      <child link="arf_jig_dummy_link" />
       <origin xyz="0 0 0" rpy="0 0 0"/>
     </joint>
-    <!-- arf slider jig link -->
-    <link name="arf_slider_jig_link">
-      <visual>
-        <origin xyz="0 0 0" rpy="0 0 0"/>
-        <geometry>
-          <xacro:get_mesh name="arf_slider_jig" type="visual"/>
-        </geometry>
-        <material name="${sec_mesh_files['arf_slider_jig']['visual']['material']['name']}">
-          <color rgba="${sec_mesh_files['arf_slider_jig']['visual']['material']['color']}"/>
-        </material>
-      </visual>
-      <collision>
-        <origin xyz="0 0 0" rpy="0 0 0"/>
-        <geometry>
-          <xacro:get_mesh name="arf_slider_jig" type="collision"/>
+    <!-- arf jig link -->
+    <link name="arf_jig_link">
+      <visual>
+        <origin xyz="0 0 0" rpy="0 0 0"/>
+        <geometry>
+          <xacro:get_mesh name="arf_jig" type="visual"/>
+        </geometry>
+        <material name="${sec_mesh_files['arf_jig']['visual']['material']['name']}">
+          <color rgba="${sec_mesh_files['arf_jig']['visual']['material']['color']}"/>
+        </material>
+      </visual>
+      <collision>
+        <origin xyz="0 0 0" rpy="0 0 0"/>
+        <geometry>
+          <xacro:get_mesh name="arf_jig" type="collision"/>
         </geometry>
       </collision>
@@ -157,13 +134,13 @@
       </inertial>
     </link>
-    <!-- ** arf_axis_2_joint **arf slider dummy to slider jig joint -->
+    <!-- arf_y_axis to arf_jig joint (prismatic) -->
     <joint name="arf_axis_2_joint" type="prismatic">
-      <parent link="arf_slider_dummy_link" />
-      <child link="arf_slider_jig_link" />
-      <origin xyz="0 0.4185 0.107" rpy="0 0 0"/>
+      <parent link="arf_jig_dummy_link" />
+      <child link="arf_jig_link" />
+      <origin xyz="0 0.300 0.107" rpy="0 0 0"/>
       <axis xyz="0 1 0"/>
       <limit lower="-0.25" upper="0" effort="100" velocity="10" />
     </joint>
-    <!-- dummy link for slider and jig joints -->
+    <!-- dummy link for aircyl joints -->
     <link name = "arf_aircyl_dummy_link">
       <inertial>
@@ -173,7 +150,7 @@
       </inertial>
     </link>
-      <!-- slider to dummy link joint -->
+      <!-- jig to dummy link joint -->
     <joint name="arf_aircyl_dummy_joint" type="fixed">
-      <parent link="arf_slider_jig_link" />
+      <parent link="arf_jig_link" />
       <child link="arf_aircyl_dummy_link" />
       <origin xyz="0 0 0" rpy="0 0 0"/>
@@ -202,9 +179,9 @@
       </inertial>
     </link>
-    <!-- arf slider jig to front aircyl joint ****** PRISMATIC ****** -->
+    <!-- arf jig to front aircyl joint (prismatic) -->
     <joint name="arf_gripper_joint_1" type="prismatic">
       <parent link="arf_aircyl_dummy_link" />
       <child link="arf_front_aircyl_link" />
-      <origin xyz="0.226 0.0 0.065" rpy="0 0 0"/>
+      <origin xyz="0.211 0.0 0.065" rpy="0 0 0"/>
       <axis xyz="1 0 0"/>
       <limit lower="-0.25" upper="1.0" effort="100" velocity="10" />
@@ -233,9 +210,9 @@
       </inertial>
     </link>
-    <!-- arf slider jig to front aircyl joint ****** PRISMATIC ****** -->
+    <!-- arf jig to back aircyl joint (prismatic) -->
     <joint name="arf_gripper_joint_2" type="prismatic">
       <parent link="arf_aircyl_dummy_link" />
       <child link="arf_back_aircyl_link" />
-      <origin xyz="-0.226 0.0 0.065" rpy="0 0 0"/>
+      <origin xyz="-0.211 0.0 0.065" rpy="0 0 0"/>
       <axis xyz="1 0 0"/>
       <limit lower="-0.25" upper="1.0" effort="100" velocity="10" />

File: src/descriptions/ur_description/urdf/denso.xacro (robot description, xacro)
@@ -22,7 +22,7 @@
       </visual>
       <collision>
-        <origin xyz="0 0 0" rpy="0 0 0"/>
+        <origin xyz="${sec_mesh_files['denso_trolley']['collision']['box']['origin']}" rpy="0 0 0"/>
         <geometry>
-          <xacro:get_mesh name="denso_trolley" type="collision"/>
+          <box size="${sec_mesh_files['denso_trolley']['collision']['box']['size']}"/>
         </geometry>
       </collision>
@@ -66,5 +66,5 @@
       <parent link="denso_trolley_link" />
       <child link="denso_slider_jig_link" />
-      <origin xyz="0.025 -0.025 0.82" rpy="0 0 0"/>
+      <origin xyz="0.025 -0.025 0.0" rpy="0 0 0"/>
     </joint>
     <!-- Add Denso robot connected to the slider jig -->

File: src/descriptions/ur_description/urdf/gazebo_materials.xacro (robot description, xacro)
@@ -105,15 +105,12 @@
     <material>Gazebo/LightGrey</material>
   </gazebo>
-  <gazebo reference="arf_base_plate_link">
-    <material>Gazebo/DarkGrey</material>
-  </gazebo>
-  <gazebo reference="arf_slider_base_link">
+  <gazebo reference="arf_x_axis_link">
     <material>Gazebo/Grey</material>
   </gazebo>
-  <gazebo reference="arf_slider_link">
+  <gazebo reference="arf_y_axis_link">
+    <material>Gazebo/Grey</material>
+  </gazebo>
+  <gazebo reference="arf_jig_link">
     <material>Gazebo/Green</material>
-  </gazebo>
-  <gazebo reference="arf_slider_jig_link">
-    <material>Gazebo/Yellow</material>
   </gazebo>
   <gazebo reference="arf_front_aircyl_link">
@@ -124,8 +121,8 @@
   </gazebo>
   <!-- ARF Joint Components -->
-  <gazebo reference="arf_base_plate_joint">
+  <gazebo reference="arf_x_axis_joint">
     <preserveFixedJoint>true</preserveFixedJoint>
   </gazebo>
-  <gazebo reference="arf_slider_base_joint">
+  <gazebo reference="arf_y_axis_joint">
     <preserveFixedJoint>true</preserveFixedJoint>
   </gazebo>

File: src/descriptions/ur_description/urdf/toolchanger.xacro (robot description, xacro)
@@ -20,7 +20,7 @@
       </visual>
       <collision>
-        <origin xyz="0 0 0" rpy="0 0 0"/>
+        <origin xyz="${sec_mesh_files['toolchanger_trolley']['collision']['box']['origin']}" rpy="0 0 0"/>
         <geometry>
-          <xacro:get_mesh name="toolchanger_trolley" type="collision"/>
+          <box size="${sec_mesh_files['toolchanger_trolley']['collision']['box']['size']}"/>
         </geometry>
       </collision>
@@ -64,5 +64,5 @@
       <parent link="toolchanger_trolley_link" />
       <child link="tool_changer_link" />
-      <origin xyz="0.2 0.15 0.82" rpy="0 0 0"/>
+      <origin xyz="0.2 0.15 0.0" rpy="0 0 0"/>
     </joint>
   </xacro:macro>

File: src/descriptions/ur_description/urdf/ur_macro.xacro (robot description, xacro)
@@ -145,7 +145,7 @@
       </visual>
       <collision>
-        <origin xyz="0 0 0" rpy="0 0 0"/>
-        <geometry>
-          <xacro:get_mesh name="trolley" type="collision"/>
+        <origin xyz="${sec_mesh_files['trolley']['collision']['box']['origin']}" rpy="0 0 0"/>
+        <geometry>
+          <box size="${sec_mesh_files['trolley']['collision']['box']['size']}"/>
         </geometry>
       </collision>
@@ -189,5 +189,5 @@
       <parent link="${tf_prefix}ur10_trolley_link" />
       <child link="${tf_prefix}ur10_feeder_link" />
-      <origin xyz="0.525 0.025 0.82" rpy="0 0 0"/>
+      <origin xyz="0.525 0.025 0.0" rpy="0 0 0"/>
     </joint>
     <!-- UR plate link-->
@@ -218,5 +218,5 @@
       <parent link="${tf_prefix}ur10_trolley_link" />
       <child link="${tf_prefix}ur10_plate_link" />
-      <origin xyz="0 0 0.835" rpy="0 0 0"/>
+      <origin xyz="0 0 0.015" rpy="0 0 0"/>
     </joint>
     <!-- ur robot base link -->

File: src/descriptions/ur_description/urdf/vision.xacro (robot description, xacro)
@@ -20,7 +20,7 @@
       </visual>
       <collision>
-        <origin xyz="0 0 0" rpy="0 0 0"/>
+        <origin xyz="${sec_mesh_files['vision_trolley']['collision']['box']['origin']}" rpy="0 0 0"/>
         <geometry>
-          <xacro:get_mesh name="vision_trolley" type="collision"/>
+          <box size="${sec_mesh_files['vision_trolley']['collision']['box']['size']}"/>
         </geometry>
       </collision>
@@ -64,5 +64,5 @@
       <parent link="vision_trolley_link" />
       <child link="vision_cam_jig_link" />
-      <origin xyz="0.05 0 0.82" rpy="0 0 0"/>
+      <origin xyz="0.05 0 0.0" rpy="0 0 0"/>
     </joint>
     <!-- vision feeder link -->
@@ -93,5 +93,5 @@
       <parent link="vision_trolley_link" />
       <child link="vision_feeder_link" />
-      <origin xyz="-0.2 -0.15 0.82" rpy="0 0 0"/>
+      <origin xyz="-0.2 -0.15 0.0" rpy="0 0 0"/>
     </joint>
   </xacro:macro>

Commit message: edited origin for collision/inertia for trolleys (+0.43 to -0.43)

File: src/descriptions/ur_description/urdf/arf.xacro (robot description, xacro)
@@ -27,5 +27,5 @@
       <inertial>
         <mass value="5.0"/>
-        <origin xyz="0 0 0" rpy="0 0 0"/>
+        <origin xyz="0 0 -0.43" rpy="0 0 0"/>
         <inertia ixx="0.1" ixy="0" ixz="0" iyy="0.1" iyz="0" izz="0.1"/>
       </inertial>

File: src/descriptions/ur_description/urdf/denso.xacro (robot description, xacro)
@@ -29,5 +29,5 @@
       <inertial>
         <mass value="5.0"/>
-        <origin xyz="0 0 0" rpy="0 0 0"/>
+        <origin xyz="0 0 -0.43" rpy="0 0 0"/>
         <inertia ixx="0.1" ixy="0" ixz="0" iyy="0.1" iyz="0" izz="0.1"/>
       </inertial>

File: src/descriptions/ur_description/urdf/toolchanger.xacro (robot description, xacro)
@@ -27,5 +27,5 @@
       <inertial>
         <mass value="5.0"/>
-        <origin xyz="0 0 0" rpy="0 0 0"/>
+        <origin xyz="0 0 -0.43" rpy="0 0 0"/>
         <inertia ixx="0.1" ixy="0" ixz="0" iyy="0.1" iyz="0" izz="0.1"/>
       </inertial>

File: src/descriptions/ur_description/urdf/ur_macro.xacro (robot description, xacro)
@@ -152,5 +152,5 @@
       <inertial>
         <mass value="50.0"/>
-        <origin xyz="0 0 0.4" rpy="0 0 0"/>
+        <origin xyz="0 0 -0.43" rpy="0 0 0"/>
         <inertia ixx="8.33" ixy="0" ixz="0" iyy="8.33" iyz="0" izz="2.08"/>
       </inertial>

File: src/descriptions/ur_description/urdf/vision.xacro (robot description, xacro)
@@ -27,5 +27,5 @@
       <inertial>
         <mass value="5.0"/>
-        <origin xyz="0 0 0" rpy="0 0 0"/>
+        <origin xyz="0 0 -0.43" rpy="0 0 0"/>
         <inertia ixx="0.1" ixy="0" ixz="0" iyy="0.1" iyz="0" izz="0.1"/>
       </inertial>

Commit message: rotated arf gripper direction

File: src/descriptions/ur_description/urdf/arf.xacro (robot description, xacro)
@@ -190,5 +190,5 @@
     <link name="arf_back_aircyl_link">
       <visual>
-        <origin xyz="0 0 0" rpy="0 0 -3.141592"/>
+        <origin xyz="0 0 0" rpy="0 0 0"/>
         <geometry>
           <xacro:get_mesh name="arf_back_aircyl" type="visual"/>
@@ -199,5 +199,5 @@
       </visual>
       <collision>
-        <origin xyz="0 0 0" rpy="0 0 -3.141592"/>
+        <origin xyz="0 0 0" rpy="0 0 0"/>
         <geometry>
           <xacro:get_mesh name="arf_back_aircyl" type="collision"/>

File: src/descriptions/ur_description/urdf/feeder.xacro (robot description, xacro)
@@ -119,5 +119,5 @@
       </inertial>
     </link>
-    <!-- feeder y axis plate to feeder arm base joint (needs to be prismatic??) **********-->
+    <!-- feeder x axis mobile base to feeder arm base joint (needs to be prismatic??) **********-->
     <joint name="feeder_arm_base_joint" type="prismatic">
       <parent link="feeder_x_axis_mobile_base_link" />
