Commit message: edited arf spawn positions (gripper tooltip still not spawning properly)

File: src/descriptions/ur_description/urdf/arf.xacro (robot description, xacro)
@@ -93,5 +93,5 @@
       <parent link="arf_x_axis_link" />
       <child link="arf_y_axis_link" />
-      <origin xyz="-0.360 0.0 0.054" rpy="0 0 0"/>
+      <origin xyz="-0.1413 0.0 0.054" rpy="0 0 0"/>
       <axis xyz="-1 0 0"/>
       <limit lower="0.0" upper="0.35" effort="100" velocity="10" />
@@ -138,5 +138,5 @@
       <parent link="arf_jig_dummy_link" />
       <child link="arf_jig_link" />
-      <origin xyz="0 0.300 0.107" rpy="0 0 0"/>
+      <origin xyz="0 0.418 0.107" rpy="0 0 0"/>
       <axis xyz="0 1 0"/>
       <limit lower="-0.25" upper="0" effort="100" velocity="10" />

File: src/descriptions/ur_description/urdf/arf_elec.xacro (robot description, xacro)
@@ -93,5 +93,5 @@
       <parent link="arf_elec_x_axis_link" />
       <child link="arf_elec_y_axis_link" />
-      <origin xyz="0.2555 0.0 0.049" rpy="0 0 0"/>
+      <origin xyz="0.395 0.0 0.049" rpy="0 0 0"/>
     </joint>
   <!-- dummy link for jig joint -->
@@ -109,4 +109,5 @@
       <origin xyz="0 0 0" rpy="0 0 0"/>
     </joint>
+-
     <!-- arf jig link -->
     <link name="arf_elec_jig_link">
@@ -136,5 +137,5 @@
       <parent link="arf_elec_jig_dummy_link" />
       <child link="arf_elec_jig_link" />
-      <origin xyz="0 0.01 0.1215" rpy="0 0 0"/>
+      <origin xyz="0 0.1 0.1215" rpy="0 0 0"/>
     </joint>
     <!-- dummy link for aircyl joints -->
