Commit message: removed collision for gripper & disabled collision between trolleys and robot base

File: src/descriptions/ur_description/urdf/quickchanger_grippers.xacro (robot description, xacro)
@@ -16,10 +16,4 @@
         </material>
       </visual>
-      <collision>
-        <origin xyz="0 0 0" rpy="0 0 0"/>
-        <geometry>
-          <xacro:get_mesh name="quickchanger" type="collision"/>
-        </geometry>
-      </collision>
       <inertial>
         <mass value="2.0"/>
@@ -46,10 +40,4 @@
         </material>
       </visual>
-      <collision>
-        <origin xyz="0 0 0" rpy="0 0 0"/>
-        <geometry>
-          <xacro:get_mesh name="suction_master" type="collision"/>
-        </geometry>
-      </collision>
       <inertial>
         <mass value="1.0"/>
@@ -98,10 +86,4 @@
         </material>
       </visual>
-      <collision>
-        <origin xyz="0 0 0" rpy="0 0 0"/>
-        <geometry>
-          <xacro:get_mesh name="gripper" type="collision"/>
-        </geometry>
-      </collision>
       <inertial>
         <mass value="1.0"/>
@@ -127,10 +109,4 @@
         </material>
       </visual>
-      <collision>
-        <origin xyz="0 0 0" rpy="0 0 0"/>
-        <geometry>
-          <xacro:get_mesh name="tooltip1" type="collision"/>
-        </geometry>
-      </collision>
       <inertial>
         <mass value="0.5"/>
@@ -158,10 +134,4 @@
         </material>
       </visual>
-      <collision>
-        <origin xyz="0 0 0" rpy="0 0 0"/>
-        <geometry>
-          <xacro:get_mesh name="tooltip2" type="collision"/>
-        </geometry>
-      </collision>
       <inertial>
         <mass value="0.5"/>

File: src/moveit_config/srdf/ur_macro.srdf.xacro (robot description, xacro)
@@ -53,5 +53,7 @@
     <disable_collisions link1="${prefix}wrist_1_link" link2="${prefix}wrist_3_link" reason="Never" />
     <disable_collisions link1="${prefix}wrist_2_link" link2="${prefix}wrist_3_link" reason="Adjacent" />
-    <disable_collisions link1="${prefix}shoulder_link" link2="${prefix}arf_trolley_link" reason="Never" />
+    <!-- Disable collisions between trolleys and robot base -->
+    <disable_collisions link1="${prefix}base_link" link2="arf_trolley_link" reason="Never" />
+    <disable_collisions link1="${prefix}base_link" link2="${prefix}ur10_trolley_link" reason="Never" />
   </xacro:macro>
 </robot>

Commit message: replaced tooltip adpater (tooltip not attached properly yet_

File: src/descriptions/ur_description/urdf/quickchanger_grippers.xacro (robot description, xacro)
@@ -55,5 +55,5 @@
     <link name="tooltip_adapter_1_link">
       <visual>
-        <origin xyz="0 0 0" rpy="0 0 3.14159"/>
+        <origin xyz="0 0 0" rpy="0 0 0"/>
         <geometry>
           <xacro:get_mesh name="tooltip_adapter_1" type="visual"/>
@@ -65,5 +65,5 @@
       <inertial>
         <mass value="0.5"/>
-        <origin xyz="0 0 0" rpy="0 0 3.14159"/>
+        <origin xyz="0 0 0" rpy="0 0 0"/>
         <inertia ixx="0.001" ixy="0" ixz="0" iyy="0.001" iyz="0" izz="0.001"/>
       </inertial>
@@ -73,6 +73,6 @@
       <parent link="quickchanger_link"/>
       <child link="tooltip_adapter_1_link"/>
-      <origin xyz="-0.1341 0.053 0.1221" rpy="0.785398 0 -1.5708"/>
-      <axis xyz="1 0 0"/>
+      <origin xyz="0 0 0" rpy="0 0 0"/>
+      <axis xyz="0 -1 0"/>
       <limit lower="-0.041" upper="0.041" effort="50" velocity="10"/>
     </joint>
@@ -98,6 +98,6 @@
       <parent link="quickchanger_link"/>
       <child link="tooltip_adapter_2_link"/>
-      <origin xyz="-0.1341 -0.053 0.1221" rpy="0.785398 0 -1.5708"/>
-      <axis xyz="0 1 0"/>
+      <origin xyz="0 0 0" rpy="0 0 0"/>
+      <axis xyz="0 -1 0"/>
       <limit lower="-0.041" upper="0.041" effort="50" velocity="10"/>
     </joint>
@@ -123,5 +123,5 @@
       <parent link="tooltip_adapter_1_link"/>
       <child link="tooltip1_link"/>
-      <origin xyz="-0.002 0 0.04" rpy="0 0 0"/>
+      <origin xyz="-0.1624 0.051 0.1504" rpy="0 0 -1.5708"/>
     </joint>
     <!-- tooltip2_link -->
@@ -146,5 +146,5 @@
       <parent link="tooltip_adapter_2_link"/>
       <child link="tooltip2_link"/>
-      <origin xyz="0.002 0 0.04" rpy="0 0 3.14"/>
+      <origin xyz="-0.1624 -0.051 0.1504" rpy="0 0 1.5708"/>
     </joint>
   </xacro:macro>

Commit message: added trays and objects spawn for elec feeder

File: src/descriptions/ur_description/urdf/quickchanger_grippers.xacro (robot description, xacro)
@@ -76,4 +76,5 @@
       <axis xyz="0 -1 0"/>
       <limit lower="-0.041" upper="0.041" effort="50" velocity="10"/>
+      <dynamics damping="100" friction="10"/>
     </joint>
     <!-- tooltip_adapter_2_link -->
@@ -101,50 +102,5 @@
       <axis xyz="0 -1 0"/>
       <limit lower="-0.041" upper="0.041" effort="50" velocity="10"/>
-    </joint>
-    <!-- tooltip1_link -->
-    <link name="tooltip1_link">
-      <visual>
-        <origin xyz="0 0 0" rpy="0 0 1.5708"/>
-        <geometry>
-          <xacro:get_mesh name="tooltip1" type="visual"/>
-        </geometry>
-        <material name="${sec_mesh_files['tooltip1']['visual']['material']['name']}">
-          <color rgba="${sec_mesh_files['tooltip1']['visual']['material']['color']}"/>
-        </material>
-      </visual>
-      <inertial>
-        <mass value="0.5"/>
-        <origin xyz="0 0 0" rpy="0 0 1.5708"/>
-        <inertia ixx="0.001" ixy="0" ixz="0" iyy="0.001" iyz="0" izz="0.001"/>
-      </inertial>
-    </link>
-    <!-- tooltip1_joint -->
-    <joint name="tooltip1_joint" type="fixed">
-      <parent link="tooltip_adapter_1_link"/>
-      <child link="tooltip1_link"/>
-      <origin xyz="-0.1624 0.051 0.1504" rpy="0 0 -1.5708"/>
-    </joint>
-    <!-- tooltip2_link -->
-    <link name="tooltip2_link">
-      <visual>
-        <origin xyz="0 0 0" rpy="0 0 1.5708"/>
-        <geometry>
-          <xacro:get_mesh name="tooltip2" type="visual"/>
-        </geometry>
-        <material name="${sec_mesh_files['tooltip2']['visual']['material']['name']}">
-          <color rgba="${sec_mesh_files['tooltip2']['visual']['material']['color']}"/>
-        </material>
-      </visual>
-      <inertial>
-        <mass value="0.5"/>
-        <origin xyz="0 0 0" rpy="0 0 1.5708"/>
-        <inertia ixx="0.001" ixy="0" ixz="0" iyy="0.001" iyz="0" izz="0.001"/>
-      </inertial>
-    </link>
-    <!-- tooltip2_joint -->
-    <joint name="tooltip2_joint" type="fixed">
-      <parent link="tooltip_adapter_2_link"/>
-      <child link="tooltip2_link"/>
-      <origin xyz="-0.1624 -0.051 0.1504" rpy="0 0 1.5708"/>
+      <dynamics damping="100" friction="10"/>
     </joint>
   </xacro:macro>

Commit message: added tooltips and friction/damping to ur joints to prevent shift

File: src/descriptions/ur_description/urdf/quickchanger_grippers.xacro (robot description, xacro)
@@ -29,27 +29,4 @@
       <origin xyz="0 0 0.012" rpy="1.57 3.14 1.57"/>
     </joint>
-    <!-- suction_link -->
-    <link name="suction_link">
-      <visual>
-        <origin xyz="0 0 0" rpy="0 0 0"/>
-        <geometry>
-          <xacro:get_mesh name="suction" type="visual"/>
-        </geometry>
-        <material name="${sec_mesh_files['suction']['visual']['material']['name']}">
-          <color rgba="${sec_mesh_files['suction']['visual']['material']['color']}"/>
-        </material>
-      </visual>
-      <inertial>
-        <mass value="1.0"/>
-        <origin xyz="0 0 0" rpy="0 0 0"/>
-        <inertia ixx="1e-5" ixy="0" ixz="0" iyy="1e-5" iyz="0" izz="1e-5"/>
-      </inertial>
-    </link>
-    <!-- suction_joint -->
-    <joint name="suction_joint" type="fixed">
-      <parent link="quickchanger_link"/>
-      <child link="suction_link"/>
-      <origin xyz="0.1208 0.0019 0.1088" rpy="0 0.785 0"/>
-    </joint>
     <!-- tooltip_adapter_1_link -->
     <link name="tooltip_adapter_1_link">
@@ -76,5 +53,5 @@
       <axis xyz="0 -1 0"/>
       <limit lower="-0.041" upper="0.041" effort="50" velocity="10"/>
-      <dynamics damping="100" friction="10"/>
+      <dynamics damping="10" friction="10"/>
     </joint>
     <!-- tooltip_adapter_2_link -->
@@ -102,5 +79,4 @@
       <axis xyz="0 -1 0"/>
       <limit lower="-0.041" upper="0.041" effort="50" velocity="10"/>
-      <dynamics damping="100" friction="10"/>
     </joint>
   </xacro:macro>

File: src/descriptions/ur_description/urdf/ur_macro.xacro (robot description, xacro)
@@ -302,5 +302,5 @@
          <safety_controller soft_lower_limit="${shoulder_pan_lower_limit + safety_pos_margin}" soft_upper_limit="${shoulder_pan_upper_limit - safety_pos_margin}" k_position="${safety_k_position}" k_velocity="0.0"/>
       </xacro:if>
-      <dynamics damping="0" friction="0"/>
+      <dynamics damping="50" friction="10"/>
     </joint>
     <!-- ur robot upper arm link -->
@@ -342,5 +342,5 @@
          <safety_controller soft_lower_limit="${shoulder_lift_lower_limit + safety_pos_margin}" soft_upper_limit="${shoulder_lift_upper_limit - safety_pos_margin}" k_position="${safety_k_position}" k_velocity="0.0"/>
       </xacro:if>
-      <dynamics damping="0" friction="0"/>
+      <dynamics damping="50" friction="10"/>
     </joint>
     <!-- ur robot forearm link -->
@@ -382,5 +382,5 @@
          <safety_controller soft_lower_limit="${elbow_joint_lower_limit + safety_pos_margin}" soft_upper_limit="${elbow_joint_upper_limit - safety_pos_margin}" k_position="${safety_k_position}" k_velocity="0.0"/>
       </xacro:if>
-      <dynamics damping="0" friction="0"/>
+      <dynamics damping="30" friction="5"/>
     </joint>
     <!-- ur robot wrist 1 link -->
@@ -423,5 +423,5 @@
          <safety_controller soft_lower_limit="${wrist_1_lower_limit + safety_pos_margin}" soft_upper_limit="${wrist_1_upper_limit - safety_pos_margin}" k_position="${safety_k_position}" k_velocity="0.0"/>
       </xacro:if>
-      <dynamics damping="0" friction="0"/>
+      <dynamics damping="10" friction="2"/>
     </joint>
     <!-- ur robot wrist 2 link -->
@@ -464,5 +464,5 @@
          <safety_controller soft_lower_limit="${wrist_2_lower_limit + safety_pos_margin}" soft_upper_limit="${wrist_2_upper_limit - safety_pos_margin}" k_position="${safety_k_position}" k_velocity="0.0"/>
       </xacro:if>
-      <dynamics damping="0" friction="0"/>
+      <dynamics damping="10" friction="2"/>
     </joint>
     <!-- ur robot wrist 3 link -->
@@ -519,5 +519,5 @@
         </xacro:if>
       </xacro:unless>
-      <dynamics damping="0" friction="0"/>
+      <dynamics damping="5" friction="1"/>
     </joint>
     <!-- ft_frame link -->

Commit message: flange to tool

File: src/descriptions/ur_description/urdf/quickchanger_grippers.xacro (robot description, xacro)
@@ -8,5 +8,5 @@
     <link name="quickchanger_link">
       <visual>
-        <origin xyz="0 0 0" rpy="0 0 0"/>
+        <origin xyz="0 0 0" rpy="0 0 3.14"/>
         <geometry>
           <xacro:get_mesh name="quickchanger" type="visual"/>
@@ -19,18 +19,18 @@
         <mass value="2.0"/>
         <origin xyz="0 0 0" rpy="0 0 0"/>
-        <inertia ixx="1e-5" ixy="0" ixz="0" iyy="1e-5" iyz="0" izz="1e-5"/>
+        <inertia ixx="0.002" ixy="0" ixz="0" iyy="0.002" iyz="0" izz="0.002"/>
       </inertial>
     </link>
-    <!-- quickchanger_joint -->
+    <!-- quickchanger_joint - attached to tool0, rpy="0 0 0" -->
     <joint name="quickchanger_joint" type="fixed">
       <parent link="${parent}"/>
       <child link="quickchanger_link"/>
-      <!-- adjust quickchanger orientation to match flange orientation -->
-      <origin xyz="0 0 0.012" rpy="1.57 3.14 1.57"/>
+      <origin xyz="0 0 0.012" rpy="0 0 0"/>
+      <dynamics damping="100" friction="100"/>
     </joint>
     <!-- tooltip_adapter_1_link -->
     <link name="tooltip_adapter_1_link">
       <visual>
-        <origin xyz="0 0 0" rpy="0 0 0"/>
+        <origin xyz="0 0 0" rpy="0 0 3.14"/>
         <geometry>
           <xacro:get_mesh name="tooltip_adapter_1" type="visual"/>
@@ -58,5 +58,5 @@
     <link name="tooltip_adapter_2_link">
       <visual>
-        <origin xyz="0 0 0" rpy="0 0 0"/>
+        <origin xyz="0 0 0" rpy="0 0 3.14"/>
         <geometry>
           <xacro:get_mesh name="tooltip_adapter_2" type="visual"/>
@@ -79,4 +79,5 @@
       <axis xyz="0 -1 0"/>
       <limit lower="-0.041" upper="0.041" effort="50" velocity="10"/>
+      <dynamics damping="10" friction="10"/>
     </joint>
   </xacro:macro>

File: src/descriptions/ur_description/urdf/ur.urdf.xacro (robot description, xacro)
@@ -169,6 +169,6 @@
      <origin xyz="${ur_pos['x']} ${ur_pos['y']} ${ur_pos['z']}" rpy="${ur_pos['roll']} ${ur_pos['pitch']} ${ur_pos['yaw']}" />
    </xacro:ur_robot>
-     <!-- attach gripper -->
-   <xacro:quickchanger_grippers parent="$(arg tf_prefix)flange"/>
+    <!-- attach gripper -->
+  <xacro:quickchanger_grippers parent="$(arg tf_prefix)tool0"/>
    <xacro:if value="$(arg sim_gazebo)">
     <!-- Gazebo plugins -->

File: src/descriptions/ur_description/urdf/ur_macro.xacro (robot description, xacro)
@@ -423,5 +423,5 @@
          <safety_controller soft_lower_limit="${wrist_1_lower_limit + safety_pos_margin}" soft_upper_limit="${wrist_1_upper_limit - safety_pos_margin}" k_position="${safety_k_position}" k_velocity="0.0"/>
       </xacro:if>
-      <dynamics damping="10" friction="2"/>
+      <dynamics damping="30" friction="5"/>
     </joint>
     <!-- ur robot wrist 2 link -->
@@ -464,5 +464,5 @@
          <safety_controller soft_lower_limit="${wrist_2_lower_limit + safety_pos_margin}" soft_upper_limit="${wrist_2_upper_limit - safety_pos_margin}" k_position="${safety_k_position}" k_velocity="0.0"/>
       </xacro:if>
-      <dynamics damping="10" friction="2"/>
+      <dynamics damping="30" friction="5"/>
     </joint>
     <!-- ur robot wrist 3 link -->
@@ -519,5 +519,5 @@
         </xacro:if>
       </xacro:unless>
-      <dynamics damping="5" friction="1"/>
+      <dynamics damping="30" friction="5"/>
     </joint>
     <!-- ft_frame link -->
