Commit message: supply to feeder

File: src/descriptions/ur_description/urdf/feeder.xacro (robot description, xacro)
@@ -1,20 +1,20 @@
 <?xml version="1.0"?>
 <robot xmlns:xacro="http://wiki.ros.org/xacro">
-  <xacro:macro name="supply" params="parent">
-  <xacro:property name="supply_visual_params" value="${xacro.load_yaml('$(find ur_description)/config/supply_visual_parameters.yaml')}"/>
-  <xacro:property name="sec_mesh_files" value="${supply_visual_params['mesh_files']}" scope="parent"/>
+  <xacro:macro name="feeder" params="parent">
+  <xacro:property name="feeder_visual_params" value="${xacro.load_yaml('$(find ur_description)/config/feeder_visual_parameters.yaml')}"/>
+  <xacro:property name="sec_mesh_files" value="${feeder_visual_params['mesh_files']}" scope="parent"/>
   <xacro:property name="force_abs_paths" value="true" scope="parent"/>
   <!-- Load trolley positions configuration -->
   <xacro:property name="trolley_positions" value="${xacro.load_yaml('$(find ur_description)/config/trolley_positions.yaml')}"/>
-  <xacro:property name="supply_pos" value="${trolley_positions['trolley_positions']['supply']}"/>
-<!-- supply base link -->
-    <link name="supply_base_link">
+  <xacro:property name="feeder_pos" value="${trolley_positions['trolley_positions']['feeder']}"/>
+<!-- feeder base link -->
+    <link name="feeder_base_link">
       <visual>
         <origin xyz="0 0 0" rpy="0 0 0"/>
         <geometry>
-          <xacro:get_mesh name="supply_base" type="visual"/>
+          <xacro:get_mesh name="feeder_base" type="visual"/>
         </geometry>
-        <material name="${sec_mesh_files['supply_base']['visual']['material']['name']}">
-          <color rgba="${sec_mesh_files['supply_base']['visual']['material']['color']}"/>
+        <material name="${sec_mesh_files['feeder_base']['visual']['material']['name']}">
+          <color rgba="${sec_mesh_files['feeder_base']['visual']['material']['color']}"/>
         </material>
       </visual>
@@ -22,5 +22,5 @@
         <origin xyz="0 0 0" rpy="0 0 0"/>
         <geometry>
-          <xacro:get_mesh name="supply_base" type="collision"/>
+          <xacro:get_mesh name="feeder_base" type="collision"/>
         </geometry>
       </collision>
@@ -31,19 +31,19 @@
       </inertial>
     </link>
-    <!-- world to supply base joint -->
-   <joint name="supply_base_joint" type="fixed">
+    <!-- world to feeder base joint -->
+   <joint name="feeder_base_joint" type="fixed">
       <parent link="${parent}" />
-      <child link="supply_base_link" />
-      <origin xyz="${supply_pos['x']} ${supply_pos['y']} ${supply_pos['z']}" rpy="${supply_pos['roll']} ${supply_pos['pitch']} ${supply_pos['yaw']}"/>
+      <child link="feeder_base_link" />
+      <origin xyz="${feeder_pos['x']} ${feeder_pos['y']} ${feeder_pos['z']}" rpy="${feeder_pos['roll']} ${feeder_pos['pitch']} ${feeder_pos['yaw']}"/>
     </joint>
-<!-- supply y axis plate link -->
-    <link name="supply_y_axis_plate_link">
+<!-- feeder y axis plate link -->
+    <link name="feeder_y_axis_plate_link">
       <visual>
         <origin xyz="0 0 0" rpy="0 0 0"/>
         <geometry>
-          <xacro:get_mesh name="supply_y_axis_plate" type="visual"/>
+          <xacro:get_mesh name="feeder_y_axis_plate" type="visual"/>
         </geometry>
-        <material name="${sec_mesh_files['supply_y_axis_plate']['visual']['material']['name']}">
-          <color rgba="${sec_mesh_files['supply_y_axis_plate']['visual']['material']['color']}"/>
+        <material name="${sec_mesh_files['feeder_y_axis_plate']['visual']['material']['name']}">
+          <color rgba="${sec_mesh_files['feeder_y_axis_plate']['visual']['material']['color']}"/>
         </material>
       </visual>
@@ -51,5 +51,5 @@
         <origin xyz="0 0 0" rpy="0 0 0"/>
         <geometry>
-          <xacro:get_mesh name="supply_y_axis_plate" type="collision"/>
+          <xacro:get_mesh name="feeder_y_axis_plate" type="collision"/>
         </geometry>
       </collision>
@@ -60,21 +60,21 @@
       </inertial>
     </link>
-    <!-- supply base to supply y axis plate joint (needs to be prismatic) **********-->
-    <joint name="supply_y_axis_plate_joint" type="prismatic">
-      <parent link="supply_base_link" />
-      <child link="supply_y_axis_plate_link" />
+    <!-- feeder base to feeder y axis plate joint (needs to be prismatic) **********-->
+    <joint name="feeder_y_axis_plate_joint" type="prismatic">
+      <parent link="feeder_base_link" />
+      <child link="feeder_y_axis_plate_link" />
       <origin xyz="0.0 -0.98 0.0" rpy="0 0 0"/>
       <axis xyz="0 0 1"/>
       <limit lower="-0.98" upper="0.98" effort="100" velocity="10" />
     </joint>
-<!-- supply x axis mobile base link -->
-    <link name="supply_x_axis_mobile_base_link">
+<!-- feeder x axis mobile base link -->
+    <link name="feeder_x_axis_mobile_base_link">
       <visual>
         <origin xyz="0 0 0" rpy="0 0 0"/>
         <geometry>
-          <xacro:get_mesh name="supply_x_axis_mobile_base" type="visual"/>
+          <xacro:get_mesh name="feeder_x_axis_mobile_base" type="visual"/>
         </geometry>
-        <material name="${sec_mesh_files['supply_x_axis_mobile_base']['visual']['material']['name']}">
-          <color rgba="${sec_mesh_files['supply_x_axis_mobile_base']['visual']['material']['color']}"/>
+        <material name="${sec_mesh_files['feeder_x_axis_mobile_base']['visual']['material']['name']}">
+          <color rgba="${sec_mesh_files['feeder_x_axis_mobile_base']['visual']['material']['color']}"/>
         </material>
       </visual>
@@ -82,5 +82,5 @@
         <origin xyz="0 0 0" rpy="0 0 0"/>
         <geometry>
-          <xacro:get_mesh name="supply_x_axis_mobile_base" type="collision"/>
+          <xacro:get_mesh name="feeder_x_axis_mobile_base" type="collision"/>
         </geometry>
       </collision>
@@ -91,18 +91,18 @@
       </inertial>
     </link>
-      <!-- supply base to supply x axis mobile base joint (needs to be prismatic) **********-->
-  <joint name="supply_x_axis_mobile_base_joint" type="prismatic">
-      <parent link="supply_base_link" />
-      <child link="supply_x_axis_mobile_base_link" />
+      <!-- feeder base to feeder x axis mobile base joint (needs to be prismatic) **********-->
+  <joint name="feeder_x_axis_mobile_base_joint" type="prismatic">
+      <parent link="feeder_base_link" />
+      <child link="feeder_x_axis_mobile_base_link" />
       <origin xyz="0.0 0.0 0.01" rpy="0 0 0"/>
       <axis xyz="0 1 0"/>
       <limit lower="-0.98" upper="0.98" effort="100" velocity="10" />
     </joint>
-<!-- supply arm base link -->
-    <link name="supply_arm_base_link">
+<!-- feeder arm base link -->
+    <link name="feeder_arm_base_link">
       <visual>
         <origin xyz="0 0 0" rpy="0 0 0"/>
         <geometry>
-          <xacro:get_mesh name="supply_arm_base" type="visual"/>
+          <xacro:get_mesh name="feeder_arm_base" type="visual"/>
         </geometry>
       </visual>
@@ -110,5 +110,5 @@
         <origin xyz="0 0 0" rpy="0 0 0"/>
         <geometry>
-          <xacro:get_mesh name="supply_arm_base" type="collision"/>
+          <xacro:get_mesh name="feeder_arm_base" type="collision"/>
         </geometry>
       </collision>
@@ -119,18 +119,18 @@
       </inertial>
     </link>
-    <!-- supply y axis plate to supply arm base joint (needs to be prismatic??) **********-->
-    <joint name="supply_arm_base_joint" type="prismatic">
-      <parent link="supply_x_axis_mobile_base_link" />
-      <child link="supply_arm_base_link" />
+    <!-- feeder y axis plate to feeder arm base joint (needs to be prismatic??) **********-->
+    <joint name="feeder_arm_base_joint" type="prismatic">
+      <parent link="feeder_x_axis_mobile_base_link" />
+      <child link="feeder_arm_base_link" />
       <origin xyz="0.0 0.0 0.2566" rpy="0 0 0"/>
       <axis xyz="0 0 1"/>
       <limit lower="-0.98" upper="0.98" effort="100" velocity="10" />
     </joint>
-<!-- supply arm slider link -->
-    <link name="supply_arm_slider_link">
+<!-- feeder arm slider link -->
+    <link name="feeder_arm_slider_link">
       <visual>
         <origin xyz="0 0 0" rpy="0 0 0"/>
         <geometry>
-          <xacro:get_mesh name="supply_arm_slider" type="visual"/>
+          <xacro:get_mesh name="feeder_arm_slider" type="visual"/>
         </geometry>
       </visual>
@@ -138,5 +138,5 @@
         <origin xyz="0 0 0" rpy="0 0 0"/>
         <geometry>
-          <xacro:get_mesh name="supply_arm_slider" type="collision"/>
+          <xacro:get_mesh name="feeder_arm_slider" type="collision"/>
         </geometry>
       </collision>
@@ -147,18 +147,18 @@
       </inertial>
     </link>
-    <!-- supply arm base to supply arm slider joint (needs to be prismatic??) **********-->
-    <joint name="supply_arm_slider_joint" type="prismatic">
-      <parent link="supply_arm_base_link" />
-      <child link="supply_arm_slider_link" />
+    <!-- feeder arm base to feeder arm slider joint (needs to be prismatic??) **********-->
+    <joint name="feeder_arm_slider_joint" type="prismatic">
+      <parent link="feeder_arm_base_link" />
+      <child link="feeder_arm_slider_link" />
       <origin xyz="0.0 0.0 0.0215" rpy="0 0 0"/>
       <axis xyz="1 0 0"/>
       <limit lower="-0.98" upper="0.98" effort="100" velocity="10" />
     </joint>
-<!-- supply arm plate link -->
-    <link name="supply_arm_plate_link">
+<!-- feeder arm plate link -->
+    <link name="feeder_arm_plate_link">
       <visual>
         <origin xyz="0 0 0" rpy="0 0 0"/>
         <geometry>
-          <xacro:get_mesh name="supply_arm_plate" type="visual"/>
+          <xacro:get_mesh name="feeder_arm_plate" type="visual"/>
         </geometry>
       </visual>
@@ -166,5 +166,5 @@
         <origin xyz="0 0 0" rpy="0 0 0"/>
         <geometry>
-          <xacro:get_mesh name="supply_arm_plate" type="collision"/>
+          <xacro:get_mesh name="feeder_arm_plate" type="collision"/>
         </geometry>
       </collision>
@@ -175,8 +175,8 @@
       </inertial>
     </link>
-    <!-- supply arm slider to supply arm plate joint (needs to be prismatic?? & need z offset) **********-->
-    <joint name="supply_arm_plate_joint" type="prismatic">
-      <parent link="supply_arm_slider_link" />
-      <child link="supply_arm_plate_link" />
+    <!-- feeder arm slider to feeder arm plate joint (needs to be prismatic?? & need z offset) **********-->
+    <joint name="feeder_arm_plate_joint" type="prismatic">
+      <parent link="feeder_arm_slider_link" />
+      <child link="feeder_arm_plate_link" />
       <origin xyz="0.0 0.0 0.01" rpy="0 0 0"/>
       <axis xyz="1 0 0"/>

File: src/descriptions/ur_description/urdf/gazebo_materials.xacro (robot description, xacro)
@@ -142,42 +142,42 @@
   </gazebo>
   <!-- Supply Link Components -->
-  <gazebo reference="supply_base_link">
+  <gazebo reference="feeder_base_link">
     <material>Gazebo/LightGrey</material>
   </gazebo>
-  <gazebo reference="supply_x_axis_mobile_base_link">
+  <gazebo reference="feeder_x_axis_mobile_base_link">
     <material>Gazebo/Grey</material>
   </gazebo>
-  <gazebo reference="supply_y_axis_plate_link">
+  <gazebo reference="feeder_y_axis_plate_link">
     <material>Gazebo/Grey</material>
   </gazebo>
-  <gazebo reference="supply_arm_base_link">
+  <gazebo reference="feeder_arm_base_link">
     <material>Gazebo/LightGrey</material>
   </gazebo>
-  <gazebo reference="supply_arm_slider_link">
+  <gazebo reference="feeder_arm_slider_link">
     <material>Gazebo/Yellow</material>
   </gazebo>
-  <gazebo reference="supply_arm_plate_link">
+  <gazebo reference="feeder_arm_plate_link">
     <material>Gazebo/Green</material>
   </gazebo>
   <!-- Supply Joint Components -->
-  <gazebo reference="supply_base_joint">
+  <gazebo reference="feeder_base_joint">
     <preserveFixedJoint>true</preserveFixedJoint>
   </gazebo>
-  <gazebo reference="supply_x_axis_mobile_base_joint">
+  <gazebo reference="feeder_x_axis_mobile_base_joint">
     <preserveFixedJoint>true</preserveFixedJoint>
   </gazebo>
-  <gazebo reference="supply_y_axis_plate_joint">
+  <gazebo reference="feeder_y_axis_plate_joint">
     <preserveFixedJoint>true</preserveFixedJoint>
   </gazebo>
-  <gazebo reference="supply_y_axis_plate_supply_arm_base_joint">
+  <gazebo reference="feeder_y_axis_plate_feeder_arm_base_joint">
     <preserveFixedJoint>true</preserveFixedJoint>
   </gazebo>
-  <gazebo reference="supply_arm_base_supply_arm_slider_joint">
+  <gazebo reference="feeder_arm_base_feeder_arm_slider_joint">
     <preserveFixedJoint>true</preserveFixedJoint>
   </gazebo>
-  <gazebo reference="supply_arm_slider_supply_arm_plate_joint">
+  <gazebo reference="feeder_arm_slider_feeder_arm_plate_joint">
     <preserveFixedJoint>true</preserveFixedJoint>
   </gazebo>
-  <gazebo reference="supply_arm_plate_supply_arm_joint">
+  <gazebo reference="feeder_arm_plate_feeder_arm_joint">
     <preserveFixedJoint>true</preserveFixedJoint>
   </gazebo>

File: src/descriptions/ur_description/urdf/inc/ur_transmissions.xacro (robot description, xacro)
@@ -129,31 +129,31 @@
     </transmission>
     <!-- Supply Joints -->
-    <transmission name="supply_y_axis_plate_trans">
+    <transmission name="feeder_y_axis_plate_trans">
       <type>transmission_interface/SimpleTransmission</type>
-      <joint name="supply_y_axis_plate_joint">
+      <joint name="feeder_y_axis_plate_joint">
         <hardwareInterface>${hw_interface}</hardwareInterface>
       </joint>
     </transmission>
-    <transmission name="supply_x_axis_mobile_base_trans">
+    <transmission name="feeder_x_axis_mobile_base_trans">
       <type>transmission_interface/SimpleTransmission</type>
-      <joint name="supply_x_axis_mobile_base_joint">
+      <joint name="feeder_x_axis_mobile_base_joint">
         <hardwareInterface>${hw_interface}</hardwareInterface>
       </joint>
     </transmission>
-    <transmission name="supply_arm_base_trans">
+    <transmission name="feeder_arm_base_trans">
       <type>transmission_interface/SimpleTransmission</type>
-      <joint name="supply_arm_base_joint">
+      <joint name="feeder_arm_base_joint">
         <hardwareInterface>${hw_interface}</hardwareInterface>
       </joint>
     </transmission>
-    <transmission name="supply_arm_slider_trans">
+    <transmission name="feeder_arm_slider_trans">
       <type>transmission_interface/SimpleTransmission</type>
-      <joint name="supply_arm_slider_joint">
+      <joint name="feeder_arm_slider_joint">
         <hardwareInterface>${hw_interface}</hardwareInterface>
       </joint>
     </transmission>
-    <transmission name="supply_arm_plate_trans">
+    <transmission name="feeder_arm_plate_trans">
       <type>transmission_interface/SimpleTransmission</type>
-      <joint name="supply_arm_plate_joint">
+      <joint name="feeder_arm_plate_joint">
         <hardwareInterface>${hw_interface}</hardwareInterface>
       </joint>

File: src/descriptions/ur_description/urdf/ur.ros2_control.xacro (robot description, xacro)
@@ -240,10 +240,10 @@
       <!-- Supply Joints -->
       <!-- Supply Y Axis Plate Joint -->
-      <joint name="supply_y_axis_plate_joint">
-        <command_interface name="position"/>
-        <command_interface name="velocity"/>
-        <state_interface name="position">
-          <!-- initial position for the FakeSystem and simulation -->
-          <param name="initial_value">${initial_positions['supply_y_axis_plate_joint']}</param>
+      <joint name="feeder_y_axis_plate_joint">
+        <command_interface name="position"/>
+        <command_interface name="velocity"/>
+        <state_interface name="position">
+          <!-- initial position for the FakeSystem and simulation -->
+          <param name="initial_value">${initial_positions['feeder_y_axis_plate_joint']}</param>
         </state_interface>
         <state_interface name="velocity"/>
@@ -251,10 +251,10 @@
       </joint>
       <!-- Supply X Axis Mobile Base Joint -->
-      <joint name="supply_x_axis_mobile_base_joint">
-        <command_interface name="position"/>
-        <command_interface name="velocity"/>
-        <state_interface name="position">
-          <!-- initial position for the FakeSystem and simulation -->
-          <param name="initial_value">${initial_positions['supply_x_axis_mobile_base_joint']}</param>
+      <joint name="feeder_x_axis_mobile_base_joint">
+        <command_interface name="position"/>
+        <command_interface name="velocity"/>
+        <state_interface name="position">
+          <!-- initial position for the FakeSystem and simulation -->
+          <param name="initial_value">${initial_positions['feeder_x_axis_mobile_base_joint']}</param>
         </state_interface>
         <state_interface name="velocity"/>
@@ -262,10 +262,10 @@
       </joint>
       <!-- Supply Arm Base Joint -->
-      <joint name="supply_arm_base_joint">
-        <command_interface name="position"/>
-        <command_interface name="velocity"/>
-        <state_interface name="position">
-          <!-- initial position for the FakeSystem and simulation -->
-          <param name="initial_value">${initial_positions['supply_arm_base_joint']}</param>
+      <joint name="feeder_arm_base_joint">
+        <command_interface name="position"/>
+        <command_interface name="velocity"/>
+        <state_interface name="position">
+          <!-- initial position for the FakeSystem and simulation -->
+          <param name="initial_value">${initial_positions['feeder_arm_base_joint']}</param>
         </state_interface>
         <state_interface name="velocity"/>
@@ -273,10 +273,10 @@
       </joint>
       <!-- Supply Arm Slider Joint -->
-      <joint name="supply_arm_slider_joint">
-        <command_interface name="position"/>
-        <command_interface name="velocity"/>
-        <state_interface name="position">
-          <!-- initial position for the FakeSystem and simulation -->
-          <param name="initial_value">${initial_positions['supply_arm_slider_joint']}</param>
+      <joint name="feeder_arm_slider_joint">
+        <command_interface name="position"/>
+        <command_interface name="velocity"/>
+        <state_interface name="position">
+          <!-- initial position for the FakeSystem and simulation -->
+          <param name="initial_value">${initial_positions['feeder_arm_slider_joint']}</param>
         </state_interface>
         <state_interface name="velocity"/>
@@ -284,10 +284,10 @@
       </joint>
       <!-- Supply Arm Plate Joint -->
-      <joint name="supply_arm_plate_joint">
-        <command_interface name="position"/>
-        <command_interface name="velocity"/>
-        <state_interface name="position">
-          <!-- initial position for the FakeSystem and simulation -->
-          <param name="initial_value">${initial_positions['supply_arm_plate_joint']}</param>
+      <joint name="feeder_arm_plate_joint">
+        <command_interface name="position"/>
+        <command_interface name="velocity"/>
+        <state_interface name="position">
+          <!-- initial position for the FakeSystem and simulation -->
+          <param name="initial_value">${initial_positions['feeder_arm_plate_joint']}</param>
         </state_interface>
         <state_interface name="velocity"/>

File: src/descriptions/ur_description/urdf/ur.urdf.xacro (robot description, xacro)
@@ -15,6 +15,6 @@
    <!-- import denso macro -->
    <xacro:include filename="$(find ur_description)/urdf/denso.xacro"/>
-   <!-- import supply macro -->
-   <xacro:include filename="$(find ur_description)/urdf/supply.xacro"/>
+   <!-- import feeder macro -->
+   <xacro:include filename="$(find ur_description)/urdf/feeder.xacro"/>
    <!-- import gazebo materials -->
    <xacro:include filename="$(find ur_description)/urdf/gazebo_materials.xacro"/>
@@ -99,6 +99,6 @@
   <!-- denso components -->
   <xacro:denso parent="world"/>
-  <!-- supply components -->
-  <xacro:supply parent="world"/>
+  <!-- feeder components -->
+  <xacro:feeder parent="world"/>
    <!-- Load trolley positions configuration -->
    <xacro:property name="trolley_positions" value="${xacro.load_yaml('$(find ur_description)/config/trolley_positions.yaml')}"/>

Commit message: added materials for feeder

File: src/descriptions/ur_description/urdf/feeder.xacro (robot description, xacro)
@@ -106,4 +106,7 @@
           <xacro:get_mesh name="feeder_arm_base" type="visual"/>
         </geometry>
+        <material name="${sec_mesh_files['feeder_arm_base']['visual']['material']['name']}">
+          <color rgba="${sec_mesh_files['feeder_arm_base']['visual']['material']['color']}"/>
+        </material>
       </visual>
       <collision>
@@ -134,4 +137,7 @@
           <xacro:get_mesh name="feeder_arm_slider" type="visual"/>
         </geometry>
+        <material name="${sec_mesh_files['feeder_arm_slider']['visual']['material']['name']}">
+          <color rgba="${sec_mesh_files['feeder_arm_slider']['visual']['material']['color']}"/>
+        </material>
       </visual>
       <collision>
@@ -162,4 +168,7 @@
           <xacro:get_mesh name="feeder_arm_plate" type="visual"/>
         </geometry>
+        <material name="${sec_mesh_files['feeder_arm_plate']['visual']['material']['name']}">
+          <color rgba="${sec_mesh_files['feeder_arm_plate']['visual']['material']['color']}"/>
+        </material>
       </visual>
       <collision>

Commit message: edited feeder y axis position / koras colour

File: src/descriptions/ur_description/urdf/feeder.xacro (robot description, xacro)
@@ -64,5 +64,5 @@
       <parent link="feeder_base_link" />
       <child link="feeder_y_axis_plate_link" />
-      <origin xyz="0.0 -0.98 0.0" rpy="0 0 0"/>
+      <origin xyz="0.0 -0.9685 0.0" rpy="0 0 0"/>
       <axis xyz="0 0 1"/>
       <limit lower="-0.98" upper="0.98" effort="100" velocity="10" />
