Commit message: added controllers for arf elec - axis&gripper\

File: src/descriptions/urdf/arf_elec.xacro (robot description, xacro)
@@ -89,9 +89,12 @@
       </inertial>
     </link>
-    <!-- arf_x_axis to arf_y_axis joint (prismatic*********) -->
-    <joint name="arf_elec_axis_1_joint" type="fixed">
+    <!-- arf_x_axis to arf_y_axis joint (prismatic - moves along -X) -->
+    <joint name="arf_elec_axis_1_joint" type="prismatic">
       <parent link="arf_elec_x_axis_link" />
       <child link="arf_elec_y_axis_link" />
       <origin xyz="0.395 0.0 0.049" rpy="0 0 0"/>
+      <axis xyz="-1 0 0"/>
+      <limit lower="-0.3" upper="0.3" effort="100" velocity="0.5"/>
+      <dynamics damping="10" friction="1"/>
     </joint>
   <!-- dummy link for jig joint -->
@@ -133,9 +136,12 @@
       </inertial>
     </link>
-    <!-- arf_y_axis to arf_jig joint (prismatic *********) -->
-    <joint name="arf_elec_axis_2_joint" type="fixed">
+    <!-- arf_y_axis to arf_jig joint (prismatic - moves along -Y) -->
+    <joint name="arf_elec_axis_2_joint" type="prismatic">
       <parent link="arf_elec_jig_dummy_link" />
       <child link="arf_elec_jig_link" />
       <origin xyz="0 0.1 0.1215" rpy="0 0 0"/>
+      <axis xyz="0 -1 0"/>
+      <limit lower="-0.2" upper="0.2" effort="100" velocity="0.5"/>
+      <dynamics damping="10" friction="1"/>
     </joint>
     <!-- dummy link for aircyl joints -->
@@ -153,5 +159,5 @@
       <origin xyz="0 0 0" rpy="0 0 0"/>
     </joint>
-    <!-- arf front aircyl link -->
+    <!-- arf side aircyl link -->
     <link name="arf_elec_aircyl_1_link">
       <visual>
@@ -176,11 +182,14 @@
       </inertial>
     </link>
-    <!-- arf jig to front aircyl joint (prismatic *********) -->
-    <joint name="arf_elec_aircyl_1_joint" type="fixed">
+    <!-- arf jig to side aircyl joint (prismatic - moves along Y) -->
+    <joint name="arf_elec_gripper_joint_1" type="prismatic">
       <parent link="arf_elec_aircyl_dummy_link" />
       <child link="arf_elec_aircyl_1_link" />
       <origin xyz="0.145 0.214 -0.0145" rpy="0 0 0"/>
-    </joint>
-    <!-- arf front aircyl 2 link -->
+      <axis xyz="0 1 0"/>
+      <limit lower="-0.05" upper="0.05" effort="50" velocity="0.2"/>
+      <dynamics damping="5" friction="0.5"/>
+    </joint>
+    <!-- arf side aircyl 2 link -->
     <link name="arf_elec_aircyl_1_2_link">
       <visual>
@@ -205,11 +214,14 @@
       </inertial>
     </link>
-    <!-- arf front aircyl 2 joint (prismatic *********) -->
-    <joint name="arf_elec_aircyl_1_2_joint" type="fixed">
+    <!-- arf side aircyl 2 joint (prismatic - moves along Y) -->
+    <joint name="arf_elec_gripper_joint_2" type="prismatic">
       <parent link="arf_elec_aircyl_dummy_link" />
       <child link="arf_elec_aircyl_1_2_link" />
       <origin xyz="-0.145 0.214 -0.0145" rpy="0 0 0"/>
-    </joint>
-    <!-- arf back aircyl link -->
+      <axis xyz="0 1 0"/>
+      <limit lower="-0.05" upper="0.05" effort="50" velocity="0.2"/>
+      <dynamics damping="5" friction="0.5"/>
+    </joint>
+    <!-- arf front aircyl link -->
     <link name="arf_elec_aircyl_2_link">
       <visual>
@@ -234,9 +246,12 @@
       </inertial>
     </link>
-    <!-- arf jig to back aircyl joint (prismatic *********) -->
-    <joint name="arf_elec_aircyl_2_joint" type="fixed">
+    <!-- arf jig to front aircyl joint (prismatic - moves along X) -->
+    <joint name="arf_elec_gripper_joint_3" type="prismatic">
       <parent link="arf_elec_aircyl_dummy_link" />
       <child link="arf_elec_aircyl_2_link" />
       <origin xyz="0.2815 0 -0.0145" rpy="0 0 0"/>
+      <axis xyz="1 0 0"/>
+      <limit lower="-0.05" upper="0.05" effort="50" velocity="0.2"/>
+      <dynamics damping="5" friction="0.5"/>
     </joint>
   </xacro:macro>

File: src/descriptions/urdf/gazebo_materials.xacro (robot description, xacro)
@@ -132,8 +132,8 @@
   </gazebo>
   <gazebo reference="arf_elec_x_axis_link">
-    <material>Gazebo/Blue</material>
+    <material>Gazebo/Grey</material>
   </gazebo>
   <gazebo reference="arf_elec_y_axis_link">
-    <material>Gazebo/Blue</material>
+    <material>Gazebo/Grey</material>
   </gazebo>
   <gazebo reference="arf_elec_jig_link">

File: src/descriptions/urdf/workcell.ros2_control.xacro (robot description, xacro)
@@ -182,4 +182,51 @@
           <!-- initial position for the FakeSystem and simulation -->
           <param name="initial_value">${initial_positions['arf_gripper_joint_2']}</param>
+        </state_interface>
+        <state_interface name="velocity"/>
+        <state_interface name="effort"/>
+      </joint>
+      <!-- ARF Elec Axis Joints -->
+      <joint name="arf_elec_axis_1_joint">
+        <command_interface name="position"/>
+        <command_interface name="velocity"/>
+        <state_interface name="position">
+          <param name="initial_value">${initial_positions['arf_elec_axis_1_joint']}</param>
+        </state_interface>
+        <state_interface name="velocity"/>
+        <state_interface name="effort"/>
+      </joint>
+      <joint name="arf_elec_axis_2_joint">
+        <command_interface name="position"/>
+        <command_interface name="velocity"/>
+        <state_interface name="position">
+          <param name="initial_value">${initial_positions['arf_elec_axis_2_joint']}</param>
+        </state_interface>
+        <state_interface name="velocity"/>
+        <state_interface name="effort"/>
+      </joint>
+      <!-- ARF Elec Gripper Joints -->
+      <joint name="arf_elec_gripper_joint_1">
+        <command_interface name="position"/>
+        <command_interface name="velocity"/>
+        <state_interface name="position">
+          <param name="initial_value">${initial_positions['arf_elec_gripper_joint_1']}</param>
+        </state_interface>
+        <state_interface name="velocity"/>
+        <state_interface name="effort"/>
+      </joint>
+      <joint name="arf_elec_gripper_joint_2">
+        <command_interface name="position"/>
+        <command_interface name="velocity"/>
+        <state_interface name="position">
+          <param name="initial_value">${initial_positions['arf_elec_gripper_joint_2']}</param>
+        </state_interface>
+        <state_interface name="velocity"/>
+        <state_interface name="effort"/>
+      </joint>
+      <joint name="arf_elec_gripper_joint_3">
+        <command_interface name="position"/>
+        <command_interface name="velocity"/>
+        <state_interface name="position">
+          <param name="initial_value">${initial_positions['arf_elec_gripper_joint_3']}</param>
         </state_interface>
         <state_interface name="velocity"/>
