Commit message: edited position of arf elec

File: src/descriptions/urdf/arf_elec.xacro (robot description, xacro)
@@ -64,5 +64,5 @@
       <parent link="arf_elec_trolley_link" />
       <child link="arf_elec_x_axis_link" />
-      <origin xyz="-0.264 -0.025 0.014" rpy="0 0 0"/>
+      <origin xyz="-0.266 0.025 0.014" rpy="0 0 0"/>
     </joint>
     <!-- arf y axis link (slider) -->
