Commit message: repositioned trollyes + denso arf,denso feeder etc

File: src/descriptions/urdf/arf.xacro (robot description, xacro)
@@ -11,5 +11,5 @@
     <link name="arf_trolley_link">
       <visual>
-        <origin xyz="0 0 0" rpy="0 0 0"/>
+        <origin xyz="0 0 0" rpy="0 0 -1.57"/>
         <geometry>
           <xacro:get_mesh name="arf_trolley" type="visual"/>

File: src/descriptions/urdf/arf_elec.xacro (robot description, xacro)
@@ -11,5 +11,5 @@
     <link name="arf_elec_trolley_link">
       <visual>
-        <origin xyz="0 0 0" rpy="0 0 0"/>
+        <origin xyz="0 0 0" rpy="0 0 -1.57"/>
         <geometry>
           <xacro:get_mesh name="arf_elec_trolley" type="visual"/>

File: src/descriptions/urdf/denso.xacro (robot description, xacro)
@@ -11,5 +11,5 @@
     <link name="denso_trolley_link">
       <visual>
-        <origin xyz="0 0 0" rpy="0 0 0"/>
+        <origin xyz="0 0 0" rpy="0 0 -1.57"/>
         <geometry>
           <xacro:get_mesh name="denso_trolley" type="visual"/>
@@ -64,5 +64,34 @@
       <parent link="denso_trolley_link" />
       <child link="denso_slider_jig_link" />
-      <origin xyz="0.025 -0.025 0.0" rpy="0 0 0"/>
+      <origin xyz="0.025 0.175 0.0" rpy="0 0 0"/>
+    </joint>
+  <!-- vision feeder link -->
+    <link name="vision_feeder_link">
+      <visual>
+        <origin xyz="0 0 0" rpy="0 0 0"/>
+        <geometry>
+          <xacro:get_mesh name="vision_feeder" type="visual"/>
+        </geometry>
+        <material name="${sec_mesh_files['vision_feeder']['visual']['material']['name']}">
+          <color rgba="${sec_mesh_files['vision_feeder']['visual']['material']['color']}"/>
+        </material>
+      </visual>
+      <collision>
+        <origin xyz="0 0 0" rpy="0 0 0"/>
+        <geometry>
+          <xacro:get_mesh name="vision_feeder" type="visual"/>
+        </geometry>
+      </collision>
+      <inertial>
+        <mass value="3.0"/>
+        <origin xyz="0 0 0" rpy="0 0 0"/>
+        <inertia ixx="0.08" ixy="0" ixz="0" iyy="0.08" iyz="0" izz="0.08"/>
+      </inertial>
+    </link>
+    <!-- trolley to vision feeder joint -->
+    <joint name="vision_feeder_joint" type="fixed">
+      <parent link="denso_trolley_link" />
+      <child link="vision_feeder_link" />
+      <origin xyz="0.2 -0.2 0.0" rpy="0 0 0"/>
     </joint>
     <!-- ==================== DENSO ROBOT ARM ==================== -->

File: src/descriptions/urdf/toolchanger.xacro (robot description, xacro)
@@ -11,5 +11,5 @@
     <link name="toolchanger_trolley_link">
       <visual>
-        <origin xyz="0 0 0" rpy="0 0 0"/>
+        <origin xyz="0 0 0" rpy="0 0 1.57"/>
         <geometry>
           <xacro:get_mesh name="toolchanger_trolley" type="visual"/>
@@ -64,5 +64,5 @@
       <parent link="toolchanger_trolley_link" />
       <child link="tool_changer_link" />
-      <origin xyz="0.3 0.0 0.0" rpy="0 0 0"/>
+      <origin xyz="0.0 -0.25 0.0" rpy="0 0 -1.57"/>
     </joint>
   </xacro:macro>

File: src/descriptions/urdf/ur_macro.xacro (robot description, xacro)
@@ -252,5 +252,5 @@
     <link name="${tf_prefix}ur10_trolley_link">
       <visual>
-        <origin xyz="0 0 0" rpy="0 0 0"/>
+        <origin xyz="0 0 0" rpy="0 0 -1.57"/>
         <geometry>
           <xacro:get_mesh name="trolley" type="visual"/>

File: src/descriptions/urdf/vision.xacro (robot description, xacro)
@@ -11,5 +11,5 @@
     <link name="vision_trolley_link">
       <visual>
-        <origin xyz="0 0 0" rpy="0 0 0"/>
+        <origin xyz="0 0 0" rpy="0 0 -1.57"/>
         <geometry>
           <xacro:get_mesh name="vision_trolley" type="visual"/>
@@ -64,34 +64,5 @@
       <parent link="vision_trolley_link" />
       <child link="vision_cam_jig_link" />
-      <origin xyz="0.05 0 0.0" rpy="0 0 0"/>
-    </joint>
-    <!-- vision feeder link -->
-    <link name="vision_feeder_link">
-      <visual>
-        <origin xyz="0 0 0" rpy="0 0 0"/>
-        <geometry>
-          <xacro:get_mesh name="vision_feeder" type="visual"/>
-        </geometry>
-        <material name="${sec_mesh_files['vision_feeder']['visual']['material']['name']}">
-          <color rgba="${sec_mesh_files['vision_feeder']['visual']['material']['color']}"/>
-        </material>
-      </visual>
-      <collision>
-        <origin xyz="0 0 0" rpy="0 0 0"/>
-        <geometry>
-          <xacro:get_mesh name="vision_feeder" type="visual"/>
-        </geometry>
-      </collision>
-      <inertial>
-        <mass value="3.0"/>
-        <origin xyz="0 0 0" rpy="0 0 0"/>
-        <inertia ixx="0.08" ixy="0" ixz="0" iyy="0.08" iyz="0" izz="0.08"/>
-      </inertial>
-    </link>
-    <!-- trolley to feeder joint -->
-    <joint name="vision_feeder_joint" type="fixed">
-      <parent link="vision_trolley_link" />
-      <child link="vision_feeder_link" />
-      <origin xyz="-0.2 -0.15 0.0" rpy="0 0 0"/>
+      <origin xyz="-0.2 -0.25 0.0" rpy="0 0 3.141592"/>
     </joint>
   </xacro:macro>
