Commit message: edited position of arf x axis

File: src/descriptions/urdf/arf.xacro (robot description, xacro)
@@ -64,5 +64,5 @@
       <parent link="arf_trolley_link" />
       <child link="arf_x_axis_link" />
-      <origin xyz="0.37 -0.2975 0.0" rpy="0 0 0"/>
+      <origin xyz="0.31996 -0.2975 0.0" rpy="0 0 0"/>
     </joint>
     <!-- arf y axis link (slider) -->
