Commit message: Update trolley and visual parameters for UR slider jig integration

File: src/descriptions/urdf/gazebo_materials.xacro (robot description, xacro)
@@ -13,4 +13,7 @@
     <material>Gazebo/Grey</material>
   </gazebo>
+  <gazebo reference="ur10_slider_jig_link">
+    <material>Gazebo/Grey</material>
+  </gazebo>
   <!-- UR Joint Components-->
   <gazebo reference="ur10_feeder_joint">
@@ -38,4 +41,7 @@
     <preserveFixedJoint>true</preserveFixedJoint>
   </gazebo>
+  <gazebo reference="ur10_slider_jig_joint">
+    <preserveFixedJoint>true</preserveFixedJoint>
+  </gazebo>
   <!-- Quickchanger and Gripper Link Components -->
   <gazebo reference="quickchanger_link">

File: src/descriptions/urdf/toolchanger.xacro (robot description, xacro)
@@ -40,5 +40,5 @@
     <link name="tool_changer_link">
       <visual>
-        <origin xyz="0 0 0" rpy="0 0 0"/>
+        <origin xyz="0 0.25 0" rpy="0 0 1.57"/>
         <geometry>
           <xacro:get_mesh name="tool_changer" type="visual"/>
@@ -64,5 +64,5 @@
       <parent link="toolchanger_trolley_link" />
       <child link="tool_changer_link" />
-      <origin xyz="0.25 0.0 0.0" rpy="0 0 0"/>
+      <origin xyz="0.0 0.0 0.0" rpy="0 0 0"/>
     </joint>
   </xacro:macro>

File: src/descriptions/urdf/ur_macro.xacro (robot description, xacro)
@@ -278,5 +278,6 @@
       <child link="${tf_prefix}ur10_trolley_link" />
     </joint>
-    <!-- UR feeder link -->
+    <!--
+    UR feeder link
     <link name="${tf_prefix}ur10_feeder_link">
       <visual>
@@ -301,5 +302,5 @@
       </inertial>
     </link>
-    <!-- UR feeder joint -->
+    UR feeder joint
     <joint name="${tf_prefix}ur10_feeder_joint" type="fixed">
       <parent link="${tf_prefix}ur10_trolley_link" />
@@ -307,4 +308,34 @@
       <origin xyz="0.525 0.025 0.0" rpy="0 0 0"/>
     </joint>
+    -->
+    <!-- UR slider jig link -->
+    <link name="${tf_prefix}ur10_slider_jig_link">
+      <visual>
+        <origin xyz="0 0 0" rpy="0 0 0"/>
+        <geometry>
+          <xacro:get_mesh name="ur_slider_jig" type="visual"/>
+        </geometry>
+        <material name="${sec_mesh_files['ur_slider_jig']['visual']['material']['name']}">
+          <color rgba="${sec_mesh_files['ur_slider_jig']['visual']['material']['color']}"/>
+        </material>
+      </visual>
+      <collision>
+        <origin xyz="0 0 0" rpy="0 0 0"/>
+        <geometry>
+          <xacro:get_mesh name="ur_slider_jig" type="collision"/>
+        </geometry>
+      </collision>
+      <inertial>
+        <mass value="10.0"/>
+        <origin xyz="0 0 0" rpy="0 0 0"/>
+        <inertia ixx="0.083" ixy="0" ixz="0" iyy="0.083" iyz="0" izz="0.083"/>
+      </inertial>
+    </link>
+    <!-- trolley to slider jig joint -->
+    <joint name="${tf_prefix}ur10_slider_jig_joint" type="fixed">
+      <parent link="${tf_prefix}ur10_trolley_link" />
+      <child link="${tf_prefix}ur10_slider_jig_link" />
+      <origin xyz="0 0 0" rpy="0 0 0"/>
+    </joint>
     <!-- UR plate link-->
     <link name="${tf_prefix}ur10_plate_link">
@@ -330,9 +361,9 @@
       </inertial>
     </link>
-    <!-- trolley1 to UR plate joint -->
+    <!-- slider jig to UR plate joint -->
     <joint name="${tf_prefix}ur10_plate_joint" type="fixed">
-      <parent link="${tf_prefix}ur10_trolley_link" />
+      <parent link="${tf_prefix}ur10_slider_jig_link" />
       <child link="${tf_prefix}ur10_plate_link" />
-      <origin xyz="0 0 0.015" rpy="0 0 0"/>
+      <origin xyz="-0.2 0 0.135" rpy="0 0 0"/>
     </joint>
     <!-- ur robot base link -->

File: src/descriptions/urdf/vision.xacro (robot description, xacro)
@@ -64,5 +64,5 @@
       <parent link="vision_trolley_link" />
       <child link="vision_cam_jig_link" />
-      <origin xyz="-0.2 -0.25 0.0" rpy="0 0 3.141592"/>
+      <origin xyz="-0.2 0.25 0.0" rpy="0 0 -2.35"/>
     </joint>
   </xacro:macro>
