Commit message: edited feeder arm and gripper adapter direction

File: src/descriptions/urdf/feeder.xacro (robot description, xacro)
@@ -158,5 +158,5 @@
       <child link="feeder_arm_slider_link" />
       <origin xyz="0.0 0.0 0.0215" rpy="0 0 0"/>
-      <axis xyz="1 0 0"/>
+      <axis xyz="-1 0 0"/>
       <limit lower="-0.98" upper="0.98" effort="100" velocity="10" />
     </joint>
@@ -189,5 +189,5 @@
       <child link="feeder_arm_plate_link" />
       <origin xyz="0.0 0.0 0.01" rpy="0 0 0"/>
-      <axis xyz="1 0 0"/>
+      <axis xyz="-1 0 0"/>
       <limit lower="-0.98" upper="0.98" effort="100" velocity="10" />
     </joint>

File: src/descriptions/urdf/quickchanger_grippers.xacro (robot description, xacro)
@@ -51,5 +51,5 @@
       <child link="tooltip_adapter_1_link"/>
       <origin xyz="0 0 0" rpy="0 0 0"/>
-      <axis xyz="0 -1 0"/>
+      <axis xyz="0 1 0"/>
       <limit lower="-0.041" upper="0.041" effort="50" velocity="10"/>
       <dynamics damping="10" friction="10"/>
@@ -77,5 +77,5 @@
       <child link="tooltip_adapter_2_link"/>
       <origin xyz="0 0 0" rpy="0 0 0"/>
-      <axis xyz="0 -1 0"/>
+      <axis xyz="0 1 0"/>
       <limit lower="-0.041" upper="0.041" effort="50" velocity="10"/>
       <dynamics damping="10" friction="10"/>

Commit message: edited feeder mobile base to be child of y axis plate

File: src/descriptions/urdf/feeder.xacro (robot description, xacro)
@@ -91,9 +91,9 @@
       </inertial>
     </link>
-      <!-- feeder base to feeder x axis mobile base joint -->
+      <!-- feeder y axis plate to feeder x axis mobile base joint -->
   <joint name="feeder_x_axis_mobile_base_joint" type="prismatic">
-      <parent link="feeder_base_link" />
+      <parent link="feeder_y_axis_plate_link" />
       <child link="feeder_x_axis_mobile_base_link" />
-      <origin xyz="0.0 0.0 0.01" rpy="0 0 0"/>
+      <origin xyz="0.0 0.9685 0.01" rpy="0 0 0"/>
       <axis xyz="0 1 0"/>
       <limit lower="-0.98" upper="0.98" effort="100" velocity="10" />
