Commit message: repositioned toolchanger trolley and toolchanger stand

File: src/descriptions/urdf/toolchanger.xacro (robot description, xacro)
@@ -11,5 +11,5 @@
     <link name="toolchanger_trolley_link">
       <visual>
-        <origin xyz="0 0 0" rpy="0 0 1.57"/>
+        <origin xyz="0 0 0" rpy="0 0 -1.57"/>
         <geometry>
           <xacro:get_mesh name="toolchanger_trolley" type="visual"/>
@@ -64,5 +64,5 @@
       <parent link="toolchanger_trolley_link" />
       <child link="tool_changer_link" />
-      <origin xyz="0.0 -0.25 0.0" rpy="0 0 -1.57"/>
+      <origin xyz="0.25 0.0 0.0" rpy="0 0 0"/>
     </joint>
   </xacro:macro>

Commit message: edited tooltips spawning for quickchanger link and toolstand

File: src/descriptions/urdf/toolchanger.xacro (robot description, xacro)
@@ -40,5 +40,5 @@
     <link name="tool_changer_link">
       <visual>
-        <origin xyz="0 0.25 0" rpy="0 0 1.57"/>
+        <origin xyz="0 0.0 0" rpy="0 0 1.57"/>
         <geometry>
           <xacro:get_mesh name="tool_changer" type="visual"/>
@@ -64,5 +64,5 @@
       <parent link="toolchanger_trolley_link" />
       <child link="tool_changer_link" />
-      <origin xyz="0.0 0.0 0.0" rpy="0 0 0"/>
+      <origin xyz="0.0 0.25 0.0" rpy="0 0 0"/>
     </joint>
   </xacro:macro>
