Commit message: rotated ur10 trolley

File: src/descriptions/urdf/ur_macro.xacro (robot description, xacro)
@@ -252,5 +252,5 @@
     <link name="${tf_prefix}ur10_trolley_link">
       <visual>
-        <origin xyz="0 0 0" rpy="0 0 -1.57"/>
+        <origin xyz="0 0 0" rpy="0 0 -3.14159"/>
         <geometry>
           <xacro:get_mesh name="trolley" type="visual"/>

Commit message: updated ur10 frame (rotated by 180)

File: src/descriptions/urdf/ur_macro.xacro (robot description, xacro)
@@ -409,5 +409,5 @@
            Additional 90-degree rotation added for custom orientation.
       -->
-      <origin xyz="0 0 0" rpy="0 0 ${pi + pi/2}" />
+      <origin xyz="0 0 0" rpy="0 0 ${pi/2}" />
     </joint>
     <!-- ur robot shoulder link -->
