Commit message: added new vision cam jig and ur slider jig

File: src/descriptions/urdf/ur_macro.xacro (robot description, xacro)
@@ -336,5 +336,5 @@
       <parent link="${tf_prefix}ur10_trolley_link" />
       <child link="${tf_prefix}ur10_slider_jig_link" />
-      <origin xyz="0 0 0" rpy="0 0 0"/>
+      <origin xyz="0.025 -0.025 0" rpy="0 0 0"/>
     </joint>
     <!-- UR plate link-->

File: src/descriptions/urdf/vision.xacro (robot description, xacro)
@@ -64,5 +64,5 @@
       <parent link="vision_trolley_link" />
       <child link="vision_cam_jig_link" />
-      <origin xyz="-0.2 0.25 0.0" rpy="0 0 -2.35"/>
+      <origin xyz="-0.2 0.25 0.0" rpy="0 0 -1.57"/>
     </joint>
   </xacro:macro>

Commit message: added new ur slider jig plate

File: src/descriptions/urdf/ur_macro.xacro (robot description, xacro)
@@ -365,5 +365,5 @@
       <parent link="${tf_prefix}ur10_slider_jig_link" />
       <child link="${tf_prefix}ur10_plate_link" />
-      <origin xyz="-0.2 0 0.135" rpy="0 0 0"/>
+      <origin xyz="-0.277 0 0.1545" rpy="0 0 0"/>
       <axis xyz="1 0 0"/>
       <limit lower="-0.5" upper="0.5" effort="100" velocity="0.5" />
