Commit message: edited denso xacro to include yaml

File: src/descriptions/urdf/denso.xacro (robot description, xacro)
@@ -72,14 +72,14 @@
         <origin rpy="0 0 0" xyz="0 0 0"/>
         <geometry>
-          <mesh filename="file://$(find descriptions)/meshes/denso/denso_base_link.STL" scale="1 1 1"/>
-        </geometry>
-        <material name="">
-          <color rgba="0.7 0.7 0.7 1.0"/>
-        </material>
-      </visual>
-      <collision>
-        <origin rpy="0 0 0" xyz="0 0 0"/>
-        <geometry>
-          <mesh filename="file://$(find descriptions)/meshes/denso/denso_base_link.STL" scale="1 1 1"/>
+          <xacro:get_mesh name="denso_base_link" type="visual"/>
+        </geometry>
+        <material name="${sec_mesh_files['denso_base_link']['visual']['material']['name']}">
+          <color rgba="${sec_mesh_files['denso_base_link']['visual']['material']['color']}"/>
+        </material>
+      </visual>
+      <collision>
+        <origin rpy="0 0 0" xyz="0 0 0"/>
+        <geometry>
+          <xacro:get_mesh name="denso_base_link" type="collision"/>
         </geometry>
       </collision>
@@ -115,14 +115,14 @@
         <origin rpy="0 0 0" xyz="0 0 0"/>
         <geometry>
-          <mesh filename="file://$(find descriptions)/meshes/denso/denso_link1.STL" scale="1 1 1"/>
-        </geometry>
-        <material name="">
-          <color rgba="0.7 0.7 0.7 1.0"/>
-        </material>
-      </visual>
-      <collision>
-        <origin rpy="0 0 0" xyz="0 0 0"/>
-        <geometry>
-          <mesh filename="file://$(find descriptions)/meshes/denso/denso_link1.STL" scale="1 1 1"/>
+          <xacro:get_mesh name="denso_J1" type="visual"/>
+        </geometry>
+        <material name="${sec_mesh_files['denso_J1']['visual']['material']['name']}">
+          <color rgba="${sec_mesh_files['denso_J1']['visual']['material']['color']}"/>
+        </material>
+      </visual>
+      <collision>
+        <origin rpy="0 0 0" xyz="0 0 0"/>
+        <geometry>
+          <xacro:get_mesh name="denso_J1" type="collision"/>
         </geometry>
       </collision>
@@ -145,14 +145,14 @@
         <origin rpy="0 0 0" xyz="0 0 0"/>
         <geometry>
-          <mesh filename="file://$(find descriptions)/meshes/denso/denso_link2.STL" scale="1 1 1"/>
-        </geometry>
-        <material name="">
-          <color rgba="0.7 0.7 0.7 1.0"/>
-        </material>
-      </visual>
-      <collision>
-        <origin rpy="0 0 0" xyz="0 0 0"/>
-        <geometry>
-          <mesh filename="file://$(find descriptions)/meshes/denso/denso_link2.STL" scale="1 1 1"/>
+          <xacro:get_mesh name="denso_J2" type="visual"/>
+        </geometry>
+        <material name="${sec_mesh_files['denso_J2']['visual']['material']['name']}">
+          <color rgba="${sec_mesh_files['denso_J2']['visual']['material']['color']}"/>
+        </material>
+      </visual>
+      <collision>
+        <origin rpy="0 0 0" xyz="0 0 0"/>
+        <geometry>
+          <xacro:get_mesh name="denso_J2" type="collision"/>
         </geometry>
       </collision>
@@ -175,14 +175,14 @@
         <origin rpy="0 0 0" xyz="0 0 0"/>
         <geometry>
-          <mesh filename="file://$(find descriptions)/meshes/denso/denso_link3.STL" scale="1 1 1"/>
-        </geometry>
-        <material name="">
-          <color rgba="0.7 0.7 0.7 1.0"/>
-        </material>
-      </visual>
-      <collision>
-        <origin rpy="0 0 0" xyz="0 0 0"/>
-        <geometry>
-          <mesh filename="file://$(find descriptions)/meshes/denso/denso_link3.STL" scale="1 1 1"/>
+          <xacro:get_mesh name="denso_J3" type="visual"/>
+        </geometry>
+        <material name="${sec_mesh_files['denso_J3']['visual']['material']['name']}">
+          <color rgba="${sec_mesh_files['denso_J3']['visual']['material']['color']}"/>
+        </material>
+      </visual>
+      <collision>
+        <origin rpy="0 0 0" xyz="0 0 0"/>
+        <geometry>
+          <xacro:get_mesh name="denso_J3" type="collision"/>
         </geometry>
       </collision>
@@ -205,14 +205,14 @@
         <origin rpy="0 0 0" xyz="0 0 0"/>
         <geometry>
-          <cylinder radius="0.02" length="0.04"/>
-        </geometry>
-        <material name="">
-          <color rgba="0.7 0.7 0.7 1.0"/>
-        </material>
-      </visual>
-      <collision>
-        <origin rpy="0 0 0" xyz="0 0 0"/>
-        <geometry>
-          <cylinder radius="0.02" length="0.04"/>
+          <cylinder radius="${sec_mesh_files['denso_J4']['visual']['cylinder']['radius']}" length="${sec_mesh_files['denso_J4']['visual']['cylinder']['length']}"/>
+        </geometry>
+        <material name="${sec_mesh_files['denso_J4']['visual']['material']['name']}">
+          <color rgba="${sec_mesh_files['denso_J4']['visual']['material']['color']}"/>
+        </material>
+      </visual>
+      <collision>
+        <origin rpy="0 0 0" xyz="0 0 0"/>
+        <geometry>
+          <cylinder radius="${sec_mesh_files['denso_J4']['collision']['cylinder']['radius']}" length="${sec_mesh_files['denso_J4']['collision']['cylinder']['length']}"/>
         </geometry>
       </collision>
@@ -263,8 +263,8 @@
         <origin rpy="0 0 -1.57" xyz="0 0 0"/>
         <geometry>
-          <mesh filename="file://$(find descriptions)/meshes/denso/denso_screwdriver.STL" scale="1 1 1"/>
-        </geometry>
-        <material name="">
-          <color rgba="0.7 0.7 0.7 1.0"/>
+          <xacro:get_mesh name="denso_screwdriver" type="visual"/>
+        </geometry>
+        <material name="${sec_mesh_files['denso_screwdriver']['visual']['material']['name']}">
+          <color rgba="${sec_mesh_files['denso_screwdriver']['visual']['material']['color']}"/>
         </material>
       </visual>
@@ -272,5 +272,5 @@
         <origin rpy="0 0 -1.57" xyz="0 0 0"/>
         <geometry>
-          <mesh filename="file://$(find descriptions)/meshes/denso/denso_screwdriver.STL" scale="1 1 1"/>
+          <xacro:get_mesh name="denso_screwdriver" type="collision"/>
         </geometry>
       </collision>

Commit message: rotated denso base by 90

File: src/descriptions/urdf/denso.xacro (robot description, xacro)
@@ -122,5 +122,5 @@
       <parent link="denso_slider_jig_link"/>
       <child link="denso_base_link"/>
-      <origin rpy="0 0 0" xyz="0.01 0 0.084"/>
+      <origin rpy="0 0 -1.57" xyz="0.01 0 0.084"/>
       <axis xyz="1 0 0"/>
       <limit lower="-0.5" upper="0.5" effort="100" velocity="0.5" />

Commit message: updated denso joint limits to match real

File: src/descriptions/urdf/denso.xacro (robot description, xacro)
@@ -167,5 +167,5 @@
       <origin rpy="0.0 0.0 0.0" xyz="0.0 0.0 0.4135"/>
       <axis xyz="0.0 0.0 1.0"/>
-      <limit effort="50" lower="-2.26892802759263" upper="2.26892802759263" velocity="3.08615226990019"/>
+      <limit effort="50" lower="-2.87979" upper="2.87979" velocity="3.08615226990019"/>
       <dynamics damping="0.1" friction="0.01"/>
     </joint>
@@ -197,5 +197,5 @@
       <origin rpy="0.0 0.0 0.0" xyz="0.5 0.0 0.105"/>
       <axis xyz="0.0 0.0 1.0"/>
-      <limit effort="50" lower="-2.61799387799149" upper="2.61799387799149" velocity="5.41357500737341"/>
+      <limit effort="50" lower="-2.35619" upper="2.35619" velocity="5.41357500737341"/>
       <dynamics damping="0.1" friction="0.01"/>
     </joint>

Commit message: edited denso yaml and denso xacro - use yaml for stl etc

File: src/descriptions/urdf/denso.xacro (robot description, xacro)
@@ -101,14 +101,14 @@
         <origin rpy="0 0 0" xyz="0 0 0"/>
         <geometry>
-          <mesh filename="file://$(find descriptions)/meshes/denso/denso_base_link.STL" scale="1 1 1"/>
-        </geometry>
-        <material name="">
-          <color rgba="0.7 0.7 0.7 1.0"/>
-        </material>
-      </visual>
-      <collision>
-        <origin rpy="0 0 0" xyz="0 0 0"/>
-        <geometry>
-          <mesh filename="file://$(find descriptions)/meshes/denso/denso_base_link.STL" scale="1 1 1"/>
+          <xacro:get_mesh name="denso_base_link" type="visual"/>
+        </geometry>
+        <material name="${sec_mesh_files['denso_base_link']['visual']['material']['name']}">
+          <color rgba="${sec_mesh_files['denso_base_link']['visual']['material']['color']}"/>
+        </material>
+      </visual>
+      <collision>
+        <origin rpy="0 0 0" xyz="0 0 0"/>
+        <geometry>
+          <xacro:get_mesh name="denso_base_link" type="collision"/>
         </geometry>
       </collision>
@@ -122,5 +122,5 @@
       <parent link="denso_slider_jig_link"/>
       <child link="denso_base_link"/>
-      <origin rpy="0 0 -1.57" xyz="0.01 0 0.084"/>
+      <origin rpy="0 0 0" xyz="0.01 0 0.084"/>
       <axis xyz="1 0 0"/>
       <limit lower="-0.5" upper="0.5" effort="100" velocity="0.5" />
@@ -144,14 +144,14 @@
         <origin rpy="0 0 0" xyz="0 0 0"/>
         <geometry>
-          <mesh filename="file://$(find descriptions)/meshes/denso/denso_link1.STL" scale="1 1 1"/>
-        </geometry>
-        <material name="">
-          <color rgba="0.7 0.7 0.7 1.0"/>
-        </material>
-      </visual>
-      <collision>
-        <origin rpy="0 0 0" xyz="0 0 0"/>
-        <geometry>
-          <mesh filename="file://$(find descriptions)/meshes/denso/denso_link1.STL" scale="1 1 1"/>
+          <xacro:get_mesh name="denso_J1" type="visual"/>
+        </geometry>
+        <material name="${sec_mesh_files['denso_J1']['visual']['material']['name']}">
+          <color rgba="${sec_mesh_files['denso_J1']['visual']['material']['color']}"/>
+        </material>
+      </visual>
+      <collision>
+        <origin rpy="0 0 0" xyz="0 0 0"/>
+        <geometry>
+          <xacro:get_mesh name="denso_J1" type="collision"/>
         </geometry>
       </collision>
@@ -167,5 +167,5 @@
       <origin rpy="0.0 0.0 0.0" xyz="0.0 0.0 0.4135"/>
       <axis xyz="0.0 0.0 1.0"/>
-      <limit effort="50" lower="-2.87979" upper="2.87979" velocity="3.08615226990019"/>
+      <limit effort="50" lower="-2.26892802759263" upper="2.26892802759263" velocity="3.08615226990019"/>
       <dynamics damping="0.1" friction="0.01"/>
     </joint>
@@ -174,14 +174,14 @@
         <origin rpy="0 0 0" xyz="0 0 0"/>
         <geometry>
-          <mesh filename="file://$(find descriptions)/meshes/denso/denso_link2.STL" scale="1 1 1"/>
-        </geometry>
-        <material name="">
-          <color rgba="0.7 0.7 0.7 1.0"/>
-        </material>
-      </visual>
-      <collision>
-        <origin rpy="0 0 0" xyz="0 0 0"/>
-        <geometry>
-          <mesh filename="file://$(find descriptions)/meshes/denso/denso_link2.STL" scale="1 1 1"/>
+          <xacro:get_mesh name="denso_J2" type="visual"/>
+        </geometry>
+        <material name="${sec_mesh_files['denso_J2']['visual']['material']['name']}">
+          <color rgba="${sec_mesh_files['denso_J2']['visual']['material']['color']}"/>
+        </material>
+      </visual>
+      <collision>
+        <origin rpy="0 0 0" xyz="0 0 0"/>
+        <geometry>
+          <xacro:get_mesh name="denso_J2" type="collision"/>
         </geometry>
       </collision>
@@ -197,5 +197,5 @@
       <origin rpy="0.0 0.0 0.0" xyz="0.5 0.0 0.105"/>
       <axis xyz="0.0 0.0 1.0"/>
-      <limit effort="50" lower="-2.35619" upper="2.35619" velocity="5.41357500737341"/>
+      <limit effort="50" lower="-2.61799387799149" upper="2.61799387799149" velocity="5.41357500737341"/>
       <dynamics damping="0.1" friction="0.01"/>
     </joint>
@@ -204,14 +204,14 @@
         <origin rpy="0 0 0" xyz="0 0 0"/>
         <geometry>
-          <mesh filename="file://$(find descriptions)/meshes/denso/denso_link3.STL" scale="1 1 1"/>
-        </geometry>
-        <material name="">
-          <color rgba="0.7 0.7 0.7 1.0"/>
-        </material>
-      </visual>
-      <collision>
-        <origin rpy="0 0 0" xyz="0 0 0"/>
-        <geometry>
-          <mesh filename="file://$(find descriptions)/meshes/denso/denso_link3.STL" scale="1 1 1"/>
+          <xacro:get_mesh name="denso_J3" type="visual"/>
+        </geometry>
+        <material name="${sec_mesh_files['denso_J3']['visual']['material']['name']}">
+          <color rgba="${sec_mesh_files['denso_J3']['visual']['material']['color']}"/>
+        </material>
+      </visual>
+      <collision>
+        <origin rpy="0 0 0" xyz="0 0 0"/>
+        <geometry>
+          <xacro:get_mesh name="denso_J3" type="collision"/>
         </geometry>
       </collision>
@@ -234,14 +234,14 @@
         <origin rpy="0 0 0" xyz="0 0 0"/>
         <geometry>
-          <cylinder radius="0.02" length="0.04"/>
-        </geometry>
-        <material name="">
-          <color rgba="0.7 0.7 0.7 1.0"/>
-        </material>
-      </visual>
-      <collision>
-        <origin rpy="0 0 0" xyz="0 0 0"/>
-        <geometry>
-          <cylinder radius="0.02" length="0.04"/>
+          <cylinder radius="${sec_mesh_files['denso_J4']['visual']['cylinder']['radius']}" length="${sec_mesh_files['denso_J4']['visual']['cylinder']['length']}"/>
+        </geometry>
+        <material name="${sec_mesh_files['denso_J4']['visual']['material']['name']}">
+          <color rgba="${sec_mesh_files['denso_J4']['visual']['material']['color']}"/>
+        </material>
+      </visual>
+      <collision>
+        <origin rpy="0 0 0" xyz="0 0 0"/>
+        <geometry>
+          <cylinder radius="${sec_mesh_files['denso_J4']['collision']['cylinder']['radius']}" length="${sec_mesh_files['denso_J4']['collision']['cylinder']['length']}"/>
         </geometry>
       </collision>
@@ -292,8 +292,8 @@
         <origin rpy="0 0 -1.57" xyz="0 0 0"/>
         <geometry>
-          <mesh filename="file://$(find descriptions)/meshes/denso/denso_screwdriver.STL" scale="1 1 1"/>
-        </geometry>
-        <material name="">
-          <color rgba="0.7 0.7 0.7 1.0"/>
+          <xacro:get_mesh name="denso_screwdriver" type="visual"/>
+        </geometry>
+        <material name="${sec_mesh_files['denso_screwdriver']['visual']['material']['name']}">
+          <color rgba="${sec_mesh_files['denso_screwdriver']['visual']['material']['color']}"/>
         </material>
       </visual>
@@ -301,5 +301,5 @@
         <origin rpy="0 0 -1.57" xyz="0 0 0"/>
         <geometry>
-          <mesh filename="file://$(find descriptions)/meshes/denso/denso_screwdriver.STL" scale="1 1 1"/>
+          <xacro:get_mesh name="denso_screwdriver" type="collision"/>
         </geometry>
       </collision>

Commit message: changed denso axis to fixed and ur axis to prismatic

File: src/descriptions/urdf/denso.xacro (robot description, xacro)
@@ -119,11 +119,8 @@
       </inertial>
     </link>
-    <joint name="denso_axis_joint" type="prismatic">
+    <joint name="denso_axis_joint" type="fixed">
       <parent link="denso_slider_jig_link"/>
       <child link="denso_base_link"/>
       <origin rpy="0 0 0" xyz="0.01 0 0.084"/>
-      <axis xyz="1 0 0"/>
-      <limit lower="-0.5" upper="0.5" effort="100" velocity="0.5" />
-      <dynamics damping="0.5" friction="0.1"/>
     </joint>
     <link name="denso_dummy_link">

File: src/descriptions/urdf/ur_macro.xacro (robot description, xacro)
@@ -362,8 +362,11 @@
     </link>
     <!-- slider jig to UR plate joint -->
-    <joint name="${tf_prefix}ur10_plate_joint" type="fixed">
+    <joint name="${tf_prefix}ur_axis_joint" type="prismatic">
       <parent link="${tf_prefix}ur10_slider_jig_link" />
       <child link="${tf_prefix}ur10_plate_link" />
       <origin xyz="-0.2 0 0.135" rpy="0 0 0"/>
+      <axis xyz="1 0 0"/>
+      <limit lower="-0.5" upper="0.5" effort="100" velocity="0.5" />
+      <dynamics damping="0.5" friction="0.1"/>
     </joint>
     <!-- ur robot base link -->

File: src/descriptions/urdf/workcell.ros2_control.xacro (robot description, xacro)
@@ -144,4 +144,15 @@
         <state_interface name="effort"/>
       </joint>
+      <!-- UR Axis Joint -->
+      <joint name="ur_axis_joint">
+        <command_interface name="position"/>
+        <command_interface name="velocity"/>
+        <state_interface name="position">
+          <!-- initial position for the FakeSystem and simulation -->
+          <param name="initial_value">${initial_positions['ur_axis_joint']}</param>
+        </state_interface>
+        <state_interface name="velocity"/>
+        <state_interface name="effort"/>
+      </joint>
       <!-- ARF Axis Joints -->
       <joint name="${tf_prefix}arf_axis_1_joint">
@@ -270,15 +281,4 @@
           <!-- initial position for the FakeSystem and simulation -->
           <param name="initial_value">${initial_positions['denso_joint_4']}</param>
-        </state_interface>
-        <state_interface name="velocity"/>
-        <state_interface name="effort"/>
-      </joint>
-      <!-- Denso Axis Joint -->
-      <joint name="denso_axis_joint">
-        <command_interface name="position"/>
-        <command_interface name="velocity"/>
-        <state_interface name="position">
-          <!-- initial position for the FakeSystem and simulation -->
-          <param name="initial_value">${initial_positions['denso_axis_joint']}</param>
         </state_interface>
         <state_interface name="velocity"/>
